Commit message: frames aren't being associated heirarchally it seems

File: src/urdf_models/scte_vehicle/scte_description/urdf/scte_chassis.xacro (robot description, xacro)
@@ -9,7 +9,10 @@
     <!-- vehicle params-->
     <xacro:property name="scte_chassis_length" value="0.292"/>
-    <xacro:property name="scte_chassis_width" value="0.2159"/>
+    <xacro:property name="scte_chassis_width" value="0.165"/>
     <xacro:property name="scte_chassis_depth" value="0.0635"/> <!--value="0.127"/-->
     <xacro:property name="scte_total_mass" value="3.8"/>
+    <xacro:property name="scte_wheel_mass" value="0.5"/>
+    <xacro:property name="scte_wheel_radius" value="0.0508"/>
+    <xacro:property name="scte_wheel_depth" value="0.0508"/>
     <xacro:include filename="$(find scte_description)/urdf/scte.gazebo" />
     <xacro:include filename="$(find scte_description)/urdf/scte_diff.xacro"/>

File: src/urdf_models/scte_vehicle/scte_description/urdf/scte_diff.xacro (robot description, xacro)
@@ -1,4 +1,5 @@
 <?xml version="1.0"?>
 <robot>
+    <!-- FRONT DIFF AND AXLE -->
     <link name="scte_front_diff">
         <inertial>
@@ -38,12 +39,60 @@
             <origin xyz="${scte_chassis_length * 0.63} 0 0" rpy="0 0 0"/>
             <geometry>
-                <cylinder radius="${scte_chassis_depth * 0.1}" length="${scte_chassis_width * 1.11}"/>
-            </geometry>
-            <material name="red"/>
-        </visual>
-        <collision name='collision'>
-            <origin xyz="${scte_chassis_length * 0.63} 0 0" rpy="0 0 0"/>
-            <geometry>
-                <cylinder radius="${scte_chassis_depth * 0.1}" length="${scte_chassis_width * 1.11}"/>
+                <cylinder radius="${scte_chassis_depth * 0.1}" length="${scte_chassis_width * 1.46}"/>
+            </geometry>
+            <material name="red"/>
+        </visual>
+        <collision name='collision'>
+            <origin xyz="${scte_chassis_length * 0.63} 0 0" rpy="0 0 0"/>
+            <geometry>
+                <cylinder radius="${scte_chassis_depth * 0.1}" length="${scte_chassis_width * 1.46}"/>
+            </geometry>
+        </collision>
+    </link>
+    <link name="scte_front_left_wheel">
+        <inertial>
+            <mass value="${scte_wheel_mass / 4}"/>
+            <origin xyz="0 0 0" rpy="0 0 0"/>
+            <inertia
+                    ixx="1" ixy="0" ixz="0"
+                    iyy="1" iyz="0"
+                    izz="1"
+            />
+        </inertial>
+        <visual name='visual'>
+            <origin xyz="${scte_chassis_length * 0.63} 0 ${scte_chassis_width * 0.65}" rpy="0 0 0"/>
+            <geometry>
+                <cylinder radius="${scte_wheel_radius}" length="${scte_wheel_depth}"/>
+            </geometry>
+            <material name="green"/>
+        </visual>
+        <collision name='collision'>
+            <origin xyz="${scte_chassis_length * 0.63} 0 ${scte_chassis_width * 0.65}" rpy="0 0 0"/>
+            <geometry>
+                <cylinder radius="${scte_wheel_radius}" length="${scte_wheel_depth}"/>
+            </geometry>
+        </collision>
+    </link>
+    <link name="scte_front_right_wheel">
+        <inertial>
+            <mass value="${scte_wheel_mass / 4}"/>
+            <origin xyz="0 0 0" rpy="0 0 0"/>
+            <inertia
+                    ixx="1" ixy="0" ixz="0"
+                    iyy="1" iyz="0"
+                    izz="1"
+            />
+        </inertial>
+        <visual name='visual'>
+            <origin xyz="${scte_chassis_length * 0.63} 0 ${scte_chassis_width * 0.65 * -1}" rpy="0 0 0"/>
+            <geometry>
+                <cylinder radius="${scte_wheel_radius}" length="${scte_wheel_depth}"/>
+            </geometry>
+            <material name="green"/>
+        </visual>
+        <collision name='collision'>
+            <origin xyz="${scte_chassis_length * 0.63} 0 ${scte_chassis_width * 0.65 * -1}" rpy="0 0 0"/>
+            <geometry>
+                <cylinder radius="${scte_wheel_radius}" length="${scte_wheel_depth}"/>
             </geometry>
         </collision>
@@ -55,4 +104,17 @@
         <axis xyz="0 0 0" rpy="0 0 0"/>
     </joint>
+    <joint name='scte_front_axle_JOINT_scte_front_left_wheel' type='fixed'>
+        <origin xyz="0 0 0" rpy="0 0 0"/>
+        <parent link="scte_front_axle"/>
+        <child link="scte_front_left_wheel"/>
+        <axis xyz="0 0 0" rpy="0 0 0"/>
+    </joint>
+    <joint name='scte_front_axle_JOINT_scte_front_right_wheel' type='fixed'>
+        <origin xyz="0 0 0" rpy="0 0 0"/>
+        <parent link="scte_front_axle"/>
+        <child link="scte_front_right_wheel"/>
+        <axis xyz="0 0 0" rpy="0 0 0"/>
+    </joint>
+    <!-- REAR DIFF AND AXLE -->
     <link name="scte_rear_diff">
         <inertial>
@@ -92,15 +154,65 @@
             <origin xyz="${scte_chassis_length * 0.63 * -1} 0 0" rpy="0 0 0"/>
             <geometry>
-                <cylinder radius="${scte_chassis_depth * 0.1}" length="${scte_chassis_width * 1.11}"/>
-            </geometry>
-            <material name="red"/>
-        </visual>
-        <collision name='collision'>
-            <origin xyz="${scte_chassis_length * 0.63 * -1} 0 0" rpy="0 0 0"/>
-            <geometry>
-                <cylinder radius="${scte_chassis_depth * 0.1}" length="${scte_chassis_width * 1.11}"/>
-            </geometry>
-        </collision>
-    </link>
+                <cylinder radius="${scte_chassis_depth * 0.1}" length="${scte_chassis_width * 1.46}"/>
+            </geometry>
+            <material name="red"/>
+        </visual>
+        <collision name='collision'>
+            <origin xyz="${scte_chassis_length * 0.63 * -1} 0 0" rpy="0 0 0"/>
+            <geometry>
+                <cylinder radius="${scte_chassis_depth * 0.1}" length="${scte_chassis_width * 1.46}"/>
+            </geometry>
+        </collision>
+    </link>
+<!---->
+    <link name="scte_rear_left_wheel">
+        <inertial>
+            <mass value="${scte_wheel_mass / 4}"/>
+            <origin xyz="0 0 0" rpy="0 0 0"/>
+            <inertia
+                    ixx="1" ixy="0" ixz="0"
+                    iyy="1" iyz="0"
+                    izz="1"
+            />
+        </inertial> <!--${scte_chassis_length * 0.63 * 1.1}-->
+        <visual name='visual'>
+            <origin xyz="0 0 ${scte_chassis_width * 0.65}" rpy="0 0 0"/>
+            <geometry>
+                <cylinder radius="${scte_wheel_radius}" length="${scte_wheel_depth}"/>
+            </geometry>
+            <material name="red"/>
+        </visual>
+        <collision name='collision'>
+            <origin xyz="0 0 ${scte_chassis_width * 0.65}" rpy="0 0 0"/>
+            <geometry>
+                <cylinder radius="${scte_wheel_radius}" length="${scte_wheel_depth}"/>
+            </geometry>
+        </collision>
+    </link>
+    <link name="scte_rear_right_wheel">
+        <inertial>
+            <mass value="${scte_wheel_mass / 4}"/>
+            <origin xyz="0 0 0" rpy="0 0 0"/>
+            <inertia
+                    ixx="1" ixy="0" ixz="0"
+                    iyy="1" iyz="0"
+                    izz="1"
+            />
+        </inertial>
+        <visual name='visual'>
+            <origin xyz="${scte_chassis_length * 0.63} 0 ${scte_chassis_width * 0.65 * -1}" rpy="0 0 0"/>
+            <geometry>
+                <cylinder radius="${scte_wheel_radius}" length="${scte_wheel_depth}"/>
+            </geometry>
+            <material name="red"/>
+        </visual>
+        <collision name='collision'>
+            <origin xyz="${scte_chassis_length * 0.63} 0 ${scte_chassis_width * 0.65 * -1}" rpy="0 0 0"/>
+            <geometry>
+                <cylinder radius="${scte_wheel_radius}" length="${scte_wheel_depth}"/>
+            </geometry>
+        </collision>
+    </link>
+<!---->
     <joint name='scte_rear_diff_JOINT_scte_rear_axle' type='fixed'>
         <origin xyz="0 0 0" rpy="${M_PI/2} 0 0"/>
@@ -109,3 +221,17 @@
         <axis xyz="0 0 0" rpy="0 0 0"/>
     </joint>
+<!---->
+    <joint name='scte_rear_axle_JOINT_scte_rear_left_wheel' type='fixed'>
+        <origin xyz="0 0 0" rpy="0 0 0"/>
+        <parent link="scte_rear_axle"/>
+        <child link="scte_rear_left_wheel"/>
+        <axis xyz="0 0 0" rpy="0 0 0"/>
+    </joint>
+    <joint name='scte_rear_axle_JOINT_scte_rear_right_wheel' type='fixed'>
+        <origin xyz="0 0 0" rpy="0 0 0"/>
+        <parent link="scte_rear_axle"/>
+        <child link="scte_rear_right_wheel"/>
+        <axis xyz="0 0 0" rpy="0 0 0"/>
+    </joint>
+<!---->
 </robot>

Commit message: fixed the frames so that they are relative to the joint origins

File: src/urdf_models/scte_vehicle/scte_description/urdf/scte_chassis.xacro (robot description, xacro)
@@ -10,5 +10,5 @@
     <xacro:property name="scte_chassis_length" value="0.292"/>
     <xacro:property name="scte_chassis_width" value="0.165"/>
-    <xacro:property name="scte_chassis_depth" value="0.0635"/> <!--value="0.127"/-->
+    <xacro:property name="scte_chassis_depth" value="0.00635"/> <!--value="0.127"/-->
     <xacro:property name="scte_total_mass" value="3.8"/>
     <xacro:property name="scte_wheel_mass" value="0.5"/>
@@ -56,5 +56,5 @@
     </link>
     <joint name='scte_chassis_JOINT_scte_front_diff' type='fixed'>
-        <origin xyz="0 0 0" rpy="0 0 0"/>
+        <origin xyz="${scte_chassis_length * 0.63} 0 0" rpy="0 0 0"/>
         <parent link="scte_chassis"/>
         <child link="scte_front_diff"/>
@@ -62,5 +62,5 @@
     </joint>
     <joint name='scte_chassis_JOINT_scte_rear_diff' type='fixed'>
-        <origin xyz="0 0 0" rpy="0 0 0"/>
+        <origin xyz="${scte_chassis_length * 0.63 * -1} 0 0" rpy="0 0 0"/>
         <parent link="scte_chassis"/>
         <child link="scte_rear_diff"/>

File: src/urdf_models/scte_vehicle/scte_description/urdf/scte_diff.xacro (robot description, xacro)
@@ -5,13 +5,11 @@
         <inertial>
             <mass value="${scte_total_mass * 0.05}"/>
-            <origin xyz="0 0 0" rpy="0 0 0"/>
-            <inertia
-                    ixx="1" ixy="0" ixz="0"
-                    iyy="1" iyz="0"
-                    izz="1"
-            />
-        </inertial>
-        <visual name='visual'>
-            <origin xyz="${scte_chassis_length * 0.63} 0 0" rpy="0 0 0"/>
+            <inertia
+                    ixx="1" ixy="0" ixz="0"
+                    iyy="1" iyz="0"
+                    izz="1"
+            />
+        </inertial>
+        <visual name='visual'>
             <geometry>
                 <box size="${scte_chassis_length * 0.26} ${scte_chassis_width * 0.38} ${scte_chassis_depth}"/>
@@ -20,5 +18,4 @@
         </visual>
         <collision name='collision'>
-            <origin xyz="${scte_chassis_length * 0.63} 0 0" rpy="0 0 0"/>
             <geometry>
                 <box size="${scte_chassis_length * 0.26} ${scte_chassis_width * 0.38} ${scte_chassis_depth}"/>
@@ -29,22 +26,19 @@
         <inertial>
             <mass value="${scte_total_mass * 0.02}"/>
-            <origin xyz="0 0 0" rpy="0 0 0"/>
-            <inertia
-                    ixx="1" ixy="0" ixz="0"
-                    iyy="1" iyz="0"
-                    izz="1"
-            />
-        </inertial>
-        <visual name='visual'>
-            <origin xyz="${scte_chassis_length * 0.63} 0 0" rpy="0 0 0"/>
-            <geometry>
-                <cylinder radius="${scte_chassis_depth * 0.1}" length="${scte_chassis_width * 1.46}"/>
-            </geometry>
-            <material name="red"/>
-        </visual>
-        <collision name='collision'>
-            <origin xyz="${scte_chassis_length * 0.63} 0 0" rpy="0 0 0"/>
-            <geometry>
-                <cylinder radius="${scte_chassis_depth * 0.1}" length="${scte_chassis_width * 1.46}"/>
+            <inertia
+                    ixx="1" ixy="0" ixz="0"
+                    iyy="1" iyz="0"
+                    izz="1"
+            />
+        </inertial>
+        <visual name='visual'>
+            <geometry>
+                <cylinder radius="${scte_chassis_depth * 0.35}" length="${scte_chassis_width * 1.46}"/>
+            </geometry>
+            <material name="red"/>
+        </visual>
+        <collision name='collision'>
+            <geometry>
+                <cylinder radius="${scte_chassis_depth * 0.35}" length="${scte_chassis_width * 1.46}"/>
             </geometry>
         </collision>
@@ -53,13 +47,11 @@
         <inertial>
             <mass value="${scte_wheel_mass / 4}"/>
-            <origin xyz="0 0 0" rpy="0 0 0"/>
-            <inertia
-                    ixx="1" ixy="0" ixz="0"
-                    iyy="1" iyz="0"
-                    izz="1"
-            />
-        </inertial>
-        <visual name='visual'>
-            <origin xyz="${scte_chassis_length * 0.63} 0 ${scte_chassis_width * 0.65}" rpy="0 0 0"/>
+            <inertia
+                    ixx="1" ixy="0" ixz="0"
+                    iyy="1" iyz="0"
+                    izz="1"
+            />
+        </inertial>
+        <visual name='visual'>
             <geometry>
                 <cylinder radius="${scte_wheel_radius}" length="${scte_wheel_depth}"/>
@@ -68,5 +60,4 @@
         </visual>
         <collision name='collision'>
-            <origin xyz="${scte_chassis_length * 0.63} 0 ${scte_chassis_width * 0.65}" rpy="0 0 0"/>
             <geometry>
                 <cylinder radius="${scte_wheel_radius}" length="${scte_wheel_depth}"/>
@@ -77,13 +68,11 @@
         <inertial>
             <mass value="${scte_wheel_mass / 4}"/>
-            <origin xyz="0 0 0" rpy="0 0 0"/>
-            <inertia
-                    ixx="1" ixy="0" ixz="0"
-                    iyy="1" iyz="0"
-                    izz="1"
-            />
-        </inertial>
-        <visual name='visual'>
-            <origin xyz="${scte_chassis_length * 0.63} 0 ${scte_chassis_width * 0.65 * -1}" rpy="0 0 0"/>
+            <inertia
+                    ixx="1" ixy="0" ixz="0"
+                    iyy="1" iyz="0"
+                    izz="1"
+            />
+        </inertial>
+        <visual name='visual'>
             <geometry>
                 <cylinder radius="${scte_wheel_radius}" length="${scte_wheel_depth}"/>
@@ -92,5 +81,4 @@
         </visual>
         <collision name='collision'>
-            <origin xyz="${scte_chassis_length * 0.63} 0 ${scte_chassis_width * 0.65 * -1}" rpy="0 0 0"/>
             <geometry>
                 <cylinder radius="${scte_wheel_radius}" length="${scte_wheel_depth}"/>
@@ -105,5 +93,5 @@
     </joint>
     <joint name='scte_front_axle_JOINT_scte_front_left_wheel' type='fixed'>
-        <origin xyz="0 0 0" rpy="0 0 0"/>
+        <origin xyz="0 0 ${scte_chassis_width * 0.65 * -1}" rpy="0 0 0"/>
         <parent link="scte_front_axle"/>
         <child link="scte_front_left_wheel"/>
@@ -111,5 +99,5 @@
     </joint>
     <joint name='scte_front_axle_JOINT_scte_front_right_wheel' type='fixed'>
-        <origin xyz="0 0 0" rpy="0 0 0"/>
+        <origin xyz="0 0 ${scte_chassis_width * 0.65}" rpy="0 0 0"/>
         <parent link="scte_front_axle"/>
         <child link="scte_front_right_wheel"/>
@@ -120,20 +108,17 @@
         <inertial>
             <mass value="${scte_total_mass * 0.05}"/>
-            <origin xyz="0 0 0" rpy="0 0 0"/>
-            <inertia
-                    ixx="1" ixy="0" ixz="0"
-                    iyy="1" iyz="0"
-                    izz="1"
-            />
-        </inertial>
-        <visual name='visual'>
-            <origin xyz="${scte_chassis_length * 0.63 * -1} 0 0" rpy="0 0 0"/>
-            <geometry>
-                <box size="${scte_chassis_length * 0.26} ${scte_chassis_width * 0.38} ${scte_chassis_depth}"/>
-            </geometry>
-            <material name="red"/>
-        </visual>
-        <collision name='collision'>
-            <origin xyz="${scte_chassis_length * 0.63 * -1} 0 0" rpy="0 0 0"/>
+            <inertia
+                    ixx="1" ixy="0" ixz="0"
+                    iyy="1" iyz="0"
+                    izz="1"
+            />
+        </inertial>
+        <visual name='visual'>
+            <geometry>
+                <box size="${scte_chassis_length * 0.26} ${scte_chassis_width * 0.38} ${scte_chassis_depth}"/>
+            </geometry>
+            <material name="red"/>
+        </visual>
+        <collision name='collision'>
             <geometry>
                 <box size="${scte_chassis_length * 0.26} ${scte_chassis_width * 0.38} ${scte_chassis_depth}"/>
@@ -144,45 +129,38 @@
         <inertial>
             <mass value="${scte_total_mass * 0.02}"/>
-            <origin xyz="0 0 0" rpy="0 0 0"/>
-            <inertia
-                    ixx="1" ixy="0" ixz="0"
-                    iyy="1" iyz="0"
-                    izz="1"
-            />
-        </inertial>
-        <visual name='visual'>
-            <origin xyz="${scte_chassis_length * 0.63 * -1} 0 0" rpy="0 0 0"/>
-            <geometry>
-                <cylinder radius="${scte_chassis_depth * 0.1}" length="${scte_chassis_width * 1.46}"/>
-            </geometry>
-            <material name="red"/>
-        </visual>
-        <collision name='collision'>
-            <origin xyz="${scte_chassis_length * 0.63 * -1} 0 0" rpy="0 0 0"/>
-            <geometry>
-                <cylinder radius="${scte_chassis_depth * 0.1}" length="${scte_chassis_width * 1.46}"/>
-            </geometry>
-        </collision>
-    </link>
-<!---->
+            <inertia
+                    ixx="1" ixy="0" ixz="0"
+                    iyy="1" iyz="0"
+                    izz="1"
+            />
+        </inertial>
+        <visual name='visual'>
+            <geometry>
+                <cylinder radius="${scte_chassis_depth * 0.35}" length="${scte_chassis_width * 1.46}"/>
+            </geometry>
+            <material name="red"/>
+        </visual>
+        <collision name='collision'>
+            <geometry>
+                <cylinder radius="${scte_chassis_depth * 0.35}" length="${scte_chassis_width * 1.46}"/>
+            </geometry>
+        </collision>
+    </link>
     <link name="scte_rear_left_wheel">
         <inertial>
             <mass value="${scte_wheel_mass / 4}"/>
-            <origin xyz="0 0 0" rpy="0 0 0"/>
-            <inertia
-                    ixx="1" ixy="0" ixz="0"
-                    iyy="1" iyz="0"
-                    izz="1"
-            />
-        </inertial> <!--${scte_chassis_length * 0.63 * 1.1}-->
-        <visual name='visual'>
-            <origin xyz="0 0 ${scte_chassis_width * 0.65}" rpy="0 0 0"/>
-            <geometry>
-                <cylinder radius="${scte_wheel_radius}" length="${scte_wheel_depth}"/>
-            </geometry>
-            <material name="red"/>
-        </visual>
-        <collision name='collision'>
-            <origin xyz="0 0 ${scte_chassis_width * 0.65}" rpy="0 0 0"/>
+            <inertia
+                    ixx="1" ixy="0" ixz="0"
+                    iyy="1" iyz="0"
+                    izz="1"
+            />
+        </inertial>
+        <visual name='visual'>
+            <geometry>
+                <cylinder radius="${scte_wheel_radius}" length="${scte_wheel_depth}"/>
+            </geometry>
+            <material name="red"/>
+        </visual>
+        <collision name='collision'>
             <geometry>
                 <cylinder radius="${scte_wheel_radius}" length="${scte_wheel_depth}"/>
@@ -193,26 +171,22 @@
         <inertial>
             <mass value="${scte_wheel_mass / 4}"/>
-            <origin xyz="0 0 0" rpy="0 0 0"/>
-            <inertia
-                    ixx="1" ixy="0" ixz="0"
-                    iyy="1" iyz="0"
-                    izz="1"
-            />
-        </inertial>
-        <visual name='visual'>
-            <origin xyz="${scte_chassis_length * 0.63} 0 ${scte_chassis_width * 0.65 * -1}" rpy="0 0 0"/>
-            <geometry>
-                <cylinder radius="${scte_wheel_radius}" length="${scte_wheel_depth}"/>
-            </geometry>
-            <material name="red"/>
-        </visual>
-        <collision name='collision'>
-            <origin xyz="${scte_chassis_length * 0.63} 0 ${scte_chassis_width * 0.65 * -1}" rpy="0 0 0"/>
-            <geometry>
-                <cylinder radius="${scte_wheel_radius}" length="${scte_wheel_depth}"/>
-            </geometry>
-        </collision>
-    </link>
-<!---->
+            <inertia
+                    ixx="1" ixy="0" ixz="0"
+                    iyy="1" iyz="0"
+                    izz="1"
+            />
+        </inertial>
+        <visual name='visual'>
+            <geometry>
+                <cylinder radius="${scte_wheel_radius}" length="${scte_wheel_depth}"/>
+            </geometry>
+            <material name="red"/>
+        </visual>
+        <collision name='collision'>
+            <geometry>
+                <cylinder radius="${scte_wheel_radius}" length="${scte_wheel_depth}"/>
+            </geometry>
+        </collision>
+    </link>
     <joint name='scte_rear_diff_JOINT_scte_rear_axle' type='fixed'>
         <origin xyz="0 0 0" rpy="${M_PI/2} 0 0"/>
@@ -221,17 +195,15 @@
         <axis xyz="0 0 0" rpy="0 0 0"/>
     </joint>
-<!---->
+    <joint name='scte_rear_axle_JOINT_scte_rear_right_wheel' type='fixed'>
+        <origin xyz="0 0 ${scte_chassis_width * 0.65}" rpy="0 0 0"/>
+        <parent link="scte_rear_axle"/>
+        <child link="scte_rear_right_wheel"/>
+        <axis xyz="0 0 0" rpy="0 0 0"/>
+    </joint>
     <joint name='scte_rear_axle_JOINT_scte_rear_left_wheel' type='fixed'>
-        <origin xyz="0 0 0" rpy="0 0 0"/>
+        <origin xyz="0 0 ${scte_chassis_width * 0.65 * -1}" rpy="0 0 0"/>
         <parent link="scte_rear_axle"/>
         <child link="scte_rear_left_wheel"/>
         <axis xyz="0 0 0" rpy="0 0 0"/>
     </joint>
-    <joint name='scte_rear_axle_JOINT_scte_rear_right_wheel' type='fixed'>
-        <origin xyz="0 0 0" rpy="0 0 0"/>
-        <parent link="scte_rear_axle"/>
-        <child link="scte_rear_right_wheel"/>
-        <axis xyz="0 0 0" rpy="0 0 0"/>
-    </joint>
-<!---->
 </robot>
