Commit message: changes to scte chassis xacro, bringing dimensions out to the top level file

File: src/models/scte_vehicle/scte_description/urdf/scte_axle_components.xacro (robot description, xacro)
@@ -1,10 +1,27 @@
 <?xml version="1.0"?>
 <robot name="scte_diff_axle" xmlns:xacro="http://www.ros.org/wiki/xacro">
-    <xacro:macro name="scte_diff_axle" params="suffix parent_link joint_xyz joint_rpy">
-        <!--diff-->
-        <link name="diff_${suffix}">
-            <!--xacro:insert_block name="inertial"/>
-            <xacro:insert_block name="visual"/>
-            <xacro:insert_block name="collision"/-->
+    <xacro:macro name="scte_axle_components" params="suffix parent_link
+diff_plate_size
+diff_joint_xyz
+diff_joint_rpy
+drive_axle_radius
+drive_axle_length
+drive_axle_joint_origin
+drive_axle_joint_rpy
+shock_tower_size
+shock_tower_joint_origin
+shock_tower_joint_rpy">
+<!--
+left_wheel_radius
+left_wheel_length
+left_wheel_joint_origin
+left_wheel_joint_rpy
+right_wheel_radius
+right_wheel_length
+right_wheel_joint_origin
+right_wheel_joint_rpy">
+-->
+        <!--diff base plate-->
+        <link name="diff_base_plate_${suffix}">
             <intertial>
                 <mass value="${scte_total_mass * 0.05}"/>
@@ -17,5 +34,5 @@
             <visual>
                 <geometry>
-                    <box size="${scte_chassis_length * 0.26} ${scte_chassis_width * 0.38} ${scte_chassis_depth}"/>
+                    <box size="${diff_plate_size}"/>
                 </geometry>
                 <material name="green"/>
@@ -23,5 +40,5 @@
             <collision>
                 <geometry>
-                    <box size="${scte_chassis_length * 0.26} ${scte_chassis_width * 0.38} ${scte_chassis_depth}"/>
+                    <box size="${diff_plate_size}"/>
                 </geometry>
             </collision>
@@ -29,9 +46,40 @@
         <joint name="diff_${suffix}_JOINT_${parent_link}" type="fixed">
             <axis xyz="0 0 1"/>
-            <origin xyz="${joint_xyz}" rpy="${joint_rpy}"/>
+            <origin xyz="${diff_joint_xyz}" rpy="${diff_joint_rpy}"/>
             <parent link="${parent_link}"/>
-            <child link="diff_${suffix}"/>
+            <child link="diff_base_plate_${suffix}"/>
         </joint>
+        <!--shock tower-->
+        <!---->
+        <link name="shock_tower_${suffix}">
+            <inertial>
+                <mass value="${scte_wheel_mass / 4}"/>
+                <inertia
+                        ixx="1" ixy="0" ixz="0"
+                        iyy="1" iyz="0"
+                        izz="1"
+                />
+            </inertial>
+            <visual name='visual'>
+                <geometry>
+                    <box size="${shock_tower_size}"/>
+                </geometry>
+                <material name="red"/>
+            </visual>
+            <collision name='collision'>
+                <geometry>
+                    <box size="${shock_tower_size}"/>
+                </geometry>
+            </collision>
+        </link>
+        <joint name='shock_tower_${suffix}_JOINT_diff_${suffix}' type='fixed'>
+            <origin xyz="${shock_tower_joint_origin}" rpy="${shock_tower_joint_rpy}"/>
+            <parent link="diff_base_plate_${suffix}"/>
+            <child link="shock_tower_${suffix}"/>
+            <axis xyz="0 0 0" rpy="0 0 0"/>
+        </joint>
+        <!---->
         <!--axle-->
+        <!---->
         <link name="axle_${suffix}">
             <inertial>
@@ -45,5 +93,5 @@
             <visual name='visual'>
                 <geometry>
-                    <cylinder radius="${scte_chassis_depth * 0.35}" length="${scte_chassis_width * 1.46}"/>
+                    <cylinder radius="${drive_axle_radius}" length="${drive_axle_length}"/>
                 </geometry>
                 <material name="red"/>
@@ -51,15 +99,17 @@
             <collision name='collision'>
                 <geometry>
-                    <cylinder radius="${scte_chassis_depth * 0.35}" length="${scte_chassis_width * 1.46}"/>
+                    <cylinder radius="${drive_axle_radius}" length="${drive_axle_length}"/>
                 </geometry>
             </collision>
         </link>
         <joint name='diff_${suffix}_JOINT_axle_${suffix}' type='fixed'>
-            <origin xyz="0 0 0" rpy="${M_PI/2} 0 0"/>
-            <parent link="diff_${suffix}"/>
+            <origin xyz="${drive_axle_joint_origin}" rpy="${drive_axle_joint_rpy}"/>
+            <parent link="diff_base_plate_${suffix}"/>
             <child link="axle_${suffix}"/>
             <axis xyz="0 0 0" rpy="0 0 0"/>
         </joint>
+        <!---->
         <!--wheels-->
+        <!--
         <link name="left_wheel_${suffix}">
             <inertial>
@@ -73,5 +123,5 @@
             <visual name='visual'>
                 <geometry>
-                    <cylinder radius="${scte_wheel_radius}" length="${scte_wheel_depth}"/>
+                    <cylinder radius="${left_wheel_radius}" length="${left_wheel_length}"/>
                 </geometry>
                 <material name="green"/>
@@ -79,10 +129,10 @@
             <collision name='collision'>
                 <geometry>
-                    <cylinder radius="${scte_wheel_radius}" length="${scte_wheel_depth}"/>
+                    <cylinder radius="${left_wheel_radius}" length="${left_wheel_length}"/>
                 </geometry>
             </collision>
         </link>
         <joint name='left_wheel_${suffix}_JOINT_axle_${suffix}' type='fixed'>
-            <origin xyz="0 0 ${scte_chassis_width * -0.65}" rpy="0 0 0"/>
+            <origin xyz="${left_wheel_joint_origin}" rpy="${left_wheel_joint_rpy}"/>
             <parent link="axle_${suffix}"/>
             <child link="left_wheel_${suffix}"/>
@@ -100,5 +150,5 @@
             <visual name='visual'>
                 <geometry>
-                    <cylinder radius="${scte_wheel_radius}" length="${scte_wheel_depth}"/>
+                    <cylinder radius="${right_wheel_radius}" length="${right_wheel_length}"/>
                 </geometry>
                 <material name="red"/>
@@ -106,42 +156,15 @@
             <collision name='collision'>
                 <geometry>
-                    <cylinder radius="${scte_wheel_radius}" length="${scte_wheel_depth}"/>
+                    <cylinder radius="${right_wheel_radius}" length="${right_wheel_lengths}"/>
                 </geometry>
             </collision>
         </link>
         <joint name='right_wheel_${suffix}_JOINT_axle_${suffix}' type='fixed'>
-            <origin xyz="0 0 ${scte_chassis_width * 0.65}" rpy="0 0 0"/>
+            <origin xyz="${right_wheel_joint_origin}" rpy="${right_wheel_joint_rpy}"/>
             <parent link="axle_${suffix}"/>
             <child link="right_wheel_${suffix}"/>
             <axis xyz="0 0 0" rpy="0 0 0"/>
         </joint>
-        <!--shock tower-->
-        <link name="shock_tower_${suffix}">
-            <inertial>
-                <mass value="${scte_wheel_mass / 4}"/>
-                <inertia
-                        ixx="1" ixy="0" ixz="0"
-                        iyy="1" iyz="0"
-                        izz="1"
-                />
-            </inertial>
-            <visual name='visual'>
-                <geometry>
-                    <box size="${scte_chassis_depth} ${scte_chassis_length * 0.26} ${scte_chassis_width * 0.38}"/>
-                </geometry>
-                <material name="red"/>
-            </visual>
-            <collision name='collision'>
-                <geometry>
-                    <box size="${scte_chassis_depth} ${scte_chassis_length * 0.26} ${scte_chassis_width * 0.38}"/>
-                </geometry>
-            </collision>
-        </link>
-        <joint name='shock_tower_${suffix}_JOINT_diff_${suffix}' type='fixed'>
-            <origin xyz="0 0 ${scte_chassis_width * 0.38 / 2 + scte_chassis_depth / 2}" rpy="0 0 0"/>
-            <parent link="diff_${suffix}"/>
-            <child link="shock_tower_${suffix}"/>
-            <axis xyz="0 0 0" rpy="0 0 0"/>
-        </joint>
+        -->
     </xacro:macro>
 </robot>

File: src/models/scte_vehicle/scte_description/urdf/scte_chassis.xacro (robot description, xacro)
@@ -8,5 +8,15 @@
 <robot name="scteBot" xmlns:xacro="http://www.ros.org/wiki/xacro">
     <xacro:property name="M_PI" value="3.14159265358979323846264338327950288"/>
-    <!-- vehicle params-->
+    <xacro:include filename="$(find scte_description)/urdf/scte.gazebo" />
+    <xacro:include filename="$(find scte_description)/urdf/materials.xacro" />
+    <xacro:include filename="$(find scte_description)/urdf/macros.xacro" />
+    <link name="base_link">
+    </link>
+    <joint name="base_link" type="fixed">
+        <origin xyz="0 0.0 0.0" rpy="0 -0 0"/>
+        <parent link="base_link"/>
+        <child link="scte_chassis"/>
+    </joint>
+    <!--CHASSIS-->
     <xacro:property name="scte_chassis_length" value="0.292"/>
     <xacro:property name="scte_chassis_width" value="0.165"/>
@@ -16,19 +26,4 @@
     <xacro:property name="scte_wheel_radius" value="0.0508"/>
     <xacro:property name="scte_wheel_depth" value="0.0508"/>
-    <xacro:include filename="$(find scte_description)/urdf/scte.gazebo" />
-    <xacro:include filename="$(find scte_description)/urdf/materials.xacro" />
-    <xacro:include filename="$(find scte_description)/urdf/macros.xacro" />
-    <!--LIDAR-->
-    <!--xacro:include filename="$(find SOMESENSOR_description)/urdf/SENSOR.urdf.xacro"/>
-    <SOMESENSOR parent="scte_chassis" name="SOMESENSOR_sensor" hz="10" samples="220" lasers="16">
-        <origin xyz="0 0 0" rpy="0 0 0" />
-    </SOMESENSOR-->
-    <link name="base_link">
-    </link>
-    <joint name="base_link" type="fixed">
-        <origin xyz="0 0.0 0.0" rpy="0 -0 0"/>
-        <parent link="base_link"/>
-        <child link="scte_chassis"/>
-    </joint>
     <link name='scte_chassis'>
         <inertial>
@@ -55,11 +50,67 @@
         </collision>
     </link>
-    <xacro:include filename="$(find scte_description)/urdf/scte_diff_axle.xacro"/>
-    <xacro:scte_diff_axle suffix="scte_front" parent_link="scte_chassis" joint_xyz="${scte_chassis_length * 0.63} 0 0" joint_rpy="0 0 0"/>
-    <xacro:scte_diff_axle suffix="scte_rear" parent_link="scte_chassis" joint_xyz="${scte_chassis_length * -0.63} 0 0" joint_rpy="0 0 0"/>
+    <xacro:include filename="$(find scte_description)/urdf/scte_axle_components.xacro"/>
+    <xacro:scte_axle_components suffix="scte_front"
+        parent_link="scte_chassis"
+        diff_joint_xyz="${scte_chassis_length * 0.63} 0 0"
+        diff_joint_rpy="0 0 0"
+        diff_plate_size="0.07 0.07 ${scte_chassis_depth}"
+        drive_axle_radius="0.005"
+        drive_axle_length="0.25"
+        drive_axle_joint_origin="0 0 0.03"
+        drive_axle_joint_rpy="${M_PI/2} 0 0"
+        shock_tower_size="0.015 0.14 0.105"
+        shock_tower_joint_origin="0 0 ${0.105 * 0.5}"
+        shock_tower_joint_rpy="0 0 0"
+    />
+    <!--xacro:scte_diff_axle suffix="scte_rear" parent_link="scte_chassis" joint_xyz="${scte_chassis_length * -0.63} 0 0" joint_rpy="0 0 0"/-->
+    <!--CHASSIS-->
+    <!--mounting bards-->
+    <!--
+    <xacro:property name="mounting_bars_length_scale_value" value="1.60"/>
+    <xacro:property name="mounting_bars_width_scale_value" value="0.15"/>
+    <xacro:property name="mounting_bars_depth_scale_value" value="0.05"/>
+    <link name="driver_side_mounting_bar">
+        <inertial>
+            <mass value="${scte_total_mass * 0.02}"/>
+            <origin xyz="0 0 0" rpy="0 0 0"/>
+            <inertia
+                    ixx="1" ixy="0" ixz="0"
+                    iyy="1" iyz="0"
+                    izz="1"
+            />
+        </inertial>
+        <visual name='visual'>
+            <origin xyz="${scte_chassis_length * -0.63} 0 0" rpy="0 0 0"/>
+            <geometry>
+                <box size="${scte_chassis_length * mounting_bars_length_scale_value} ${scte_chassis_width * mounting_bars_width_scale_value} ${scte_chassis_depth * mounting_bars_depth_scale_value}"/>
+            </geometry>
+            <material name="green"/>
+        </visual>
+        <collision name='collision'>
+            <origin xyz="${scte_chassis_length * -0.63} 0 0" rpy="0 0 0"/>
+            <geometry>
+                <box size="${scte_chassis_length * mounting_bars_length_scale_value} ${scte_chassis_width * mounting_bars_width_scale_value} ${scte_chassis_depth * mounting_bars_depth_scale_value}"/>
+            </geometry>
+        </collision>
+    </link>
+    <joint name="shock_tower_scte_front_LINKED_driver_side_mounting_bar" type="fixed">
+        <origin xyz="0 0.0 0.0" rpy="0 -0 0"/>
+        <parent link="shock_tower_scte_front"/>
+        <child link="driver_side_mounting_bar"/>
+    </joint>
+    -->
+    <!-- chassis -->
     <!--sensors-->
+    <!--
     <xacro:include filename="$(find logitech_c270_camera)/urdf/logitech_c270.xacro"/>
     <xacro:logitech_c270_camera parent_link="axle_scte_front" camera_link="left_cam" joint_xyz="0 0.15 ${scte_chassis_width * 0.65 * -1.0}" joint_rpy="0 0 0"/>
     <xacro:logitech_c270_camera parent_link="axle_scte_front" camera_link="right_cam" joint_xyz="0 0.15 ${scte_chassis_width * 0.65}" joint_rpy="0 0 0"/>
+    -->
+    <!--LIDAR-->
+    <!--xacro:include filename="$(find SOMESENSOR_description)/urdf/SENSOR.urdf.xacro"/>
+    <SOMESENSOR parent="scte_chassis" name="SOMESENSOR_sensor" hz="10" samples="220" lasers="16">
+        <origin xyz="0 0 0" rpy="0 0 0" />
+    </SOMESENSOR-->
     <!--link name='main_computer'>
     <inertial>

Commit message: axles added

File: src/models/scte_vehicle/scte_description/urdf/scte_axle_components.xacro (robot description, xacro)
@@ -11,6 +11,5 @@
 shock_tower_size
 shock_tower_joint_origin
-shock_tower_joint_rpy">
-<!--
+shock_tower_joint_rpy
 left_wheel_radius
 left_wheel_length
@@ -21,5 +20,4 @@
 right_wheel_joint_origin
 right_wheel_joint_rpy">
--->
         <!--diff base plate-->
         <link name="diff_base_plate_${suffix}">
@@ -111,5 +109,5 @@
         <!---->
         <!--wheels-->
-        <!--
+        <!---->
         <link name="left_wheel_${suffix}">
             <inertial>
@@ -139,4 +137,5 @@
             <axis xyz="0 0 0" rpy="0 0 0"/>
         </joint>
+        <!---->
         <link name="right_wheel_${suffix}">
             <inertial>
@@ -156,5 +155,5 @@
             <collision name='collision'>
                 <geometry>
-                    <cylinder radius="${right_wheel_radius}" length="${right_wheel_lengths}"/>
+                    <cylinder radius="${right_wheel_radius}" length="${right_wheel_length}"/>
                 </geometry>
             </collision>
@@ -166,5 +165,5 @@
             <axis xyz="0 0 0" rpy="0 0 0"/>
         </joint>
-        -->
+        <!---->
     </xacro:macro>
 </robot>

File: src/models/scte_vehicle/scte_description/urdf/scte_chassis.xacro (robot description, xacro)
@@ -51,4 +51,6 @@
     </link>
     <xacro:include filename="$(find scte_description)/urdf/scte_axle_components.xacro"/>
+    <xacro:property name="drive_axle_length" value="0.25"/>
+    <xacro:property name="drive_axle_radius" value="0.005"/>
     <xacro:scte_axle_components suffix="scte_front"
         parent_link="scte_chassis"
@@ -56,13 +58,41 @@
         diff_joint_rpy="0 0 0"
         diff_plate_size="0.07 0.07 ${scte_chassis_depth}"
-        drive_axle_radius="0.005"
-        drive_axle_length="0.25"
-        drive_axle_joint_origin="0 0 0.03"
+        drive_axle_radius="${drive_axle_radius}"
+        drive_axle_length="${drive_axle_length}"
+        drive_axle_joint_origin="0 0 ${0.03 * 0.5}"
         drive_axle_joint_rpy="${M_PI/2} 0 0"
         shock_tower_size="0.015 0.14 0.105"
         shock_tower_joint_origin="0 0 ${0.105 * 0.5}"
         shock_tower_joint_rpy="0 0 0"
+        left_wheel_radius="0.05"
+        left_wheel_length="0.045"
+        left_wheel_joint_origin="0 0 ${drive_axle_length * 0.5}"
+        left_wheel_joint_rpy="0 0 0"
+        right_wheel_radius="0.05"
+        right_wheel_length="0.045"
+        right_wheel_joint_origin="0 0 ${drive_axle_length * -0.5}"
+        right_wheel_joint_rpy="0 0 0"
     />
-    <!--xacro:scte_diff_axle suffix="scte_rear" parent_link="scte_chassis" joint_xyz="${scte_chassis_length * -0.63} 0 0" joint_rpy="0 0 0"/-->
+    <xacro:scte_axle_components suffix="scte_rear"
+        parent_link="scte_chassis"
+        diff_joint_xyz="${scte_chassis_length * -0.63} 0 0"
+        diff_joint_rpy="0 0 0"
+        diff_plate_size="0.07 0.07 ${scte_chassis_depth}"
+        drive_axle_radius="${drive_axle_radius}"
+        drive_axle_length="${drive_axle_length}"
+        drive_axle_joint_origin="0 0 ${0.03 * 0.5}"
+        drive_axle_joint_rpy="${M_PI/2} 0 0"
+        shock_tower_size="0.015 0.14 0.105"
+        shock_tower_joint_origin="0 0 ${0.105 * 0.5}"
+        shock_tower_joint_rpy="0 0 0"
+        left_wheel_radius="0.05"
+        left_wheel_length="0.045"
+        left_wheel_joint_origin="0 0 ${drive_axle_length * 0.5}"
+        left_wheel_joint_rpy="0 0 0"
+        right_wheel_radius="0.05"
+        right_wheel_length="0.045"
+        right_wheel_joint_origin="0 0 ${drive_axle_length * -0.5}"
+        right_wheel_joint_rpy="0 0 0"
+    />
     <!--CHASSIS-->
     <!--mounting bards-->
