Commit message: added bumpers

File: src/models/scte_vehicle/scte_description/urdf/scte_axle_components.xacro (robot description, xacro)
@@ -43,14 +43,128 @@
         </link>
         <joint name="diff_${suffix}_JOINT_${parent_link}" type="fixed">
-            <axis xyz="0 0 1"/>
+            <axis xyz="0 0 0"/>
             <origin xyz="${diff_joint_xyz}" rpy="${diff_joint_rpy}"/>
             <parent link="${parent_link}"/>
             <child link="diff_base_plate_${suffix}"/>
         </joint>
+        <!--front bumper plate-->
+        <xacro:if value="${suffix == 'scte_front'}">
+        <link name="diff_base_bumper_plate_${suffix}">
+            <intertial>
+                <mass value="${scte_total_mass * 0.05}"/>
+                <inertia
+                        ixx="1" ixy="0" ixz="0"
+                        iyy="1" iyz="0"
+                        izz="1"
+                />
+            </intertial>
+            <visual>
+                <geometry>
+                    <box size="${diff_plate_size}"/>
+                </geometry>
+                <material name="red"/>
+            </visual>
+            <collision>
+                <geometry>
+                    <box size="${diff_plate_size}"/>
+                </geometry>
+            </collision>
+        </link>
+        <joint name="diff_bumper_${suffix}_JOINT_${parent_link}" type="fixed">
+            <axis xyz="0 0 0"/>
+            <origin xyz="${0.07} 0 ${0.07 * 0.30}" rpy="0 ${M_PI/-6}  0"/>
+            <parent link="diff_base_plate_${suffix}"/>
+            <child link="diff_base_bumper_plate_${suffix}"/>
+        </joint>
+        <link name="bumper_${suffix}">
+            <intertial>
+                <mass value="${scte_total_mass * 0.05}"/>
+                <inertia
+                        ixx="1" ixy="0" ixz="0"
+                        iyy="1" iyz="0"
+                        izz="1"
+                />
+            </intertial>
+            <visual>
+                <geometry>
+                    <box size="0.01 0.175 0.05"/>
+                </geometry>
+                <material name="red"/>
+            </visual>
+            <collision>
+                <geometry>
+                    <box size="0.01 0.175 0.05"/>
+                </geometry>
+            </collision>
+        </link>
+        <joint name="bumper_${suffix}_JOINT_${parent_link}" type="fixed">
+            <axis xyz="0 0 0"/>
+            <origin xyz="${0.07 * 0.70} 0 ${0.07 * 0.35}" rpy="0 ${M_PI/6} 0"/>
+            <parent link="diff_base_bumper_plate_${suffix}"/>
+            <child link="bumper_${suffix}"/>
+        </joint>
+        </xacro:if>
+        <!--rear bumper assembly-->
+        <xacro:if value="${suffix == 'scte_rear'}">
+        <link name="diff_base_bumper_plate_${suffix}">
+            <intertial>
+                <mass value="${scte_total_mass * 0.05}"/>
+                <inertia
+                        ixx="1" ixy="0" ixz="0"
+                        iyy="1" iyz="0"
+                        izz="1"
+                />
+            </intertial>
+            <visual>
+                <geometry>
+                    <box size="0.09 0.05 0.05"/>
+                </geometry>
+                <material name="red"/>
+            </visual>
+            <collision>
+                <geometry>
+                    <box size="0.09 0.05 0.05"/>
+                </geometry>
+            </collision>
+        </link>
+        <joint name="diff_bumper_${suffix}_JOINT_${parent_link}" type="fixed">
+            <axis xyz="0 0 0"/>
+            <origin xyz="${0.09 * -0.5} 0 0" rpy="0 0 0"/>
+            <parent link="shock_tower_${suffix}"/>
+            <child link="diff_base_bumper_plate_${suffix}"/>
+        </joint>
+        <link name="bumper_${suffix}">
+            <intertial>
+                <mass value="${scte_total_mass * 0.05}"/>
+                <inertia
+                        ixx="1" ixy="0" ixz="0"
+                        iyy="1" iyz="0"
+                        izz="1"
+                />
+            </intertial>
+            <visual>
+                <geometry>
+                    <box size="0.01 0.255 0.05"/>
+                </geometry>
+                <material name="red"/>
+            </visual>
+            <collision>
+                <geometry>
+                    <box size="0.01 0.255 0.05"/>
+                </geometry>
+            </collision>
+        </link>
+        <joint name="bumper_${suffix}_JOINT_${parent_link}" type="fixed">
+            <axis xyz="0 0 0"/>
+            <origin xyz="${0.09 * -0.5} 0 0.015" rpy="0 0 0"/>
+            <parent link="diff_base_bumper_plate_${suffix}"/>
+            <child link="bumper_${suffix}"/>
+        </joint>
+        </xacro:if>
         <!--shock tower-->
         <!---->
         <link name="shock_tower_${suffix}">
             <inertial>
-                <mass value="${scte_wheel_mass / 4}"/>
+                <mass value="${scte_total_mass * 0.25 * 0.05}"/>
                 <inertia
                         ixx="1" ixy="0" ixz="0"
@@ -112,5 +226,5 @@
         <link name="left_wheel_${suffix}">
             <inertial>
-                <mass value="${scte_wheel_mass / 4}"/>
+                <mass value="${scte_total_mass * 0.25 * 0.05}"/>
                 <inertia
                         ixx="1" ixy="0" ixz="0"
@@ -140,5 +254,5 @@
         <link name="right_wheel_${suffix}">
             <inertial>
-                <mass value="${scte_wheel_mass / 4}"/>
+                <mass value="${scte_total_mass * 0.25 * 0.05}"/>
                 <inertia
                         ixx="1" ixy="0" ixz="0"

File: src/models/scte_vehicle/scte_description/urdf/scte_chassis.xacro (robot description, xacro)
@@ -19,11 +19,8 @@
     </joint>
     <!--CHASSIS-->
+    <xacro:property name="scte_total_mass" value="3.8"/>
     <xacro:property name="scte_chassis_length" value="0.292"/>
     <xacro:property name="scte_chassis_width" value="0.165"/>
-    <xacro:property name="scte_chassis_depth" value="0.00635"/> <!--value="0.127"/-->
-    <xacro:property name="scte_total_mass" value="3.8"/>
-    <xacro:property name="scte_wheel_mass" value="0.5"/>
-    <xacro:property name="scte_wheel_radius" value="0.0508"/>
-    <xacro:property name="scte_wheel_depth" value="0.0508"/>
+    <xacro:property name="scte_chassis_depth" value="0.00635"/>
     <link name='scte_chassis'>
         <inertial>
@@ -53,4 +50,6 @@
     <xacro:property name="drive_axle_length" value="0.25"/>
     <xacro:property name="drive_axle_radius" value="0.005"/>
+    <xacro:property name="shock_tower_height" value="0.105"/>
+    <xacro:property name="shock_tower_width" value="0.14"/>
     <xacro:scte_axle_components suffix="scte_front"
         parent_link="scte_chassis"
@@ -62,6 +61,6 @@
         drive_axle_joint_origin="0 0 ${0.03 * 0.5}"
         drive_axle_joint_rpy="${M_PI/2} 0 0"
-        shock_tower_size="0.015 0.14 0.105"
-        shock_tower_joint_origin="0 0 ${0.105 * 0.5}"
+        shock_tower_size="0.015 ${shock_tower_width} ${shock_tower_height}"
+        shock_tower_joint_origin="0 0 ${shock_tower_height * 0.5}"
         shock_tower_joint_rpy="0 0 0"
         left_wheel_radius="0.05"
@@ -83,6 +82,6 @@
         drive_axle_joint_origin="0 0 ${0.03 * 0.5}"
         drive_axle_joint_rpy="${M_PI/2} 0 0"
-        shock_tower_size="0.015 0.14 0.105"
-        shock_tower_joint_origin="0 0 ${0.105 * 0.5}"
+        shock_tower_size="0.015 ${shock_tower_width} ${shock_tower_height}"
+        shock_tower_joint_origin="0 0 ${shock_tower_height * 0.5}"
         shock_tower_joint_rpy="0 0 0"
         left_wheel_radius="0.05"
@@ -95,10 +94,10 @@
         right_wheel_joint_rpy="0 0 0"
     />
-    <!--CHASSIS-->
-    <!--mounting bards-->
-    <!--
-    <xacro:property name="mounting_bars_length_scale_value" value="1.60"/>
-    <xacro:property name="mounting_bars_width_scale_value" value="0.15"/>
-    <xacro:property name="mounting_bars_depth_scale_value" value="0.05"/>
+    <!--/CHASSIS-->
+    <!--MOUNTING BARS-->
+    <!---->
+    <xacro:property name="mounting_bars_length" value="0.45"/>
+    <xacro:property name="mounting_bars_width" value="0.025"/>
+    <xacro:property name="mounting_bars_depth" value="0.005"/>
     <link name="driver_side_mounting_bar">
         <inertial>
@@ -112,24 +111,53 @@
         </inertial>
         <visual name='visual'>
-            <origin xyz="${scte_chassis_length * -0.63} 0 0" rpy="0 0 0"/>
+            <origin xyz="0 0 0" rpy="0 0 0"/>
             <geometry>
-                <box size="${scte_chassis_length * mounting_bars_length_scale_value} ${scte_chassis_width * mounting_bars_width_scale_value} ${scte_chassis_depth * mounting_bars_depth_scale_value}"/>
+                <box size="${mounting_bars_length} ${mounting_bars_width} ${mounting_bars_depth}"/>
             </geometry>
             <material name="green"/>
         </visual>
         <collision name='collision'>
-            <origin xyz="${scte_chassis_length * -0.63} 0 0" rpy="0 0 0"/>
+            <origin xyz="0 0 0" rpy="0 0 0"/>
             <geometry>
-                <box size="${scte_chassis_length * mounting_bars_length_scale_value} ${scte_chassis_width * mounting_bars_width_scale_value} ${scte_chassis_depth * mounting_bars_depth_scale_value}"/>
+                <box size="${mounting_bars_length} ${mounting_bars_width} ${mounting_bars_depth}"/>
             </geometry>
         </collision>
     </link>
     <joint name="shock_tower_scte_front_LINKED_driver_side_mounting_bar" type="fixed">
-        <origin xyz="0 0.0 0.0" rpy="0 -0 0"/>
+        <origin xyz="${scte_chassis_length * -0.63} ${shock_tower_width * 0.5} ${shock_tower_height * 0.5}" rpy="0 -0 0"/>
         <parent link="shock_tower_scte_front"/>
         <child link="driver_side_mounting_bar"/>
     </joint>
-    -->
-    <!-- chassis -->
+    <link name="passenger_side_mounting_bar">
+        <inertial>
+            <mass value="${scte_total_mass * 0.02}"/>
+            <origin xyz="0 0 0" rpy="0 0 0"/>
+            <inertia
+                    ixx="1" ixy="0" ixz="0"
+                    iyy="1" iyz="0"
+                    izz="1"
+            />
+        </inertial>
+        <visual name='visual'>
+            <origin xyz="0 0 0" rpy="0 0 0"/>
+            <geometry>
+                <box size="${mounting_bars_length} ${mounting_bars_width} ${mounting_bars_depth}"/>
+            </geometry>
+            <material name="green"/>
+        </visual>
+        <collision name='collision'>
+            <origin xyz="0 0 0" rpy="0 0 0"/>
+            <geometry>
+                <box size="${mounting_bars_length} ${mounting_bars_width} ${mounting_bars_depth}"/>
+            </geometry>
+        </collision>
+    </link>
+    <joint name="shock_tower_scte_front_LINKED_passenger_side_mounting_bar" type="fixed">
+        <origin xyz="${scte_chassis_length * -0.63} ${shock_tower_width * -0.5} ${shock_tower_height * 0.5}" rpy="0 -0 0"/>
+        <parent link="shock_tower_scte_front"/>
+        <child link="passenger_side_mounting_bar"/>
+    </joint>
+    <!---->
+    <!--/MOUNTING BARS-->
     <!--sensors-->
     <!--

Commit message: got the wheels to turn in gazebo using the scte urdf model

File: src/models/scte_vehicle/scte_description/urdf/scte_axle_components.xacro (robot description, xacro)
@@ -245,9 +245,11 @@
             </collision>
         </link>
-        <joint name='left_wheel_${suffix}_JOINT_axle_${suffix}' type='fixed'>
+        <joint name='left_wheel_${suffix}_JOINT_axle_${suffix}' type='revolute'>
             <origin xyz="${left_wheel_joint_origin}" rpy="${left_wheel_joint_rpy}"/>
             <parent link="axle_${suffix}"/>
             <child link="left_wheel_${suffix}"/>
-            <axis xyz="0 0 0" rpy="0 0 0"/>
+            <axis xyz="0 0 1" rpy="0 0 0"/>
+            <limit effort="-1" velocity="-1" lower="-2147483647" upper="2147483647"/>
+            <axis xyz="0 0 1"/>
         </joint>
         <!---->
@@ -273,9 +275,11 @@
             </collision>
         </link>
-        <joint name='right_wheel_${suffix}_JOINT_axle_${suffix}' type='fixed'>
+        <joint name='right_wheel_${suffix}_JOINT_axle_${suffix}' type='revolute'>
             <origin xyz="${right_wheel_joint_origin}" rpy="${right_wheel_joint_rpy}"/>
             <parent link="axle_${suffix}"/>
             <child link="right_wheel_${suffix}"/>
-            <axis xyz="0 0 0" rpy="0 0 0"/>
+            <axis xyz="0 0 1" rpy="0 0 0"/>
+            <limit effort="-1" velocity="-1" lower="-2147483647" upper="2147483647"/>
+            <axis xyz="0 0 1"/>
         </joint>
         <!---->

File: src/models/scte_vehicle/scte_description/urdf/scte_chassis.xacro (robot description, xacro)
@@ -5,4 +5,7 @@
 https://wiki.ros.org/action/fullsearch/urdf/Tutorials/Building%20a%20Visual%20Robot%20Model%20with%20URDF%20from%20Scratch?action=fullsearch&context=180&value=linkto%3A%22urdf%2FTutorials%2FBuilding+a+Visual+Robot+Model+with+URDF+from+Scratch%22
 http://wiki.ros.org/xacro
+http://wiki.ros.org/urdf/Tutorials/Building%20a%20Visual%20Robot%20Model%20with%20URDF%20from%20Scratch
+http://wiki.ros.org/urdf/Tutorials/Building%20a%20Movable%20Robot%20Model%20with%20URDF
+http://wiki.ros.org/urdf/XML/joint#Elements
 -->
 <robot name="scteBot" xmlns:xacro="http://www.ros.org/wiki/xacro">
@@ -19,4 +22,5 @@
     </joint>
     <!--DEBUG test link for odom testing-->
+    <!--
     <link name="test_real_link">
         <inertial>
@@ -51,4 +55,5 @@
         <child link="test_real_link"/>
     </joint>
+    -->
     <!--DEBUG test link for odom testing-->
     <!--CHASSIS-->

Commit message: tweaked xarco files and added supporting files based on gazebo rrbot example with goal of controlling the RC in gazebo and having that reflected in RViz

File: src/models/scte_vehicle/scte_description/urdf/scte_axle_components.xacro (robot description, xacro)
@@ -49,5 +49,5 @@
         </joint>
         <!--front bumper plate-->
-        <xacro:if value="${suffix == 'scte_front'}">
+        <xacro:if value="${suffix == 'front'}">
         <link name="diff_base_bumper_plate_${suffix}">
             <intertial>
@@ -106,5 +106,5 @@
         </xacro:if>
         <!--rear bumper assembly-->
-        <xacro:if value="${suffix == 'scte_rear'}">
+        <xacro:if value="${suffix == 'rear'}">
         <link name="diff_base_bumper_plate_${suffix}">
             <intertial>
@@ -245,12 +245,22 @@
             </collision>
         </link>
-        <joint name='left_wheel_${suffix}_JOINT_axle_${suffix}' type='revolute'>
+        <joint name='left_wheel_${suffix}_JOINT_axle_${suffix}' type='continuous'>
             <origin xyz="${left_wheel_joint_origin}" rpy="${left_wheel_joint_rpy}"/>
             <parent link="axle_${suffix}"/>
             <child link="left_wheel_${suffix}"/>
             <axis xyz="0 0 1" rpy="0 0 0"/>
-            <limit effort="-1" velocity="-1" lower="-2147483647" upper="2147483647"/>
             <axis xyz="0 0 1"/>
-        </joint>
+            <dynamics damping="0.7"/>
+        </joint>
+        <transmission name="tran_left_wheel_${suffix}">
+            <type>transmission_interface/SimpleTransmission</type>
+            <joint name="left_wheel_${suffix}_JOINT_axle_${suffix}">
+                <hardwareInterface>hardware_interface/EffortJointInterface</hardwareInterface>
+            </joint>
+            <actuator name="motor_left_wheel_${suffix}">
+                <hardwareInterface>hardware_interface/EffortJointInterface</hardwareInterface>
+                <mechanicalReduction>1</mechanicalReduction>
+            </actuator>
+        </transmission>
         <!---->
         <link name="right_wheel_${suffix}">
@@ -275,12 +285,22 @@
             </collision>
         </link>
-        <joint name='right_wheel_${suffix}_JOINT_axle_${suffix}' type='revolute'>
+        <joint name='right_wheel_${suffix}_JOINT_axle_${suffix}' type='continuous'>
             <origin xyz="${right_wheel_joint_origin}" rpy="${right_wheel_joint_rpy}"/>
             <parent link="axle_${suffix}"/>
             <child link="right_wheel_${suffix}"/>
             <axis xyz="0 0 1" rpy="0 0 0"/>
-            <limit effort="-1" velocity="-1" lower="-2147483647" upper="2147483647"/>
             <axis xyz="0 0 1"/>
-        </joint>
+            <dynamics damping="0.7"/>
+        </joint>
+        <transmission name="tran_right_wheel_${suffix}">
+            <type>transmission_interface/SimpleTransmission</type>
+            <joint name="right_wheel_${suffix}_JOINT_axle_${suffix}">
+                <hardwareInterface>hardware_interface/EffortJointInterface</hardwareInterface>
+            </joint>
+            <actuator name="motor_right_wheel_${suffix}">
+                <hardwareInterface>hardware_interface/EffortJointInterface</hardwareInterface>
+                <mechanicalReduction>1</mechanicalReduction>
+            </actuator>
+        </transmission>
         <!---->
     </xacro:macro>

File: src/models/scte_vehicle/scte_description/urdf/scte_chassis.xacro (robot description, xacro)
@@ -9,5 +9,6 @@
 http://wiki.ros.org/urdf/XML/joint#Elements
 -->
-<robot name="scteBot" xmlns:xacro="http://www.ros.org/wiki/xacro">
+<!--Gazebo does not seem to like capital letters in the robot namespace-->
+<robot name="sctebot" xmlns:xacro="http://www.ros.org/wiki/xacro">
     <xacro:property name="M_PI" value="3.14159265358979323846264338327950288"/>
     <xacro:include filename="$(find scte_description)/urdf/scte.gazebo" />
@@ -91,5 +92,5 @@
     <xacro:property name="shock_tower_height" value="0.105"/>
     <xacro:property name="shock_tower_width" value="0.14"/>
-    <xacro:scte_axle_components suffix="scte_front"
+    <xacro:scte_axle_components suffix="front"
         parent_link="scte_chassis"
         diff_joint_xyz="${scte_chassis_length * 0.63} 0 0"
@@ -112,5 +113,5 @@
         right_wheel_joint_rpy="0 0 0"
     />
-    <xacro:scte_axle_components suffix="scte_rear"
+    <xacro:scte_axle_components suffix="rear"
         parent_link="scte_chassis"
         diff_joint_xyz="${scte_chassis_length * -0.63} 0 0"
@@ -163,7 +164,7 @@
         </collision>
     </link>
-    <joint name="shock_tower_scte_front_LINKED_driver_side_mounting_bar" type="fixed">
+    <joint name="shock_tower_front_LINKED_driver_side_mounting_bar" type="fixed">
         <origin xyz="${scte_chassis_length * -0.63} ${shock_tower_width * 0.5} ${shock_tower_height * 0.5}" rpy="0 -0 0"/>
-        <parent link="shock_tower_scte_front"/>
+        <parent link="shock_tower_front"/>
         <child link="driver_side_mounting_bar"/>
     </joint>
@@ -192,7 +193,7 @@
         </collision>
     </link>
-    <joint name="shock_tower_scte_front_LINKED_passenger_side_mounting_bar" type="fixed">
+    <joint name="shock_tower_front_LINKED_passenger_side_mounting_bar" type="fixed">
         <origin xyz="${scte_chassis_length * -0.63} ${shock_tower_width * -0.5} ${shock_tower_height * 0.5}" rpy="0 -0 0"/>
-        <parent link="shock_tower_scte_front"/>
+        <parent link="shock_tower_front"/>
         <child link="passenger_side_mounting_bar"/>
     </joint>

File: src/models/scte_vehicle/scte_description/urdf/scte_chassis_DEBUG.xacro (robot description, xacro)
@@ -1,8 +1,9 @@
 <?xml version='1.0'?>
-<robot name="scteBot" xmlns:xacro="http://www.ros.org/wiki/xacro">
-    <link name="base_link">
-    </link>
+<robot name="sctebot" xmlns:xacro="http://www.ros.org/wiki/xacro">
+    <xacro:include filename="$(find scte_description)/urdf/scte.gazebo" />
+    <!--naming this link world will fix the model in space-->
+    <link name="base_link"/>
     <joint name="base_link" type="fixed">
-        <origin xyz="0 0 1.5" rpy="0 0 0"/>
+        <origin xyz="0 0 1" rpy="0 0 0"/>
         <parent link="base_link"/>
         <child link="scte_chassis"/>
@@ -22,5 +23,4 @@
                 <box size=".4 .2 .1"/>
             </geometry>
-            <material name="blue"/>
         </visual>
         <collision name='collision'>
@@ -58,5 +58,4 @@
         <child link="caster"/>
     </joint>
-    <!---->
     <link name="right_wheel">
         <inertial>
@@ -79,10 +78,10 @@
         </collision>
     </link>
-    <joint name="right_wheel_JOIN_scte_chassis" type="revolute">
-        <origin xyz="0.1 -0.15 0" rpy="0 1.5707 1.5707"/>
-        <limit effort="-1" velocity="-1" lower="-2147483647" upper="2147483647"/>
-        <axis xyz="0 0 1"/>
+    <joint name="right_wheel_JOIN_scte_chassis" type="continuous">
         <child link="right_wheel"/>
         <parent link="scte_chassis"/>
+        <origin xyz="0.1 -0.15 0" rpy="0 1.5707 1.5707"/>
+        <dynamics damping="0.7"/>
+        <axis xyz="0 0 1"/>
     </joint>
     <link name="left_wheel">
@@ -106,11 +105,30 @@
         </collision>
     </link>
-    <joint name="left_wheel_JOIN_scte_chassis" type="revolute">
-        <origin xyz="0.1 0.15 0" rpy="0 1.5707 1.5707"/>
-        <limit effort="-1" velocity="-1" lower="-2147483647" upper="2147483647"/>
-        <axis xyz="0 0 1"/>
+    <joint name="left_wheel_JOIN_scte_chassis" type="continuous">
         <child link="left_wheel"/>
         <parent link="scte_chassis"/>
+        <origin xyz="0.1 0.15 0" rpy="0 1.5707 1.5707"/>
+        <dynamics damping="0.7"/>
+        <axis xyz="0 0 1"/>
     </joint>
-    <!---->
+    <transmission name="tran1">
+        <type>transmission_interface/SimpleTransmission</type>
+        <joint name="left_wheel_JOIN_scte_chassis">
+            <hardwareInterface>hardware_interface/EffortJointInterface</hardwareInterface>
+        </joint>
+        <actuator name="motor1">
+            <hardwareInterface>hardware_interface/EffortJointInterface</hardwareInterface>
+            <mechanicalReduction>1</mechanicalReduction>
+        </actuator>
+    </transmission>
+    <transmission name="tran2">
+        <type>transmission_interface/SimpleTransmission</type>
+        <joint name="right_wheel_JOIN_scte_chassis">
+            <hardwareInterface>hardware_interface/EffortJointInterface</hardwareInterface>
+        </joint>
+        <actuator name="motor2">
+            <hardwareInterface>hardware_interface/EffortJointInterface</hardwareInterface>
+            <mechanicalReduction>1</mechanicalReduction>
+        </actuator>
+    </transmission>
 </robot>
