Commit message: more tweaks, may have properly setup a way to control the wheel spin through a topic

File: src/models/scte_vehicle/scte_description/urdf/scte_axle_components.xacro (robot description, xacro)
@@ -42,5 +42,5 @@
             </collision>
         </link>
-        <joint name="diff_${suffix}_JOINT_${parent_link}" type="fixed">
+        <joint name="diff_${suffix}_JOINED_${parent_link}" type="fixed">
             <axis xyz="0 0 0"/>
             <origin xyz="${diff_joint_xyz}" rpy="${diff_joint_rpy}"/>
@@ -71,5 +71,5 @@
             </collision>
         </link>
-        <joint name="diff_bumper_${suffix}_JOINT_${parent_link}" type="fixed">
+        <joint name="diff_bumper_${suffix}_JOINED_${parent_link}" type="fixed">
             <axis xyz="0 0 0"/>
             <origin xyz="${0.07} 0 ${0.07 * 0.30}" rpy="0 ${M_PI/-6}  0"/>
@@ -98,5 +98,5 @@
             </collision>
         </link>
-        <joint name="bumper_${suffix}_JOINT_${parent_link}" type="fixed">
+        <joint name="bumper_${suffix}_JOINED_${parent_link}" type="fixed">
             <axis xyz="0 0 0"/>
             <origin xyz="${0.07 * 0.70} 0 ${0.07 * 0.35}" rpy="0 ${M_PI/6} 0"/>
@@ -128,5 +128,5 @@
             </collision>
         </link>
-        <joint name="diff_bumper_${suffix}_JOINT_${parent_link}" type="fixed">
+        <joint name="diff_bumper_${suffix}_JOINED_${parent_link}" type="fixed">
             <axis xyz="0 0 0"/>
             <origin xyz="${0.09 * -0.5} 0 0" rpy="0 0 0"/>
@@ -155,5 +155,5 @@
             </collision>
         </link>
-        <joint name="bumper_${suffix}_JOINT_${parent_link}" type="fixed">
+        <joint name="bumper_${suffix}_JOINED_${parent_link}" type="fixed">
             <axis xyz="0 0 0"/>
             <origin xyz="${0.09 * -0.5} 0 0.015" rpy="0 0 0"/>
@@ -185,5 +185,5 @@
             </collision>
         </link>
-        <joint name='shock_tower_${suffix}_JOINT_diff_${suffix}' type='fixed'>
+        <joint name='shock_tower_${suffix}_JOINED_diff_${suffix}' type='fixed'>
             <origin xyz="${shock_tower_joint_origin}" rpy="${shock_tower_joint_rpy}"/>
             <parent link="diff_base_plate_${suffix}"/>
@@ -215,5 +215,5 @@
             </collision>
         </link>
-        <joint name='diff_${suffix}_JOINT_axle_${suffix}' type='fixed'>
+        <joint name='diff_${suffix}_JOINED_axle_${suffix}' type='fixed'>
             <origin xyz="${drive_axle_joint_origin}" rpy="${drive_axle_joint_rpy}"/>
             <parent link="diff_base_plate_${suffix}"/>
@@ -245,5 +245,5 @@
             </collision>
         </link>
-        <joint name='left_wheel_${suffix}_JOINT_axle_${suffix}' type='continuous'>
+        <joint name='left_wheel_${suffix}_JOINED_axle_${suffix}' type='continuous'>
             <origin xyz="${left_wheel_joint_origin}" rpy="${left_wheel_joint_rpy}"/>
             <parent link="axle_${suffix}"/>
@@ -255,5 +255,5 @@
         <transmission name="tran_left_wheel_${suffix}">
             <type>transmission_interface/SimpleTransmission</type>
-            <joint name="left_wheel_${suffix}_JOINT_axle_${suffix}">
+            <joint name="left_wheel_${suffix}_JOINED_axle_${suffix}">
                 <hardwareInterface>hardware_interface/EffortJointInterface</hardwareInterface>
             </joint>
@@ -285,5 +285,5 @@
             </collision>
         </link>
-        <joint name='right_wheel_${suffix}_JOINT_axle_${suffix}' type='continuous'>
+        <joint name='right_wheel_${suffix}_JOINED_axle_${suffix}' type='continuous'>
             <origin xyz="${right_wheel_joint_origin}" rpy="${right_wheel_joint_rpy}"/>
             <parent link="axle_${suffix}"/>
@@ -295,5 +295,5 @@
         <transmission name="tran_right_wheel_${suffix}">
             <type>transmission_interface/SimpleTransmission</type>
-            <joint name="right_wheel_${suffix}_JOINT_axle_${suffix}">
+            <joint name="right_wheel_${suffix}_JOINED_axle_${suffix}">
                 <hardwareInterface>hardware_interface/EffortJointInterface</hardwareInterface>
             </joint>

File: src/models/scte_vehicle/scte_description/urdf/scte_chassis.xacro (robot description, xacro)
@@ -164,5 +164,5 @@
         </collision>
     </link>
-    <joint name="shock_tower_front_LINKED_driver_side_mounting_bar" type="fixed">
+    <joint name="shock_tower_front_JOINED_driver_side_mounting_bar" type="fixed">
         <origin xyz="${scte_chassis_length * -0.63} ${shock_tower_width * 0.5} ${shock_tower_height * 0.5}" rpy="0 -0 0"/>
         <parent link="shock_tower_front"/>
@@ -193,5 +193,5 @@
         </collision>
     </link>
-    <joint name="shock_tower_front_LINKED_passenger_side_mounting_bar" type="fixed">
+    <joint name="shock_tower_front_JOINED_passenger_side_mounting_bar" type="fixed">
         <origin xyz="${scte_chassis_length * -0.63} ${shock_tower_width * -0.5} ${shock_tower_height * 0.5}" rpy="0 -0 0"/>
         <parent link="shock_tower_front"/>
@@ -227,5 +227,5 @@
         </collision>
     </link>
-    <joint name="main_computer_enclosure_LINKED_driver_side_mounting_bar" type="fixed">
+    <joint name="main_computer_enclosure_JOINED_driver_side_mounting_bar" type="fixed">
         <origin xyz="0 ${(scte_chassis_width * -0.5) + (mounting_bars_width * 0.5)} ${0.06 * 0.5}" rpy="0 0 0"/>
         <parent link="driver_side_mounting_bar"/>
@@ -259,5 +259,5 @@
         </collision>
     </link>
-    <joint name="stereo_camera_bar_support_LINKED_main_computer_enclosure" type="fixed">
+    <joint name="stereo_camera_bar_support_JOINED_main_computer_enclosure" type="fixed">
         <origin xyz="${0.260 * -0.45} 0 ${0.06 * 1.0}" rpy="0 0 0"/>
         <parent link="main_computer_enclosure"/>
@@ -288,5 +288,5 @@
         </collision>
     </link>
-    <joint name="stereo_camera_bar_LINKED_stereo_camera_bar_support" type="fixed">
+    <joint name="stereo_camera_bar_JOINED_stereo_camera_bar_support" type="fixed">
         <origin xyz="0 0 ${0.06 * 0.5}" rpy="0 0 0"/>
         <parent link="stereo_camera_bar_support"/>
@@ -326,5 +326,5 @@
         </collision>
     </link>
-    <joint name="debug_stereo_perception_camera_LINKED_stereo_camera_bar" type="fixed">
+    <joint name="debug_stereo_perception_camera_JOINED_stereo_camera_bar" type="fixed">
         <origin xyz="0 0.5 0" rpy="${M_PI/-2} 0 ${M_PI/-2}"/>
         <parent link="stereo_camera_bar"/>
@@ -334,5 +334,5 @@
     <!--LIDAR-->
     <xacro:include filename="$(find ydlidar_ros)/urdf/ydlidar.urdf"/>
-    <joint name="main_computer_enclosure_LINKED_ydlidar_base" type="fixed">
+    <joint name="main_computer_enclosure_JOINED_ydlidar_base" type="fixed">
         <origin xyz="0.090 0 0.0305" rpy="0 0 0"/>
         <parent link="main_computer_enclosure"/>

Commit message: got the gazebo model to respond to joystick input. Need to rework the model to be like husky demo

File: src/models/scte_vehicle/scte_description/urdf/scte_axle_components.xacro (robot description, xacro)
@@ -253,5 +253,5 @@
             <dynamics damping="0.7"/>
         </joint>
-        <transmission name="tran_left_wheel_${suffix}">
+        <!--transmission name="tran_left_wheel_${suffix}">
             <type>transmission_interface/SimpleTransmission</type>
             <joint name="left_wheel_${suffix}_JOINED_axle_${suffix}">
@@ -262,4 +262,13 @@
                 <mechanicalReduction>1</mechanicalReduction>
             </actuator>
+        </transmission-->
+        <transmission name="tran_left_wheel_${suffix}" type="SimpleTransmission">
+            <type>transmission_interface/SimpleTransmission</type>
+            <actuator name="motor_left_wheel_${suffix}">
+                <mechanicalReduction>1</mechanicalReduction>
+            </actuator>
+            <joint name="left_wheel_${suffix}_JOINED_axle_${suffix}">
+                <hardwareInterface>hardware_interface/VelocityJointInterface</hardwareInterface>
+            </joint>
         </transmission>
         <!---->
@@ -293,5 +302,5 @@
             <dynamics damping="0.7"/>
         </joint>
-        <transmission name="tran_right_wheel_${suffix}">
+        <!--transmission name="tran_right_wheel_${suffix}">
             <type>transmission_interface/SimpleTransmission</type>
             <joint name="right_wheel_${suffix}_JOINED_axle_${suffix}">
@@ -302,4 +311,13 @@
                 <mechanicalReduction>1</mechanicalReduction>
             </actuator>
+        </transmission-->
+        <transmission name="tran_right_wheel_${suffix}" type="SimpleTransmission">
+            <type>transmission_interface/SimpleTransmission</type>
+            <actuator name="motor_right_wheel_${suffix}">
+                <mechanicalReduction>1</mechanicalReduction>
+            </actuator>
+            <joint name="right_wheel_${suffix}_JOINED_axle_${suffix}">
+                <hardwareInterface>hardware_interface/VelocityJointInterface</hardwareInterface>
+            </joint>
         </transmission>
         <!---->

File: src/models/scte_vehicle/scte_description/urdf/scte_chassis.xacro (robot description, xacro)
@@ -11,6 +11,7 @@
 <!--Gazebo does not seem to like capital letters in the robot namespace-->
 <robot name="sctebot" xmlns:xacro="http://www.ros.org/wiki/xacro">
+    <xacro:arg name="robot_namespace" default="/" />
     <xacro:property name="M_PI" value="3.14159265358979323846264338327950288"/>
-    <xacro:include filename="$(find scte_description)/urdf/scte.gazebo" />
+    <!--xacro:include filename="$(find scte_description)/urdf/scte.gazebo" /-->
     <xacro:include filename="$(find scte_description)/urdf/materials.xacro" />
     <xacro:include filename="$(find scte_description)/urdf/macros.xacro" />
@@ -59,16 +60,17 @@
     <!--DEBUG test link for odom testing-->
     <!--CHASSIS-->
-    <xacro:property name="scte_total_mass" value="3.8"/>
+    <xacro:property name="scte_total_mass" value="50"/>
     <xacro:property name="scte_chassis_length" value="0.292"/>
     <xacro:property name="scte_chassis_width" value="0.165"/>
     <xacro:property name="scte_chassis_depth" value="0.00635"/>
     <link name='scte_chassis'>
+        <!-- borrowed from husky for debug-->
         <inertial>
             <mass value="${scte_total_mass * 0.86}"/>
-            <origin xyz="0 0 0" rpy="0 0 0"/>
-            <inertia
-                    ixx="1" ixy="0" ixz="0"
-                    iyy="1" iyz="0"
-                    izz="1"
+            <origin xyz="-0.00065 -0.085 0.062" rpy="0 0 0"/>
+            <inertia
+                    ixx="0.6022" ixy="-0.02364" ixz="-0.1197"
+                    iyy="1.7386" iyz="-0.001544"
+                    izz="2.0296"
             />
         </inertial>
@@ -339,3 +341,9 @@
         <child link="base_laser"/>
     </joint>
+    <gazebo>
+        <plugin name="gazebo_ros_control" filename="libgazebo_ros_control.so">
+            <!--robotNamespace>$(arg robot_namespace)</robotNamespace-->
+            <legacyModeNS>true</legacyModeNS>
+        </plugin>
+    </gazebo>
 </robot>

File: src/models/scte_vehicle/scte_description/urdf/scte_chassis_DEBUG.xacro (robot description, xacro)
@@ -1,5 +1,5 @@
 <?xml version='1.0'?>
 <robot name="sctebot" xmlns:xacro="http://www.ros.org/wiki/xacro">
-    <xacro:include filename="$(find scte_description)/urdf/scte.gazebo" />
+    <!--xacro:include filename="$(find scte_description)/urdf/scte.gazebo" /-->
     <!--naming this link world will fix the model in space-->
     <link name="base_link"/>
@@ -112,8 +112,8 @@
         <axis xyz="0 0 1"/>
     </joint>
-    <transmission name="tran1">
+    <!--transmission name="tran1">
         <type>transmission_interface/SimpleTransmission</type>
         <joint name="left_wheel_JOIN_scte_chassis">
-            <hardwareInterface>hardware_interface/EffortJointInterface</hardwareInterface>
+            <hardwareInterface>hardware_interface/VelocityJointInterface</hardwareInterface>
         </joint>
         <actuator name="motor1">
@@ -121,6 +121,15 @@
             <mechanicalReduction>1</mechanicalReduction>
         </actuator>
+    </transmission-->
+    <transmission name="tran_left" type="SimpleTransmission">
+        <type>transmission_interface/SimpleTransmission</type>
+        <actuator name="motor_left_wheel">
+            <mechanicalReduction>1</mechanicalReduction>
+        </actuator>
+        <joint name="left_wheel_JOIN_scte_chassis">
+            <hardwareInterface>hardware_interface/VelocityJointInterface</hardwareInterface>
+        </joint>
     </transmission>
-    <transmission name="tran2">
+    <!--transmission name="tran2">
         <type>transmission_interface/SimpleTransmission</type>
         <joint name="right_wheel_JOIN_scte_chassis">
@@ -131,4 +140,19 @@
             <mechanicalReduction>1</mechanicalReduction>
         </actuator>
+    </transmission-->
+    <transmission name="tran_right" type="SimpleTransmission">
+        <type>transmission_interface/SimpleTransmission</type>
+        <actuator name="motor_right_wheel">
+            <mechanicalReduction>1</mechanicalReduction>
+        </actuator>
+        <joint name="right_wheel_JOIN_scte_chassis">
+            <hardwareInterface>hardware_interface/VelocityJointInterface</hardwareInterface>
+        </joint>
     </transmission>
+    <gazebo>
+        <plugin name="gazebo_ros_control" filename="libgazebo_ros_control.so">
+            <!--robotNamespace>$(arg robot_namespace)</robotNamespace-->
+            <legacyModeNS>true</legacyModeNS>
+        </plugin>
+    </gazebo>
 </robot>

Commit message: got teleop working. needs to be tuned for odom.

File: src/models/scte_vehicle/scte_description/urdf/scte_axle_components.xacro (robot description, xacro)
@@ -163,5 +163,4 @@
         </xacro:if>
         <!--shock tower-->
-        <!---->
         <link name="shock_tower_${suffix}">
             <inertial>
@@ -191,7 +190,5 @@
             <axis xyz="0 0 0" rpy="0 0 0"/>
         </joint>
-        <!---->
         <!--axle-->
-        <!---->
         <link name="axle_${suffix}">
             <inertial>
@@ -221,15 +218,9 @@
             <axis xyz="0 0 0" rpy="0 0 0"/>
         </joint>
-        <!---->
         <!--wheels-->
-        <!---->
         <link name="left_wheel_${suffix}">
             <inertial>
                 <mass value="${scte_total_mass * 0.25 * 0.05}"/>
-                <inertia
-                        ixx="1" ixy="0" ixz="0"
-                        iyy="1" iyz="0"
-                        izz="1"
-                />
+                <inertia  ixx="0.02467" ixy="0" ixz="0" iyy="0.04411" iyz="0" izz="0.02467" />
             </inertial>
             <visual name='visual'>
@@ -245,4 +236,11 @@
             </collision>
         </link>
+        <gazebo reference="left_wheel_${suffix}">
+            <mu1 value="1.0"/>
+            <mu2 value="1.0"/>
+            <kp value="10000000.0" />
+            <kd value="1.0" />
+            <fdir1 value="1 0 0"/>
+        </gazebo>
         <joint name='left_wheel_${suffix}_JOINED_axle_${suffix}' type='continuous'>
             <origin xyz="${left_wheel_joint_origin}" rpy="${left_wheel_joint_rpy}"/>
@@ -253,14 +251,4 @@
             <dynamics damping="0.7"/>
         </joint>
-        <!--transmission name="tran_left_wheel_${suffix}">
-            <type>transmission_interface/SimpleTransmission</type>
-            <joint name="left_wheel_${suffix}_JOINED_axle_${suffix}">
-                <hardwareInterface>hardware_interface/EffortJointInterface</hardwareInterface>
-            </joint>
-            <actuator name="motor_left_wheel_${suffix}">
-                <hardwareInterface>hardware_interface/EffortJointInterface</hardwareInterface>
-                <mechanicalReduction>1</mechanicalReduction>
-            </actuator>
-        </transmission-->
         <transmission name="tran_left_wheel_${suffix}" type="SimpleTransmission">
             <type>transmission_interface/SimpleTransmission</type>
@@ -272,13 +260,8 @@
             </joint>
         </transmission>
-        <!---->
         <link name="right_wheel_${suffix}">
             <inertial>
                 <mass value="${scte_total_mass * 0.25 * 0.05}"/>
-                <inertia
-                        ixx="1" ixy="0" ixz="0"
-                        iyy="1" iyz="0"
-                        izz="1"
-                />
+                <inertia  ixx="0.02467" ixy="0" ixz="0" iyy="0.04411" iyz="0" izz="0.02467" />
             </inertial>
             <visual name='visual'>
@@ -294,4 +277,11 @@
             </collision>
         </link>
+        <gazebo reference="right_wheel_${suffix}">
+            <mu1 value="1.0"/>
+            <mu2 value="1.0"/>
+            <kp value="10000000.0" />
+            <kd value="1.0" />
+            <fdir1 value="1 0 0"/>
+        </gazebo>
         <joint name='right_wheel_${suffix}_JOINED_axle_${suffix}' type='continuous'>
             <origin xyz="${right_wheel_joint_origin}" rpy="${right_wheel_joint_rpy}"/>
@@ -302,14 +292,4 @@
             <dynamics damping="0.7"/>
         </joint>
-        <!--transmission name="tran_right_wheel_${suffix}">
-            <type>transmission_interface/SimpleTransmission</type>
-            <joint name="right_wheel_${suffix}_JOINED_axle_${suffix}">
-                <hardwareInterface>hardware_interface/EffortJointInterface</hardwareInterface>
-            </joint>
-            <actuator name="motor_right_wheel_${suffix}">
-                <hardwareInterface>hardware_interface/EffortJointInterface</hardwareInterface>
-                <mechanicalReduction>1</mechanicalReduction>
-            </actuator>
-        </transmission-->
         <transmission name="tran_right_wheel_${suffix}" type="SimpleTransmission">
             <type>transmission_interface/SimpleTransmission</type>
@@ -321,5 +301,4 @@
             </joint>
         </transmission>
-        <!---->
     </xacro:macro>
 </robot>

File: src/models/scte_vehicle/scte_description/urdf/scte_chassis.xacro (robot description, xacro)
@@ -16,63 +16,11 @@
     <xacro:include filename="$(find scte_description)/urdf/materials.xacro" />
     <xacro:include filename="$(find scte_description)/urdf/macros.xacro" />
-    <link name="base_link">
-    </link>
-    <joint name="base_link" type="fixed">
-        <origin xyz="0 0.0 0.0" rpy="0 -0 0"/>
-        <parent link="base_link"/>
-        <child link="scte_chassis"/>
-    </joint>
-    <!--DEBUG test link for odom testing-->
-    <!--
-    <link name="test_real_link">
-        <inertial>
-            <mass value="1.0"/>
-            <origin xyz="0 0 0" rpy="0 0 0"/>
-            <inertia
-                    ixx="1" ixy="0" ixz="0"
-                    iyy="1" iyz="0"
-                    izz="1"
-            />
-        </inertial>
-        <visual name='visual'>
-            <transparency>1</transparency>
-            <origin xyz="0 0 0" rpy="0 0 0"/>
-            <geometry>
-                <box size="0.075 0.075 0.075"/>
-            </geometry>
-            <material name="none1">
-                <color rgba="${255/255} ${0/255} ${0/255} 1.0"/>
-            </material>
-        </visual>
-        <collision name='collision'>
-            <origin xyz="0 0 0" rpy="0 0 0"/>
-            <geometry>
-                <box size="0.075 0.075 0.075"/>
-            </geometry>
-        </collision>
-    </link>
-    <joint name="odom_test" type="fixed">
-        <origin xyz="0 0.0 1.0" rpy="0 0 0"/>
-        <parent link="scte_chassis"/>
-        <child link="test_real_link"/>
-    </joint>
-    -->
-    <!--DEBUG test link for odom testing-->
-    <!--CHASSIS-->
     <xacro:property name="scte_total_mass" value="50"/>
     <xacro:property name="scte_chassis_length" value="0.292"/>
     <xacro:property name="scte_chassis_width" value="0.165"/>
     <xacro:property name="scte_chassis_depth" value="0.00635"/>
-    <link name='scte_chassis'>
-        <!-- borrowed from husky for debug-->
-        <inertial>
-            <mass value="${scte_total_mass * 0.86}"/>
-            <origin xyz="-0.00065 -0.085 0.062" rpy="0 0 0"/>
-            <inertia
-                    ixx="0.6022" ixy="-0.02364" ixz="-0.1197"
-                    iyy="1.7386" iyz="-0.001544"
-                    izz="2.0296"
-            />
-        </inertial>
+    <!--Wheel Properties-->
+    <xacro:property name="wheel_radius" value="0.05"/>
+    <link name='base_link'>
         <visual name='visual'>
             <origin xyz="0 0 0" rpy="0 0 0"/>
@@ -89,4 +37,30 @@
         </collision>
     </link>
+    <link name='base_footprint'/>
+    <joint name="base_footprint_joint" type="fixed">
+        <origin xyz="0 0 ${scte_chassis_depth - wheel_radius}" rpy="0 0 0"/>
+        <parent link="base_link"/>
+        <child link="base_footprint"/>
+    </joint>
+    <!-- Inertial link stores the robot's inertial information -->
+    <link name="inertial_link">
+        <inertial>
+            <mass value="${scte_total_mass * 0.90}" />
+            <origin xyz="0 0 0" />
+            <inertia ixx="0.6022" ixy="-0.02364" ixz="-0.1197" iyy="1.7386" iyz="-0.001544" izz="2.0296" />
+        </inertial>
+    </link>
+    <joint name="inertial_to_base_link_joint" type="fixed">
+        <origin xyz="0 0 0" rpy="0 0 0" />
+        <parent link="base_link" />
+        <child link="inertial_link" />
+    </joint>
+    <!--CHASSIS-->
+    <link name="scte_chassis"/>
+    <joint name="scte_chassis_to_base_link_joint" type="fixed">
+        <origin xyz="0 0 0" rpy="0 0 0"/>
+        <parent link="base_link"/>
+        <child link="scte_chassis"/>
+    </joint>
     <xacro:include filename="$(find scte_description)/urdf/scte_axle_components.xacro"/>
     <xacro:property name="drive_axle_length" value="0.25"/>
@@ -106,5 +80,5 @@
         shock_tower_joint_origin="0 0 ${shock_tower_height * 0.5}"
         shock_tower_joint_rpy="0 0 0"
-        left_wheel_radius="0.05"
+        left_wheel_radius="${wheel_radius}"
         left_wheel_length="0.045"
         left_wheel_joint_origin="0 0 ${drive_axle_length * 0.5}"
@@ -341,9 +315,9 @@
         <child link="base_laser"/>
     </joint>
-    <gazebo>
-        <plugin name="gazebo_ros_control" filename="libgazebo_ros_control.so">
+    <!--gazebo>
+        <plugin name="gazebo_ros_control" filename="libgazebo_ros_control.so"-->
             <!--robotNamespace>$(arg robot_namespace)</robotNamespace-->
-            <legacyModeNS>true</legacyModeNS>
+            <!--legacyModeNS>true</legacyModeNS>
         </plugin>
-    </gazebo>
+    </gazebo-->
 </robot>
