Commit message: using steer_bot example from srmainwaring to get working steer_bot_gazebo plugin and ackermann in ros

File: src/models/scte_vehicle/scte_description/urdf/materials.xacro (robot description, xacro)
@@ -1,27 +1,35 @@
-<?xml version="1.0"?>
-<robot>
-    <material name="black">
-        <color rgba="0.0 0.0 0.0 1.0"/>
+<?xml version="1.0" ?>
+<!--  xacro macros for robot materials.
+ -->
+<robot name="materials" xmlns:xacro="http://wiki.ros.org/xacro">
+    <material name="red">
+        <color rgba="0.8 0 0 1"/>
+    </material>
+    <material name="green">
+        <color rgba="0 0.8 0 1"/>
     </material>
     <material name="blue">
-        <color rgba="0.0 0.0 0.8 1.0"/>
+        <color rgba="0 0 0.8 1"/>
     </material>
-    <material name="green">
-        <color rgba="0.0 0.8 0.0 1.0"/>
-    </material>
-    <material name="grey">
-        <color rgba="0.2 0.2 0.2 1.0"/>
+    <material name="yellow">
+        <color rgba="0.8 0.8 0 1"/>
     </material>
     <material name="orange">
-        <color rgba="${255/255} ${108/255} ${10/255} 1.0"/>
+        <color rgba="0.8 0.25 0 1"/>
     </material>
-    <material name="brown">
-        <color rgba="${222/255} ${207/255} ${195/255} 1.0"/>
+    <material name="black">
+        <color rgba="0 0 0 1"/>
     </material>
-    <material name="red">
-        <color rgba="0.8 0.0 0.0 1.0"/>
+    <material name="dark_gray">
+        <color rgba="0.5 0.5 0.5 1"/>
+    </material>
+    <material name="gray">
+        <color rgba="0.753 0.753 0.753 1"/>
+    </material>
+    <material name="silver">
+        <color rgba="0.88 0.88 0.88 1"/>
     </material>
     <material name="white">
-        <color rgba="1.0 1.0 1.0 1.0"/>
+        <color rgba="1 1 1 1"/>
     </material>
 </robot>

File: src/models/scte_vehicle/scte_description/urdf/scte_chassis.xacro (robot description, xacro)
@@ -11,9 +11,9 @@
 <!--Gazebo does not seem to like capital letters in the robot namespace-->
 <robot name="sctebot" xmlns:xacro="http://www.ros.org/wiki/xacro">
-    <xacro:arg name="robot_namespace" default="/DEFAULTNAMESPACE2"/>
+    <xacro:arg name="robot_namespace" default="/"/>
     <xacro:arg name="tf_freq" default="100.0"/>
     <xacro:arg name="pub_tf" default="true"/>
     <xacro:property name="M_PI" value="3.14159265358979323846264338327950288"/>
-    <xacro:include filename="plugins/scte_plugins.gazebo" />
+    <xacro:include filename="$(find scte_description)/urdf/plugins/scte_plugins.gazebo" />
     <!--xacro:include filename="$(find scte_description)/urdf/plugins/scte_audi_bot_plugin.gazebo"/-->
     <!--xacro:include filename="plugins/scte_sensors.gazebo" /-->
@@ -261,3 +261,4 @@
     <xacro:logitech_c270_camera parent_link="camera_rig_bar" camera_link="passenger_side_camera" joint_xyz="0.0 -0.05 ${0.025 * 0.5}" joint_rpy="0 0 0"/>
     <!---->
+    <gazebo reference="base_link"/>
 </robot>
