Commit message: improving urdf xacro files

File: src/models/scte_vehicle/scte_description/urdf/scte_chassis.xacro (robot description, xacro)
@@ -4,4 +4,5 @@
 http://gazebosim.org/tutorials?tut=ros_urdf
 https://wiki.ros.org/action/fullsearch/urdf/Tutorials/Building%20a%20Visual%20Robot%20Model%20with%20URDF%20from%20Scratch?action=fullsearch&context=180&value=linkto%3A%22urdf%2FTutorials%2FBuilding+a+Visual+Robot+Model+with+URDF+from+Scratch%22
+http://wiki.ros.org/xacro
 -->
 <robot name="scteBot" xmlns:xacro="http://www.ros.org/wiki/xacro">
@@ -16,5 +17,4 @@
     <xacro:property name="scte_wheel_depth" value="0.0508"/>
     <xacro:include filename="$(find scte_description)/urdf/scte.gazebo" />
-    <xacro:include filename="$(find scte_description)/urdf/scte_diff.xacro"/>
     <xacro:include filename="$(find scte_description)/urdf/materials.xacro" />
     <xacro:include filename="$(find scte_description)/urdf/macros.xacro" />
@@ -24,4 +24,9 @@
         <origin xyz="0 0 0" rpy="0 0 0" />
     </SOMESENSOR-->
+    <!--sensors>
+    <xacro:include filename="$(find logitech_c270_camera)/urdf/logitech_c270.xacro"/>
+    <xacro:logitech_c270_camera parent_link="scte_front_axle" camera_link="left_cam" joint_xyz="0 0.15 ${scte_chassis_width * 0.65 * -1.0}" joint_rpy="0 0 0"/>
+    <xacro:logitech_c270_camera parent_link="scte_front_axle" camera_link="right_cam" joint_xyz="0 0.15 ${scte_chassis_width * 0.65}" joint_rpy="0 0 0"/>
+    -->
     <link name="base_link">
     </link>
@@ -55,4 +60,8 @@
         </collision>
     </link>
+    <xacro:include filename="$(find scte_description)/urdf/scte_diff_axle.xacro"/>
+    <xacro:scte_diff_axle suffix="scte_front" parent_link="scte_chassis" joint_xyz="${scte_chassis_length * 0.63} 0 0" joint_rpy="0 0 0"/>
+    <xacro:scte_diff_axle suffix="scte_rear" parent_link="scte_chassis" joint_xyz="${scte_chassis_length * -0.63} 0 0" joint_rpy="0 0 0"/>
+    <!--
     <joint name='scte_chassis_JOINT_scte_front_diff' type='fixed'>
         <origin xyz="${scte_chassis_length * 0.63} 0 0" rpy="0 0 0"/>
@@ -67,4 +76,13 @@
         <axis xyz="0 0 0" rpy="0 0 0"/>
     </joint>
+    -->
+    <!--sensors-->
+    <!--cameras-->
+    <!--joint name="scte_chassis_JOINT_left_camera" type="fixed">
+        <origin xyz="0 0 0" rpy="0 0 0"/>
+        <parent link="scte_chassis"/>
+        <child link="left_cam"/>
+        <axis xyz="0 0 0" rpy="0 0 0"/>
+    </joint-->
     <!--link name='main_computer'>
     <inertial>

File: src/models/scte_vehicle/scte_description/urdf/scte_diff_axle.xacro (robot description, xacro)
@@ -1,5 +1,66 @@
 <?xml version="1.0"?>
-<robot>
-    <!-- FRONT DIFF AND AXLE -->
+<robot name="scte_diff_axle" xmlns:xacro="http://www.ros.org/wiki/xacro">
+    <xacro:macro name="scte_diff_axle" params="suffix parent_link joint_xyz joint_rpy">
+        <!--diff-->
+        <link name="diff_${suffix}">
+            <!--xacro:insert_block name="inertial"/>
+            <xacro:insert_block name="visual"/>
+            <xacro:insert_block name="collision"/-->
+            <intertial>
+                <mass value="${scte_total_mass * 0.05}"/>
+                <inertia
+                        ixx="1" ixy="0" ixz="0"
+                        iyy="1" iyz="0"
+                        izz="1"
+                />
+            </intertial>
+            <visual>
+                <geometry>
+                    <box size="${scte_chassis_length * 0.26} ${scte_chassis_width * 0.38} ${scte_chassis_depth}"/>
+                </geometry>
+                <material name="green"/>
+            </visual>
+            <collision>
+                <geometry>
+                    <box size="${scte_chassis_length * 0.26} ${scte_chassis_width * 0.38} ${scte_chassis_depth}"/>
+                </geometry>
+            </collision>
+        </link>
+        <joint name="diff_${suffix}_JOINT_${parent_link}" type="fixed">
+            <axis xyz="0 0 1"/>
+            <origin xyz="${joint_xyz}" rpy="${joint_rpy}"/>
+            <parent link="${parent_link}"/>
+            <child link="diff_${suffix}"/>
+        </joint>
+        <!--axle-->
+        <link name="axle_${suffix}">
+            <inertial>
+                <mass value="${scte_total_mass * 0.02}"/>
+                <inertia
+                        ixx="1" ixy="0" ixz="0"
+                        iyy="1" iyz="0"
+                        izz="1"
+                />
+            </inertial>
+            <visual name='visual'>
+                <geometry>
+                    <cylinder radius="${scte_chassis_depth * 0.35}" length="${scte_chassis_width * 1.46}"/>
+                </geometry>
+                <material name="red"/>
+            </visual>
+            <collision name='collision'>
+                <geometry>
+                    <cylinder radius="${scte_chassis_depth * 0.35}" length="${scte_chassis_width * 1.46}"/>
+                </geometry>
+            </collision>
+        </link>
+        <joint name='diff_${suffix}_JOINT_axle_${suffix}' type='fixed'>
+            <origin xyz="0 0 0" rpy="${M_PI/2} 0 0"/>
+            <parent link="diff_${suffix}"/>
+            <child link="axle_${suffix}"/>
+            <axis xyz="0 0 0" rpy="0 0 0"/>
+        </joint>
+    </xacro:macro>
+    <!-- FRONT DIFF AND AXLE>
     <link name="scte_front_diff">
         <inertial>
@@ -20,67 +81,4 @@
             <geometry>
                 <box size="${scte_chassis_length * 0.26} ${scte_chassis_width * 0.38} ${scte_chassis_depth}"/>
-            </geometry>
-        </collision>
-    </link>
-    <link name="scte_front_axle">
-        <inertial>
-            <mass value="${scte_total_mass * 0.02}"/>
-            <inertia
-                    ixx="1" ixy="0" ixz="0"
-                    iyy="1" iyz="0"
-                    izz="1"
-            />
-        </inertial>
-        <visual name='visual'>
-            <geometry>
-                <cylinder radius="${scte_chassis_depth * 0.35}" length="${scte_chassis_width * 1.46}"/>
-            </geometry>
-            <material name="red"/>
-        </visual>
-        <collision name='collision'>
-            <geometry>
-                <cylinder radius="${scte_chassis_depth * 0.35}" length="${scte_chassis_width * 1.46}"/>
-            </geometry>
-        </collision>
-    </link>
-    <link name="scte_front_left_wheel">
-        <inertial>
-            <mass value="${scte_wheel_mass / 4}"/>
-            <inertia
-                    ixx="1" ixy="0" ixz="0"
-                    iyy="1" iyz="0"
-                    izz="1"
-            />
-        </inertial>
-        <visual name='visual'>
-            <geometry>
-                <cylinder radius="${scte_wheel_radius}" length="${scte_wheel_depth}"/>
-            </geometry>
-            <material name="green"/>
-        </visual>
-        <collision name='collision'>
-            <geometry>
-                <cylinder radius="${scte_wheel_radius}" length="${scte_wheel_depth}"/>
-            </geometry>
-        </collision>
-    </link>
-    <link name="scte_front_right_wheel">
-        <inertial>
-            <mass value="${scte_wheel_mass / 4}"/>
-            <inertia
-                    ixx="1" ixy="0" ixz="0"
-                    iyy="1" iyz="0"
-                    izz="1"
-            />
-        </inertial>
-        <visual name='visual'>
-            <geometry>
-                <cylinder radius="${scte_wheel_radius}" length="${scte_wheel_depth}"/>
-            </geometry>
-            <material name="green"/>
-        </visual>
-        <collision name='collision'>
-            <geometry>
-                <cylinder radius="${scte_wheel_radius}" length="${scte_wheel_depth}"/>
             </geometry>
         </collision>
@@ -92,17 +90,83 @@
         <axis xyz="0 0 0" rpy="0 0 0"/>
     </joint>
-    <joint name='scte_front_axle_JOINT_scte_front_left_wheel' type='fixed'>
-        <origin xyz="0 0 ${scte_chassis_width * 0.65 * -1}" rpy="0 0 0"/>
-        <parent link="scte_front_axle"/>
-        <child link="scte_front_left_wheel"/>
-        <axis xyz="0 0 0" rpy="0 0 0"/>
-    </joint>
-    <joint name='scte_front_axle_JOINT_scte_front_right_wheel' type='fixed'>
-        <origin xyz="0 0 ${scte_chassis_width * 0.65}" rpy="0 0 0"/>
-        <parent link="scte_front_axle"/>
-        <child link="scte_front_right_wheel"/>
-        <axis xyz="0 0 0" rpy="0 0 0"/>
-    </joint>
-    <!-- REAR DIFF AND AXLE -->
+    <link name="scte_front_axle">
+        <inertial>
+            <mass value="${scte_total_mass * 0.02}"/>
+            <inertia
+                    ixx="1" ixy="0" ixz="0"
+                    iyy="1" iyz="0"
+                    izz="1"
+            />
+        </inertial>
+        <visual name='visual'>
+            <geometry>
+                <cylinder radius="${scte_chassis_depth * 0.35}" length="${scte_chassis_width * 1.46}"/>
+            </geometry>
+            <material name="red"/>
+        </visual>
+        <collision name='collision'>
+            <geometry>
+                <cylinder radius="${scte_chassis_depth * 0.35}" length="${scte_chassis_width * 1.46}"/>
+            </geometry>
+        </collision>
+    </link>
+-->
+    <!--
+        <link name="scte_front_left_wheel">
+            <inertial>
+                <mass value="${scte_wheel_mass / 4}"/>
+                <inertia
+                        ixx="1" ixy="0" ixz="0"
+                        iyy="1" iyz="0"
+                        izz="1"
+                />
+            </inertial>
+            <visual name='visual'>
+                <geometry>
+                    <cylinder radius="${scte_wheel_radius}" length="${scte_wheel_depth}"/>
+                </geometry>
+                <material name="green"/>
+            </visual>
+            <collision name='collision'>
+                <geometry>
+                    <cylinder radius="${scte_wheel_radius}" length="${scte_wheel_depth}"/>
+                </geometry>
+            </collision>
+        </link>
+        <link name="scte_front_right_wheel">
+            <inertial>
+                <mass value="${scte_wheel_mass / 4}"/>
+                <inertia
+                        ixx="1" ixy="0" ixz="0"
+                        iyy="1" iyz="0"
+                        izz="1"
+                />
+            </inertial>
+            <visual name='visual'>
+                <geometry>
+                    <cylinder radius="${scte_wheel_radius}" length="${scte_wheel_depth}"/>
+                </geometry>
+                <material name="green"/>
+            </visual>
+            <collision name='collision'>
+                <geometry>
+                    <cylinder radius="${scte_wheel_radius}" length="${scte_wheel_depth}"/>
+                </geometry>
+            </collision>
+        </link>
+        <joint name='scte_front_axle_JOINT_scte_front_left_wheel' type='fixed'>
+            <origin xyz="0 0 ${scte_chassis_width * 0.65 * -1}" rpy="0 0 0"/>
+            <parent link="scte_front_axle"/>
+            <child link="scte_front_left_wheel"/>
+            <axis xyz="0 0 0" rpy="0 0 0"/>
+        </joint>
+        <joint name='scte_front_axle_JOINT_scte_front_right_wheel' type='fixed'>
+            <origin xyz="0 0 ${scte_chassis_width * 0.65}" rpy="0 0 0"/>
+            <parent link="scte_front_axle"/>
+            <child link="scte_front_right_wheel"/>
+            <axis xyz="0 0 0" rpy="0 0 0"/>
+        </joint>
+    -->
+    <!-- REAR DIFF AND AXLE
     <link name="scte_rear_diff">
         <inertial>
@@ -207,3 +271,4 @@
         <axis xyz="0 0 0" rpy="0 0 0"/>
     </joint>
+    -->
 </robot>

Commit message: added back cameras

File: src/models/scte_vehicle/scte_description/urdf/scte_chassis.xacro (robot description, xacro)
@@ -24,9 +24,4 @@
         <origin xyz="0 0 0" rpy="0 0 0" />
     </SOMESENSOR-->
-    <!--sensors>
-    <xacro:include filename="$(find logitech_c270_camera)/urdf/logitech_c270.xacro"/>
-    <xacro:logitech_c270_camera parent_link="scte_front_axle" camera_link="left_cam" joint_xyz="0 0.15 ${scte_chassis_width * 0.65 * -1.0}" joint_rpy="0 0 0"/>
-    <xacro:logitech_c270_camera parent_link="scte_front_axle" camera_link="right_cam" joint_xyz="0 0.15 ${scte_chassis_width * 0.65}" joint_rpy="0 0 0"/>
-    -->
     <link name="base_link">
     </link>
@@ -63,18 +58,9 @@
     <xacro:scte_diff_axle suffix="scte_front" parent_link="scte_chassis" joint_xyz="${scte_chassis_length * 0.63} 0 0" joint_rpy="0 0 0"/>
     <xacro:scte_diff_axle suffix="scte_rear" parent_link="scte_chassis" joint_xyz="${scte_chassis_length * -0.63} 0 0" joint_rpy="0 0 0"/>
-    <!--
-    <joint name='scte_chassis_JOINT_scte_front_diff' type='fixed'>
-        <origin xyz="${scte_chassis_length * 0.63} 0 0" rpy="0 0 0"/>
-        <parent link="scte_chassis"/>
-        <child link="scte_front_diff"/>
-        <axis xyz="0 0 0" rpy="0 0 0"/>
-    </joint>
-    <joint name='scte_chassis_JOINT_scte_rear_diff' type='fixed'>
-        <origin xyz="${scte_chassis_length * 0.63 * -1} 0 0" rpy="0 0 0"/>
-        <parent link="scte_chassis"/>
-        <child link="scte_rear_diff"/>
-        <axis xyz="0 0 0" rpy="0 0 0"/>
-    </joint>
-    -->
+    <!--sensors-->
+    <xacro:include filename="$(find logitech_c270_camera)/urdf/logitech_c270.xacro"/>
+    <xacro:logitech_c270_camera parent_link="axle_scte_front" camera_link="left_cam" joint_xyz="0 0.15 ${scte_chassis_width * 0.65 * -1.0}" joint_rpy="0 0 0"/>
+    <xacro:logitech_c270_camera parent_link="axle_scte_front" camera_link="right_cam" joint_xyz="0 0.15 ${scte_chassis_width * 0.65}" joint_rpy="0 0 0"/>
+    <!---->
     <!--sensors-->
     <!--cameras-->

Commit message: modified c270 camera launch file and created a stereo launch file. added a doc with links to setup ros in netbeans

File: src/models/scte_vehicle/scte_description/urdf/scte_chassis.xacro (robot description, xacro)
@@ -62,13 +62,4 @@
     <xacro:logitech_c270_camera parent_link="axle_scte_front" camera_link="left_cam" joint_xyz="0 0.15 ${scte_chassis_width * 0.65 * -1.0}" joint_rpy="0 0 0"/>
     <xacro:logitech_c270_camera parent_link="axle_scte_front" camera_link="right_cam" joint_xyz="0 0.15 ${scte_chassis_width * 0.65}" joint_rpy="0 0 0"/>
-    <!---->
-    <!--sensors-->
-    <!--cameras-->
-    <!--joint name="scte_chassis_JOINT_left_camera" type="fixed">
-        <origin xyz="0 0 0" rpy="0 0 0"/>
-        <parent link="scte_chassis"/>
-        <child link="left_cam"/>
-        <axis xyz="0 0 0" rpy="0 0 0"/>
-    </joint-->
     <!--link name='main_computer'>
     <inertial>

Commit message: added computer box and placed cameras on top of it

File: src/models/scte_vehicle/scte_description/urdf/scte_chassis.xacro (robot description, xacro)
@@ -160,10 +160,41 @@
     <!---->
     <!--/MOUNTING BARS-->
-    <!--sensors-->
-    <!--
+    <!--COMPUTER ENCLOSURE-->
+    <link name="main_computer_enclosure">
+        <inertial>
+            <mass value="${scte_total_mass * 0.02}"/>
+            <origin xyz="0 0 0" rpy="0 0 0"/>
+            <inertia
+                    ixx="1" ixy="0" ixz="0"
+                    iyy="1" iyz="0"
+                    izz="1"
+            />
+        </inertial>
+        <visual name='visual'>
+            <origin xyz="0 0 0" rpy="0 0 0"/>
+            <geometry>
+                <box size="0.263 0.185 0.06"/>
+            </geometry>
+            <material name="blue"/>
+        </visual>
+        <collision name='collision'>
+            <origin xyz="0 0 0" rpy="0 0 0"/>
+            <geometry>
+                <box size="0.263 0.185 0.06"/>
+            </geometry>
+        </collision>
+    </link>
+    <joint name="main_computer_enclosure_LINKED_driver_side_mounting_bar" type="fixed">
+        <origin xyz="0 ${(scte_chassis_width * -0.5) + (mounting_bars_width * 0.5)} ${0.06 * 0.5}" rpy="0 0 0"/>
+        <parent link="driver_side_mounting_bar"/>
+        <child link="main_computer_enclosure"/>
+    </joint>
+    <!--/COMPUTER ENCLOSURE-->
+    <!--SENSORS-->
+    <!---->
     <xacro:include filename="$(find logitech_c270_camera)/urdf/logitech_c270.xacro"/>
-    <xacro:logitech_c270_camera parent_link="axle_scte_front" camera_link="left_cam" joint_xyz="0 0.15 ${scte_chassis_width * 0.65 * -1.0}" joint_rpy="0 0 0"/>
-    <xacro:logitech_c270_camera parent_link="axle_scte_front" camera_link="right_cam" joint_xyz="0 0.15 ${scte_chassis_width * 0.65}" joint_rpy="0 0 0"/>
-    -->
+    <xacro:logitech_c270_camera parent_link="main_computer_enclosure" camera_link="left_cam" joint_xyz="0 -0.05 0.05" joint_rpy="${M_PI/2} 0 0"/>
+    <xacro:logitech_c270_camera parent_link="main_computer_enclosure" camera_link="right_cam" joint_xyz="0 0.05 0.05" joint_rpy="${M_PI/2} 0 0"/>
+    <!---->
     <!--LIDAR-->
     <!--xacro:include filename="$(find SOMESENSOR_description)/urdf/SENSOR.urdf.xacro"/>
@@ -171,24 +202,3 @@
         <origin xyz="0 0 0" rpy="0 0 0" />
     </SOMESENSOR-->
-    <!--link name='main_computer'>
-    <inertial>
-        <mass value="1"/>
-        <inertia
-                ixx="1" ixy="0" ixz="0"
-                iyy="1" iyz="0"
-                izz="1"
-        />
-    </inertial>
-    <visual name='visual'>
-        <geometry>
-            <box size="1 1 1"/>
-        </geometry>
-        <material name="white"/>
-    </visual>
-    <collision name='collision'>
-        <geometry>
-            <box size="1 1 1"/>
-        </geometry>
-    </collision>
-    </link-->
 </robot>

Commit message: added an optical frame

File: src/models/scte_vehicle/scte_description/urdf/scte_chassis.xacro (robot description, xacro)
@@ -194,6 +194,6 @@
     <!---->
     <xacro:include filename="$(find logitech_c270_camera)/urdf/logitech_c270.xacro"/>
-    <xacro:logitech_c270_camera parent_link="main_computer_enclosure" camera_link="left_cam" joint_xyz="0 -0.05 0.05" joint_rpy="${M_PI/2} 0 0"/>
-    <xacro:logitech_c270_camera parent_link="main_computer_enclosure" camera_link="right_cam" joint_xyz="0 0.05 0.05" joint_rpy="${M_PI/2} 0 0"/>
+    <xacro:logitech_c270_camera parent_link="main_computer_enclosure" camera_link="driver_side_camera" joint_xyz="0 -0.05 0.05" joint_rpy="0 0 0"/>
+    <xacro:logitech_c270_camera parent_link="main_computer_enclosure" camera_link="passenger_side_camera" joint_xyz="0 0.05 0.05" joint_rpy="0 0 0"/>
     <!---->
     <!--LIDAR-->

File: src/sensors/logitech_c270_camera/urdf/logitech_c270.xacro (robot description, xacro)
@@ -4,7 +4,4 @@
     <!--https://answers.ros.org/question/331432/pass-parameters-of-xacro-file-in-another-xacro-file/-->
     <xacro:macro name="logitech_c270_camera" params="parent_link camera_link joint_xyz joint_rpy">
-        <!--camera params-->
-        <xacro:property name="logitech_c270_radius" value="0.02"/>
-        <xacro:property name="logitech_c270_length" value="0.08"/>
         <link name='${camera_link}'>
             <inertial>
@@ -18,14 +15,17 @@
             </inertial>
             <visual name='visual'>
+                <transparency>1</transparency>
                 <origin xyz="0 0 0" rpy="0 0 0"/>
                 <geometry>
-                    <cylinder radius="${logitech_c270_radius}" length="${logitech_c270_length}"/>
+                    <box size="0.075 0.075 0.025"/>
                 </geometry>
-                <material name="blue"/>
+                <material name="none">
+                    <color rgba="${122/255} ${125/255} ${121/255} 0.5"/>
+                </material>
             </visual>
             <collision name='collision'>
                 <origin xyz="0 0 0" rpy="0 0 0"/>
                 <geometry>
-                    <cylinder radius="${logitech_c270_radius}" length="${logitech_c270_length}"/>
+                    <box size="0.075 0.075 0.025"/>
                 </geometry>
             </collision>
@@ -36,4 +36,24 @@
             <child link="${camera_link}"/>
         </joint>
+        <link name="${camera_link}_optical">
+            <visual name='visual'>
+                <origin xyz="0 0 0" rpy="0 0 0"/>
+                <geometry>
+                    <box size="0.01 0.01 0.01"/>
+                </geometry>
+                <material name="red"/>
+            </visual>
+            <collision name='collision'>
+                <origin xyz="0 0 0" rpy="0 0 0"/>
+                <geometry>
+                    <box size="0.01 0.01 0.01"/>
+                </geometry>
+            </collision>
+        </link>
+        <joint name="${camera_link}_base_optical_JOINT_${camera_link}_link" type="fixed">
+            <origin xyz="0.03 0.015 0" rpy="${M_PI/-2} 0 ${M_PI/-2}"/>
+            <parent link="${camera_link}"/>
+            <child link="${camera_link}_optical"/>
+        </joint>
     </xacro:macro>
 </robot>

Commit message: added ydlidar to model and rViz

File: src/models/scte_vehicle/scte_description/urdf/scte_chassis.xacro (robot description, xacro)
@@ -194,11 +194,13 @@
     <!---->
     <xacro:include filename="$(find logitech_c270_camera)/urdf/logitech_c270.xacro"/>
-    <xacro:logitech_c270_camera parent_link="main_computer_enclosure" camera_link="driver_side_camera" joint_xyz="0 0.05 0.5" joint_rpy="0 ${M_PI/-6} 0"/>
-    <xacro:logitech_c270_camera parent_link="main_computer_enclosure" camera_link="passenger_side_camera" joint_xyz="0 -0.05 0.5" joint_rpy="0 ${M_PI/-6} 0"/>
+    <xacro:logitech_c270_camera parent_link="main_computer_enclosure" camera_link="driver_side_camera" joint_xyz="0.105 0.05 0.05" joint_rpy="0 0 0"/>
+    <xacro:logitech_c270_camera parent_link="main_computer_enclosure" camera_link="passenger_side_camera" joint_xyz="0.105 -0.05 0.05" joint_rpy="0 0 0"/>
     <!---->
     <!--LIDAR-->
-    <!--xacro:include filename="$(find SOMESENSOR_description)/urdf/SENSOR.urdf.xacro"/>
-    <SOMESENSOR parent="scte_chassis" name="SOMESENSOR_sensor" hz="10" samples="220" lasers="16">
-        <origin xyz="0 0 0" rpy="0 0 0" />
-    </SOMESENSOR-->
+    <xacro:include filename="$(find ydlidar_ros)/urdf/ydlidar.urdf"/>
+    <joint name="main_computer_enclosure_LINKED_ydlidar_base" type="fixed">
+        <origin xyz="0 0 0.0305" rpy="0 0 0"/>
+        <parent link="main_computer_enclosure"/>
+        <child link="base_laser"/>
+    </joint>
 </robot>
