Commit message: added camera mount and moved lidar

File: src/models/scte_vehicle/scte_description/urdf/scte_chassis.xacro (robot description, xacro)
@@ -176,5 +176,7 @@
                 <box size="0.263 0.185 0.06"/>
             </geometry>
-            <material name="blue"/>
+            <material name="none">
+                <color rgba="${122/255} ${125/255} ${121/255} 0.5"/>
+            </material>
         </visual>
         <collision name='collision'>
@@ -193,12 +195,70 @@
     <!--SENSORS-->
     <!---->
+    <link name="stereo_camera_bar_support">
+        <inertial>
+            <mass value="${scte_total_mass * 0.01}"/>
+            <origin xyz="0 0 0" rpy="0 0 0"/>
+            <inertia
+                    ixx="1" ixy="0" ixz="0"
+                    iyy="1" iyz="0"
+                    izz="1"
+            />
+        </inertial>
+        <visual name='visual'>
+            <origin xyz="0 0 0" rpy="0 0 0"/>
+            <geometry>
+                <cylinder radius="0.01" length="0.06"/>
+            </geometry>
+            <material name="blue"/>
+        </visual>
+        <collision name='collision'>
+            <origin xyz="0 0 0" rpy="0 0 0"/>
+            <geometry>
+                <cylinder radius="0.01" length="0.06"/>
+            </geometry>
+        </collision>
+    </link>
+    <joint name="stereo_camera_bar_support_LINKED_main_computer_enclosure" type="fixed">
+        <origin xyz="${0.263 * -0.45} 0 ${0.06 * 1.0}" rpy="0 0 0"/>
+        <parent link="main_computer_enclosure"/>
+        <child link="stereo_camera_bar_support"/>
+    </joint>
+    <link name="stereo_camera_bar">
+        <inertial>
+            <mass value="${scte_total_mass * 0.01}"/>
+            <origin xyz="0 0 0" rpy="0 0 0"/>
+            <inertia
+                    ixx="1" ixy="0" ixz="0"
+                    iyy="1" iyz="0"
+                    izz="1"
+            />
+        </inertial>
+        <visual name='visual'>
+            <origin xyz="0 0 0" rpy="0 0 0"/>
+            <geometry>
+                <box size="0.03 0.202 0.004"/>
+            </geometry>
+            <material name="blue"/>
+        </visual>
+        <collision name='collision'>
+            <origin xyz="0 0 0" rpy="0 0 0"/>
+            <geometry>
+                <box size="0.03 0.202 0.004"/>
+            </geometry>
+        </collision>
+    </link>
+    <joint name="stereo_camera_bar_LINKED_stereo_camera_bar_support" type="fixed">
+        <origin xyz="0 0 ${0.06 * 0.5}" rpy="0 0 0"/>
+        <parent link="stereo_camera_bar_support"/>
+        <child link="stereo_camera_bar"/>
+    </joint>
     <xacro:include filename="$(find logitech_c270_camera)/urdf/logitech_c270.xacro"/>
-    <xacro:logitech_c270_camera parent_link="main_computer_enclosure" camera_link="driver_side_camera" joint_xyz="0.105 0.05 0.05" joint_rpy="0 0 0"/>
-    <xacro:logitech_c270_camera parent_link="main_computer_enclosure" camera_link="passenger_side_camera" joint_xyz="0.105 -0.05 0.05" joint_rpy="0 0 0"/>
+    <xacro:logitech_c270_camera parent_link="stereo_camera_bar" camera_link="driver_side_camera" joint_xyz="0.0 0.05 ${0.025 * 0.5}" joint_rpy="0 0 0"/>
+    <xacro:logitech_c270_camera parent_link="stereo_camera_bar" camera_link="passenger_side_camera" joint_xyz="0.0 -0.05 ${0.025 * 0.5}" joint_rpy="0 0 0"/>
     <!---->
     <!--LIDAR-->
     <xacro:include filename="$(find ydlidar_ros)/urdf/ydlidar.urdf"/>
     <joint name="main_computer_enclosure_LINKED_ydlidar_base" type="fixed">
-        <origin xyz="0 0 0.0305" rpy="0 0 0"/>
+        <origin xyz="0.090 0 0.0305" rpy="0 0 0"/>
         <parent link="main_computer_enclosure"/>
         <child link="base_laser"/>

Commit message: corrected LIDAR transform frame

File: src/models/scte_vehicle/scte_description/urdf/scte_chassis.xacro (robot description, xacro)
@@ -174,5 +174,5 @@
             <origin xyz="0 0 0" rpy="0 0 0"/>
             <geometry>
-                <box size="0.263 0.185 0.06"/>
+                <box size="0.26 0.185 0.06"/>
             </geometry>
             <material name="none">
@@ -183,5 +183,5 @@
             <origin xyz="0 0 0" rpy="0 0 0"/>
             <geometry>
-                <box size="0.263 0.185 0.06"/>
+                <box size="0.26 0.185 0.06"/>
             </geometry>
         </collision>
@@ -220,5 +220,5 @@
     </link>
     <joint name="stereo_camera_bar_support_LINKED_main_computer_enclosure" type="fixed">
-        <origin xyz="${0.263 * -0.45} 0 ${0.06 * 1.0}" rpy="0 0 0"/>
+        <origin xyz="${0.260 * -0.45} 0 ${0.06 * 1.0}" rpy="0 0 0"/>
         <parent link="main_computer_enclosure"/>
         <child link="stereo_camera_bar_support"/>

Commit message: still debugging the stereo point cloud ref frame

File: src/models/scte_vehicle/scte_description/urdf/scte_chassis.xacro (robot description, xacro)
@@ -254,7 +254,42 @@
     </joint>
     <xacro:include filename="$(find logitech_c270_camera)/urdf/logitech_c270.xacro"/>
+    <!--https://answers.ros.org/question/9840/how-do-you-get-stereo_image_proc-to-include-a-frame_id-so-that-rviz-will-accept-the-point-cloud-messages/-->
+    <!--stereo projection/point cloud uses the left cameras frame_id to determine how to draw the image-->
+    <!-- may need to use image_rect for the video to align with the model
+    https://berndpfrommer.github.io/tagslam_web/visualization/
+    -->
     <xacro:logitech_c270_camera parent_link="stereo_camera_bar" camera_link="driver_side_camera" joint_xyz="0.0 0.05 ${0.025 * 0.5}" joint_rpy="0 0 0"/>
     <xacro:logitech_c270_camera parent_link="stereo_camera_bar" camera_link="passenger_side_camera" joint_xyz="0.0 -0.05 ${0.025 * 0.5}" joint_rpy="0 0 0"/>
-    <!---->
+    <!--
+    <link name="debug_stereo_perception_camera">
+        <inertial>
+            <mass value="${scte_total_mass * 0.0001}"/>
+            <origin xyz="0 0 0" rpy="0 0 0"/>
+            <inertia
+                    ixx="1" ixy="0" ixz="0"
+                    iyy="1" iyz="0"
+                    izz="1"
+            />
+        </inertial>
+        <visual name='visual'>
+            <origin xyz="0 0 0" rpy="0 0 0"/>
+            <geometry>
+                <box size="0.05 0.05 0.05"/>
+            </geometry>
+            <material name="blue"/>
+        </visual>
+        <collision name='collision'>
+            <origin xyz="0 0 0" rpy="0 0 0"/>
+            <geometry>
+                <box size="0.05 0.05 0.05"/>
+            </geometry>
+        </collision>
+    </link>
+    <joint name="debug_stereo_perception_camera_LINKED_stereo_camera_bar" type="fixed">
+        <origin xyz="0 0.5 0" rpy="${M_PI/-2} 0 ${M_PI/-2}"/>
+        <parent link="stereo_camera_bar"/>
+        <child link="debug_stereo_perception_camera"/>
+    </joint>
+    -->
     <!--LIDAR-->
     <xacro:include filename="$(find ydlidar_ros)/urdf/ydlidar.urdf"/>

Commit message: further tweaks to odom and robot localization integration

File: src/models/scte_vehicle/scte_description/urdf/scte_chassis.xacro (robot description, xacro)
@@ -18,4 +18,38 @@
         <child link="scte_chassis"/>
     </joint>
+    <!--DEBUG test link for odom testing-->
+    <link name="test_real_link">
+        <inertial>
+            <mass value="1.0"/>
+            <origin xyz="0 0 0" rpy="0 0 0"/>
+            <inertia
+                    ixx="1" ixy="0" ixz="0"
+                    iyy="1" iyz="0"
+                    izz="1"
+            />
+        </inertial>
+        <visual name='visual'>
+            <transparency>1</transparency>
+            <origin xyz="0 0 0" rpy="0 0 0"/>
+            <geometry>
+                <box size="0.075 0.075 0.075"/>
+            </geometry>
+            <material name="none1">
+                <color rgba="${255/255} ${0/255} ${0/255} 1.0"/>
+            </material>
+        </visual>
+        <collision name='collision'>
+            <origin xyz="0 0 0" rpy="0 0 0"/>
+            <geometry>
+                <box size="0.075 0.075 0.075"/>
+            </geometry>
+        </collision>
+    </link>
+    <joint name="odom_test" type="fixed">
+        <origin xyz="0 0.0 1.0" rpy="0 0 0"/>
+        <parent link="scte_chassis"/>
+        <child link="test_real_link"/>
+    </joint>
+    <!--DEBUG test link for odom testing-->
     <!--CHASSIS-->
     <xacro:property name="scte_total_mass" value="3.8"/>

Commit message: still working on cleaning up the model

File: src/models/scte_vehicle/scte_description/urdf/scte_chassis.xacro (robot description, xacro)
@@ -22,4 +22,15 @@
     <!--Wheel Properties-->
     <xacro:property name="wheel_radius" value="0.05"/>
+    <xacro:property name="wheel_length" value="0.045"/>
+    <xacro:property name="shock_tower_height" value="0.105"/>
+    <xacro:property name="shock_tower_width" value="0.14"/>
+    <xacro:property name="drive_axle_length" value="0.25"/>
+    <xacro:property name="drive_axle_radius" value="0.005"/>
+    <link name='base_footprint'/>
+    <joint name="base_footprint_joint" type="fixed">
+        <origin xyz="0 0 ${scte_chassis_depth - wheel_radius}" rpy="0 0 0"/>
+        <parent link="base_link"/>
+        <child link="base_footprint"/>
+    </joint>
     <link name='base_link'>
         <visual name='visual'>
@@ -37,10 +48,4 @@
         </collision>
     </link>
-    <link name='base_footprint'/>
-    <joint name="base_footprint_joint" type="fixed">
-        <origin xyz="0 0 ${scte_chassis_depth - wheel_radius}" rpy="0 0 0"/>
-        <parent link="base_link"/>
-        <child link="base_footprint"/>
-    </joint>
     <!-- Inertial link stores the robot's inertial information -->
     <link name="inertial_link">
@@ -63,9 +68,89 @@
         <child link="scte_chassis"/>
     </joint>
-    <xacro:include filename="$(find scte_description)/urdf/scte_axle_components.xacro"/>
+    <xacro:include filename="$(find scte_description)/urdf/scte_diff_and_shock_tower.xacro"/>
+    <xacro:scte_diff_and_shock_tower link_name="front_diff_tower"
+                                parent_link="scte_chassis"
+                                diff_joint_xyz="${scte_chassis_length * 0.63} 0 0"
+                                diff_joint_rpy="0 0 0"
+                                diff_plate_size="0.07 0.07 ${scte_chassis_depth}"
+                                shock_tower_size="0.015 ${shock_tower_width} ${shock_tower_height}"
+                                shock_tower_joint_origin="0 0 ${shock_tower_height * 0.5}"
+                                shock_tower_joint_rpy="0 0 0"
+    />
+    <xacro:scte_diff_and_shock_tower link_name="rear_diff_tower"
+                                     parent_link="scte_chassis"
+                                     diff_joint_xyz="${scte_chassis_length * -0.63} 0 0"
+                                     diff_joint_rpy="0 0 0"
+                                     diff_plate_size="0.07 0.07 ${scte_chassis_depth}"
+                                     shock_tower_size="0.015 ${shock_tower_width} ${shock_tower_height}"
+                                     shock_tower_joint_origin="0 0 ${shock_tower_height * 0.5}"
+                                     shock_tower_joint_rpy="0 0 0"
+    />
+    <xacro:include filename="$(find scte_description)/urdf/scte_front_bumper.xacro"/>
+    <xacro:scte_front_bumper link_name="front_bumper"
+                             parent_link="front_diff_tower"
+                             front_skid_plate_size="0.07 0.07 ${scte_chassis_depth}"
+                             front_skid_plate_joint_xyz="${0.07} 0 ${0.07 * 0.30}"
+                             front_skid_plate_joint_rpy="0 ${M_PI/-6}  0"
+                             front_bumper_size="0.01 0.175 0.05"
+    />
+    <xacro:include filename="$(find scte_description)/urdf/scte_rear_bumper.xacro"/>
+    <xacro:scte_rear_bumper link_name="rear_bumper"
+                            parent_link="rear_diff_tower"
+                            rear_bumper_size="0.01 0.255 0.05"
+                            rear_bumper_mount_size="0.09 0.05 0.05"
+                            rear_bumper_mount_joint_xyz="${0.09 * -0.6} 0 ${shock_tower_height * 0.5}"
+                            rear_bumper_mount_joint_rpy="0 0 0"
+    />
+    <link name="front_axle">
+        <visual name='visual'>
+            <geometry>
+                <cylinder radius="${drive_axle_radius}" length="${drive_axle_length}"/>
+            </geometry>
+            <material name="red"/>
+        </visual>
+        <collision name='collision'>
+            <geometry>
+                <cylinder radius="${drive_axle_radius}" length="${drive_axle_length}"/>
+            </geometry>
+        </collision>
+    </link>
+    <joint name='front_axle_TO_front_diff_tower' type='fixed'>
+        <origin xyz="0 0 ${0.03 * 0.5}" rpy="${M_PI * 0.5} 0 0"/>
+        <parent link="front_diff_tower"/>
+        <child link="front_axle"/>
+    </joint>
+    <link name="rear_axle">
+        <visual name='visual'>
+            <geometry>
+                <cylinder radius="${drive_axle_radius}" length="${drive_axle_length}"/>
+            </geometry>
+            <material name="red"/>
+        </visual>
+        <collision name='collision'>
+            <geometry>
+                <cylinder radius="${drive_axle_radius}" length="${drive_axle_length}"/>
+            </geometry>
+        </collision>
+    </link>
+    <joint name='rear_axle_TO_front_diff_tower' type='fixed'>
+        <origin xyz="0 0 ${0.03 * 0.5}" rpy="${M_PI * 0.5} 0 0"/>
+        <parent link="rear_diff_tower"/>
+        <child link="rear_axle"/>
+    </joint>
+    <xacro:include filename="$(find scte_description)/urdf/scte_wheel.xacro"/>
+    <xacro:scte_wheel link_name="front_left_wheel"
+                      parent_link="front_axle"
+                      wheel_radius="${wheel_radius}"
+                      wheel_length="${wheel_length}"
+                      wheel_joint_origin="0 0 ${drive_axle_length * 0.5}"
+                      wheel_joint_rpy="0 0 0"
+    />
+    <!--
     <xacro:property name="drive_axle_length" value="0.25"/>
     <xacro:property name="drive_axle_radius" value="0.005"/>
     <xacro:property name="shock_tower_height" value="0.105"/>
     <xacro:property name="shock_tower_width" value="0.14"/>
+    <xacro:include filename="$(find scte_description)/urdf/scte_axle_components.xacro"/>
     <xacro:scte_axle_components suffix="front"
         parent_link="scte_chassis"
@@ -110,214 +195,5 @@
         right_wheel_joint_rpy="0 0 0"
     />
+    -->
     <!--/CHASSIS-->
-    <!--MOUNTING BARS-->
-    <!---->
-    <xacro:property name="mounting_bars_length" value="0.45"/>
-    <xacro:property name="mounting_bars_width" value="0.025"/>
-    <xacro:property name="mounting_bars_depth" value="0.005"/>
-    <link name="driver_side_mounting_bar">
-        <inertial>
-            <mass value="${scte_total_mass * 0.02}"/>
-            <origin xyz="0 0 0" rpy="0 0 0"/>
-            <inertia
-                    ixx="1" ixy="0" ixz="0"
-                    iyy="1" iyz="0"
-                    izz="1"
-            />
-        </inertial>
-        <visual name='visual'>
-            <origin xyz="0 0 0" rpy="0 0 0"/>
-            <geometry>
-                <box size="${mounting_bars_length} ${mounting_bars_width} ${mounting_bars_depth}"/>
-            </geometry>
-            <material name="green"/>
-        </visual>
-        <collision name='collision'>
-            <origin xyz="0 0 0" rpy="0 0 0"/>
-            <geometry>
-                <box size="${mounting_bars_length} ${mounting_bars_width} ${mounting_bars_depth}"/>
-            </geometry>
-        </collision>
-    </link>
-    <joint name="shock_tower_front_JOINED_driver_side_mounting_bar" type="fixed">
-        <origin xyz="${scte_chassis_length * -0.63} ${shock_tower_width * 0.5} ${shock_tower_height * 0.5}" rpy="0 -0 0"/>
-        <parent link="shock_tower_front"/>
-        <child link="driver_side_mounting_bar"/>
-    </joint>
-    <link name="passenger_side_mounting_bar">
-        <inertial>
-            <mass value="${scte_total_mass * 0.02}"/>
-            <origin xyz="0 0 0" rpy="0 0 0"/>
-            <inertia
-                    ixx="1" ixy="0" ixz="0"
-                    iyy="1" iyz="0"
-                    izz="1"
-            />
-        </inertial>
-        <visual name='visual'>
-            <origin xyz="0 0 0" rpy="0 0 0"/>
-            <geometry>
-                <box size="${mounting_bars_length} ${mounting_bars_width} ${mounting_bars_depth}"/>
-            </geometry>
-            <material name="green"/>
-        </visual>
-        <collision name='collision'>
-            <origin xyz="0 0 0" rpy="0 0 0"/>
-            <geometry>
-                <box size="${mounting_bars_length} ${mounting_bars_width} ${mounting_bars_depth}"/>
-            </geometry>
-        </collision>
-    </link>
-    <joint name="shock_tower_front_JOINED_passenger_side_mounting_bar" type="fixed">
-        <origin xyz="${scte_chassis_length * -0.63} ${shock_tower_width * -0.5} ${shock_tower_height * 0.5}" rpy="0 -0 0"/>
-        <parent link="shock_tower_front"/>
-        <child link="passenger_side_mounting_bar"/>
-    </joint>
-    <!---->
-    <!--/MOUNTING BARS-->
-    <!--COMPUTER ENCLOSURE-->
-    <link name="main_computer_enclosure">
-        <inertial>
-            <mass value="${scte_total_mass * 0.02}"/>
-            <origin xyz="0 0 0" rpy="0 0 0"/>
-            <inertia
-                    ixx="1" ixy="0" ixz="0"
-                    iyy="1" iyz="0"
-                    izz="1"
-            />
-        </inertial>
-        <visual name='visual'>
-            <origin xyz="0 0 0" rpy="0 0 0"/>
-            <geometry>
-                <box size="0.26 0.185 0.06"/>
-            </geometry>
-            <material name="none">
-                <color rgba="${122/255} ${125/255} ${121/255} 0.5"/>
-            </material>
-        </visual>
-        <collision name='collision'>
-            <origin xyz="0 0 0" rpy="0 0 0"/>
-            <geometry>
-                <box size="0.26 0.185 0.06"/>
-            </geometry>
-        </collision>
-    </link>
-    <joint name="main_computer_enclosure_JOINED_driver_side_mounting_bar" type="fixed">
-        <origin xyz="0 ${(scte_chassis_width * -0.5) + (mounting_bars_width * 0.5)} ${0.06 * 0.5}" rpy="0 0 0"/>
-        <parent link="driver_side_mounting_bar"/>
-        <child link="main_computer_enclosure"/>
-    </joint>
-    <!--/COMPUTER ENCLOSURE-->
-    <!--SENSORS-->
-    <!---->
-    <link name="stereo_camera_bar_support">
-        <inertial>
-            <mass value="${scte_total_mass * 0.01}"/>
-            <origin xyz="0 0 0" rpy="0 0 0"/>
-            <inertia
-                    ixx="1" ixy="0" ixz="0"
-                    iyy="1" iyz="0"
-                    izz="1"
-            />
-        </inertial>
-        <visual name='visual'>
-            <origin xyz="0 0 0" rpy="0 0 0"/>
-            <geometry>
-                <cylinder radius="0.01" length="0.06"/>
-            </geometry>
-            <material name="blue"/>
-        </visual>
-        <collision name='collision'>
-            <origin xyz="0 0 0" rpy="0 0 0"/>
-            <geometry>
-                <cylinder radius="0.01" length="0.06"/>
-            </geometry>
-        </collision>
-    </link>
-    <joint name="stereo_camera_bar_support_JOINED_main_computer_enclosure" type="fixed">
-        <origin xyz="${0.260 * -0.45} 0 ${0.06 * 1.0}" rpy="0 0 0"/>
-        <parent link="main_computer_enclosure"/>
-        <child link="stereo_camera_bar_support"/>
-    </joint>
-    <link name="stereo_camera_bar">
-        <inertial>
-            <mass value="${scte_total_mass * 0.01}"/>
-            <origin xyz="0 0 0" rpy="0 0 0"/>
-            <inertia
-                    ixx="1" ixy="0" ixz="0"
-                    iyy="1" iyz="0"
-                    izz="1"
-            />
-        </inertial>
-        <visual name='visual'>
-            <origin xyz="0 0 0" rpy="0 0 0"/>
-            <geometry>
-                <box size="0.03 0.202 0.004"/>
-            </geometry>
-            <material name="blue"/>
-        </visual>
-        <collision name='collision'>
-            <origin xyz="0 0 0" rpy="0 0 0"/>
-            <geometry>
-                <box size="0.03 0.202 0.004"/>
-            </geometry>
-        </collision>
-    </link>
-    <joint name="stereo_camera_bar_JOINED_stereo_camera_bar_support" type="fixed">
-        <origin xyz="0 0 ${0.06 * 0.5}" rpy="0 0 0"/>
-        <parent link="stereo_camera_bar_support"/>
-        <child link="stereo_camera_bar"/>
-    </joint>
-    <xacro:include filename="$(find logitech_c270_camera)/urdf/logitech_c270.xacro"/>
-    <!--https://answers.ros.org/question/9840/how-do-you-get-stereo_image_proc-to-include-a-frame_id-so-that-rviz-will-accept-the-point-cloud-messages/-->
-    <!--stereo projection/point cloud uses the left cameras frame_id to determine how to draw the image-->
-    <!-- may need to use image_rect for the video to align with the model
-    https://berndpfrommer.github.io/tagslam_web/visualization/
-    -->
-    <xacro:logitech_c270_camera parent_link="stereo_camera_bar" camera_link="driver_side_camera" joint_xyz="0.0 0.05 ${0.025 * 0.5}" joint_rpy="0 0 0"/>
-    <xacro:logitech_c270_camera parent_link="stereo_camera_bar" camera_link="passenger_side_camera" joint_xyz="0.0 -0.05 ${0.025 * 0.5}" joint_rpy="0 0 0"/>
-    <!--
-    <link name="debug_stereo_perception_camera">
-        <inertial>
-            <mass value="${scte_total_mass * 0.0001}"/>
-            <origin xyz="0 0 0" rpy="0 0 0"/>
-            <inertia
-                    ixx="1" ixy="0" ixz="0"
-                    iyy="1" iyz="0"
-                    izz="1"
-            />
-        </inertial>
-        <visual name='visual'>
-            <origin xyz="0 0 0" rpy="0 0 0"/>
-            <geometry>
-                <box size="0.05 0.05 0.05"/>
-            </geometry>
-            <material name="blue"/>
-        </visual>
-        <collision name='collision'>
-            <origin xyz="0 0 0" rpy="0 0 0"/>
-            <geometry>
-                <box size="0.05 0.05 0.05"/>
-            </geometry>
-        </collision>
-    </link>
-    <joint name="debug_stereo_perception_camera_JOINED_stereo_camera_bar" type="fixed">
-        <origin xyz="0 0.5 0" rpy="${M_PI/-2} 0 ${M_PI/-2}"/>
-        <parent link="stereo_camera_bar"/>
-        <child link="debug_stereo_perception_camera"/>
-    </joint>
-    -->
-    <!--LIDAR-->
-    <xacro:include filename="$(find ydlidar_ros)/urdf/ydlidar.urdf"/>
-    <joint name="main_computer_enclosure_JOINED_ydlidar_base" type="fixed">
-        <origin xyz="0.090 0 0.0305" rpy="0 0 0"/>
-        <parent link="main_computer_enclosure"/>
-        <child link="base_laser"/>
-    </joint>
-    <!--gazebo>
-        <plugin name="gazebo_ros_control" filename="libgazebo_ros_control.so"-->
-            <!--robotNamespace>$(arg robot_namespace)</robotNamespace-->
-            <!--legacyModeNS>true</legacyModeNS>
-        </plugin>
-    </gazebo-->
 </robot>
