Commit message: debugging continuous link in gazebo

File: src/models/scte_vehicle/scte_description/urdf/scte_chassis.xacro (robot description, xacro)
@@ -103,4 +103,5 @@
                             rear_bumper_mount_joint_rpy="0 0 0"
     />
+    <gazebo reference="front_axle"/>
     <link name="front_axle">
         <visual name='visual'>
@@ -139,5 +140,5 @@
         <child link="rear_axle"/>
     </joint>
-    <xacro:include filename="$(find scte_description)/urdf/scte_wheel.xacro"/>
+    <!--xacro:include filename="$(find scte_description)/urdf/scte_wheel.xacro"/>
     <xacro:scte_wheel link_name="front_left_wheel"
                       parent_link="front_axle"
@@ -146,5 +147,39 @@
                       wheel_joint_origin="0 0 ${drive_axle_length * 0.5}"
                       wheel_joint_rpy="0 0 0"
-    />
+    /-->
+    <link name="left_wheel">
+        <inertial>
+            <mass value="0.5"/>
+            <inertia
+                    ixx="1" ixy="0" ixz="0"
+                    iyy="1" iyz="0"
+                    izz="1"
+            />
+        </inertial>
+        <visual name="visual">
+            <geometry>
+                <cylinder radius="0.1" length="0.05"/>
+            </geometry>
+        </visual>
+        <collision name='collision'>
+            <geometry>
+                <cylinder radius="0.1" length="0.05"/>
+            </geometry>
+        </collision>
+    </link>
+    <gazebo reference="left_wheel">
+        <mu1 value="1.0"/>
+        <mu2 value="1.0"/>
+        <kp value="10000000.0" />
+        <kd value="1.0" />
+        <fdir1 value="1 0 0"/>
+    </gazebo>
+    <joint name="left_wheel_JOIN_scte_chassis" type="continuous">
+        <child link="left_wheel"/>
+        <parent link="front_axle"/>
+        <origin xyz="0.1 0.15 0" rpy="0 1.5707 1.5707"/>
+        <dynamics damping="0.7"/>
+        <axis xyz="0 0 1"/>
+    </joint>
     <!--
     <xacro:property name="drive_axle_length" value="0.25"/>

File: src/models/scte_vehicle/scte_description/urdf/scte_wheel.xacro (robot description, xacro)
@@ -24,13 +24,4 @@
                 </collision>
             </link>
-            <joint name='${link_name}_TO_${parent_link}' type='continuous'>
-                <origin xyz="${wheel_joint_origin}" rpy="${wheel_joint_rpy}"/>
-                <parent link="${parent_link}"/>
-                <child link="${link_name}"/>
-                <axis xyz="0 0 1" rpy="0 0 0"/>
-                <axis xyz="0 0 1"/>
-                <dynamics damping="0.7"/>
-            </joint>
-            <!---->
             <gazebo reference="${link_name}">
                 <mu1 value="1.0"/>
@@ -40,4 +31,12 @@
                 <fdir1 value="1 0 0"/>
             </gazebo>
+            <joint name='${link_name}_TO_${parent_link}' type='continuous'>
+                <origin xyz="${wheel_joint_origin}" rpy="${wheel_joint_rpy}"/>
+                <parent link="${parent_link}"/>
+                <child link="${link_name}"/>
+                <axis xyz="0 0 1"/>
+                <dynamics damping="0.7"/>
+            </joint>
+            <!---->
             <!---->
             <transmission name="${link_name}_transmission" type="SimpleTransmission">

Commit message: more model work

File: src/models/scte_vehicle/scte_description/urdf/scte_chassis.xacro (robot description, xacro)
@@ -103,6 +103,13 @@
                             rear_bumper_mount_joint_rpy="0 0 0"
     />
-    <gazebo reference="front_axle"/>
-    <link name="front_axle">
+    <!--xacro:include filename="$(find scte_description)/urdf/scte_axle.xacro"/>
+    <xacro:scte_axle link_name="front_axle"
+                     parent_link="front_diff_tower"
+                     drive_axle_radius="${drive_axle_radius}"
+                     drive_axle_length="${drive_axle_length}"
+                     drive_axle_joint_xyz="0 0 ${0.03 * 0.5}"
+                     drive_axle_joint_rpy="${M_PI * 0.5} 0 0"
+    /-->
+    <!--link name="front_axle">
         <visual name='visual'>
             <geometry>
@@ -121,24 +128,6 @@
         <parent link="front_diff_tower"/>
         <child link="front_axle"/>
-    </joint>
-    <link name="rear_axle">
-        <visual name='visual'>
-            <geometry>
-                <cylinder radius="${drive_axle_radius}" length="${drive_axle_length}"/>
-            </geometry>
-            <material name="red"/>
-        </visual>
-        <collision name='collision'>
-            <geometry>
-                <cylinder radius="${drive_axle_radius}" length="${drive_axle_length}"/>
-            </geometry>
-        </collision>
-    </link>
-    <joint name='rear_axle_TO_front_diff_tower' type='fixed'>
-        <origin xyz="0 0 ${0.03 * 0.5}" rpy="${M_PI * 0.5} 0 0"/>
-        <parent link="rear_diff_tower"/>
-        <child link="rear_axle"/>
-    </joint>
-    <!--xacro:include filename="$(find scte_description)/urdf/scte_wheel.xacro"/>
+    </joint-->
+    <xacro:include filename="$(find scte_description)/urdf/scte_wheel.xacro"/>
     <xacro:scte_wheel link_name="front_left_wheel"
                       parent_link="front_axle"
@@ -147,5 +136,27 @@
                       wheel_joint_origin="0 0 ${drive_axle_length * 0.5}"
                       wheel_joint_rpy="0 0 0"
+    />
+    <xacro:scte_wheel link_name="front_right_wheel"
+                      parent_link="front_axle"
+                      wheel_radius="${wheel_radius}"
+                      wheel_length="${wheel_length}"
+                      wheel_joint_origin="0 0 ${drive_axle_length * -0.5}"
+                      wheel_joint_rpy="0 0 0"
+    />
+    <!--xacro:scte_wheel link_name="rear_left_wheel"
+                      parent_link="rear_axle"
+                      wheel_radius="${wheel_radius}"
+                      wheel_length="${wheel_length}"
+                      wheel_joint_origin="0 0 ${drive_axle_length * 0.5}"
+                      wheel_joint_rpy="0 0 0"
+    />
+    <xacro:scte_wheel link_name="rear_right_wheel"
+                      parent_link="rear_axle"
+                      wheel_radius="${wheel_radius}"
+                      wheel_length="${wheel_length}"
+                      wheel_joint_origin="0 0 ${drive_axle_length * -0.5}"
+                      wheel_joint_rpy="0 0 0"
     /-->
+    <!--
     <link name="left_wheel">
         <inertial>
@@ -182,53 +193,4 @@
         <axis xyz="0 0 1"/>
     </joint>
-    <!--
-    <xacro:property name="drive_axle_length" value="0.25"/>
-    <xacro:property name="drive_axle_radius" value="0.005"/>
-    <xacro:property name="shock_tower_height" value="0.105"/>
-    <xacro:property name="shock_tower_width" value="0.14"/>
-    <xacro:include filename="$(find scte_description)/urdf/scte_axle_components.xacro"/>
-    <xacro:scte_axle_components suffix="front"
-        parent_link="scte_chassis"
-        diff_joint_xyz="${scte_chassis_length * 0.63} 0 0"
-        diff_joint_rpy="0 0 0"
-        diff_plate_size="0.07 0.07 ${scte_chassis_depth}"
-        drive_axle_radius="${drive_axle_radius}"
-        drive_axle_length="${drive_axle_length}"
-        drive_axle_joint_origin="0 0 ${0.03 * 0.5}"
-        drive_axle_joint_rpy="${M_PI/2} 0 0"
-        shock_tower_size="0.015 ${shock_tower_width} ${shock_tower_height}"
-        shock_tower_joint_origin="0 0 ${shock_tower_height * 0.5}"
-        shock_tower_joint_rpy="0 0 0"
-        left_wheel_radius="${wheel_radius}"
-        left_wheel_length="0.045"
-        left_wheel_joint_origin="0 0 ${drive_axle_length * 0.5}"
-        left_wheel_joint_rpy="0 0 0"
-        right_wheel_radius="0.05"
-        right_wheel_length="0.045"
-        right_wheel_joint_origin="0 0 ${drive_axle_length * -0.5}"
-        right_wheel_joint_rpy="0 0 0"
-    />
-    <xacro:scte_axle_components suffix="rear"
-        parent_link="scte_chassis"
-        diff_joint_xyz="${scte_chassis_length * -0.63} 0 0"
-        diff_joint_rpy="0 0 0"
-        diff_plate_size="0.07 0.07 ${scte_chassis_depth}"
-        drive_axle_radius="${drive_axle_radius}"
-        drive_axle_length="${drive_axle_length}"
-        drive_axle_joint_origin="0 0 ${0.03 * 0.5}"
-        drive_axle_joint_rpy="${M_PI/2} 0 0"
-        shock_tower_size="0.015 ${shock_tower_width} ${shock_tower_height}"
-        shock_tower_joint_origin="0 0 ${shock_tower_height * 0.5}"
-        shock_tower_joint_rpy="0 0 0"
-        left_wheel_radius="0.05"
-        left_wheel_length="0.045"
-        left_wheel_joint_origin="0 0 ${drive_axle_length * 0.5}"
-        left_wheel_joint_rpy="0 0 0"
-        right_wheel_radius="0.05"
-        right_wheel_length="0.045"
-        right_wheel_joint_origin="0 0 ${drive_axle_length * -0.5}"
-        right_wheel_joint_rpy="0 0 0"
-    />
     -->
-    <!--/CHASSIS-->
 </robot>

File: src/models/scte_vehicle/scte_description/urdf/scte_wheel.xacro (robot description, xacro)
@@ -35,9 +35,8 @@
                 <parent link="${parent_link}"/>
                 <child link="${link_name}"/>
+                <axis xyz="0 0 1" rpy="0 0 0"/>
                 <axis xyz="0 0 1"/>
                 <dynamics damping="0.7"/>
             </joint>
-            <!---->
-            <!---->
             <transmission name="${link_name}_transmission" type="SimpleTransmission">
                 <type>transmission_interface/SimpleTransmission</type>
@@ -49,5 +48,4 @@
                 </joint>
             </transmission>
-            <!---->
         </xacro:macro>
 </robot>

Commit message: fixed wheel link, now showing up and responding to inputs. also fixed direction of travel and turns to match controller input for diff drive example

File: src/models/scte_vehicle/scte_description/urdf/scte_chassis.xacro (robot description, xacro)
@@ -103,30 +103,20 @@
                             rear_bumper_mount_joint_rpy="0 0 0"
     />
-    <!--xacro:include filename="$(find scte_description)/urdf/scte_axle.xacro"/>
-    <xacro:scte_axle link_name="front_axle"
+    <xacro:include filename="$(find scte_description)/urdf/scte_drive_axle.xacro"/>
+    <xacro:scte_drive_axle link_name="front_axle"
                      parent_link="front_diff_tower"
                      drive_axle_radius="${drive_axle_radius}"
                      drive_axle_length="${drive_axle_length}"
                      drive_axle_joint_xyz="0 0 ${0.03 * 0.5}"
-                     drive_axle_joint_rpy="${M_PI * 0.5} 0 0"
-    /-->
-    <!--link name="front_axle">
-        <visual name='visual'>
-            <geometry>
-                <cylinder radius="${drive_axle_radius}" length="${drive_axle_length}"/>
-            </geometry>
-            <material name="red"/>
-        </visual>
-        <collision name='collision'>
-            <geometry>
-                <cylinder radius="${drive_axle_radius}" length="${drive_axle_length}"/>
-            </geometry>
-        </collision>
-    </link>
-    <joint name='front_axle_TO_front_diff_tower' type='fixed'>
-        <origin xyz="0 0 ${0.03 * 0.5}" rpy="${M_PI * 0.5} 0 0"/>
-        <parent link="front_diff_tower"/>
-        <child link="front_axle"/>
-    </joint-->
+                     drive_axle_joint_rpy="${M_PI * -0.5} 0 0"
+    />
+    <xacro:include filename="$(find scte_description)/urdf/scte_drive_axle.xacro"/>
+    <xacro:scte_drive_axle link_name="rear_axle"
+                           parent_link="rear_diff_tower"
+                           drive_axle_radius="${drive_axle_radius}"
+                           drive_axle_length="${drive_axle_length}"
+                           drive_axle_joint_xyz="0 0 ${0.03 * 0.5}"
+                           drive_axle_joint_rpy="${M_PI * -0.5} 0 0"
+    />
     <xacro:include filename="$(find scte_description)/urdf/scte_wheel.xacro"/>
     <xacro:scte_wheel link_name="front_left_wheel"
@@ -144,5 +134,5 @@
                       wheel_joint_rpy="0 0 0"
     />
-    <!--xacro:scte_wheel link_name="rear_left_wheel"
+    <xacro:scte_wheel link_name="rear_left_wheel"
                       parent_link="rear_axle"
                       wheel_radius="${wheel_radius}"
@@ -157,40 +147,4 @@
                       wheel_joint_origin="0 0 ${drive_axle_length * -0.5}"
                       wheel_joint_rpy="0 0 0"
-    /-->
-    <!--
-    <link name="left_wheel">
-        <inertial>
-            <mass value="0.5"/>
-            <inertia
-                    ixx="1" ixy="0" ixz="0"
-                    iyy="1" iyz="0"
-                    izz="1"
-            />
-        </inertial>
-        <visual name="visual">
-            <geometry>
-                <cylinder radius="0.1" length="0.05"/>
-            </geometry>
-        </visual>
-        <collision name='collision'>
-            <geometry>
-                <cylinder radius="0.1" length="0.05"/>
-            </geometry>
-        </collision>
-    </link>
-    <gazebo reference="left_wheel">
-        <mu1 value="1.0"/>
-        <mu2 value="1.0"/>
-        <kp value="10000000.0" />
-        <kd value="1.0" />
-        <fdir1 value="1 0 0"/>
-    </gazebo>
-    <joint name="left_wheel_JOIN_scte_chassis" type="continuous">
-        <child link="left_wheel"/>
-        <parent link="front_axle"/>
-        <origin xyz="0.1 0.15 0" rpy="0 1.5707 1.5707"/>
-        <dynamics damping="0.7"/>
-        <axis xyz="0 0 1"/>
-    </joint>
-    -->
+    />
 </robot>

Commit message: code for ackermann steering tied to scte model, can make calls into some commands. Need to review to better understand what is going on

File: src/models/scte_vehicle/scte_description/urdf/scte_chassis.xacro (robot description, xacro)
@@ -28,8 +28,8 @@
     <xacro:property name="drive_axle_radius" value="0.005"/>
     <link name='base_footprint'/>
-    <joint name="base_footprint_joint" type="fixed">
+    <joint name="base_link_TO_base_footprint" type="fixed">
         <origin xyz="0 0 ${scte_chassis_depth - wheel_radius}" rpy="0 0 0"/>
-        <parent link="base_link"/>
-        <child link="base_footprint"/>
+        <parent link="base_footprint"/>
+        <child link="base_link"/>
     </joint>
     <link name='base_link'>

File: src/models/scte_vehicle/scte_description/urdf/scte_wheel.xacro (robot description, xacro)
@@ -48,4 +48,18 @@
                 </joint>
             </transmission>
+            <link name="${link_name}_steer">
+                <inertial>
+                    <origin xyz="-0.013054 -0.0295 0" rpy="0 0 0"/>
+                    <mass value="20.0"/>
+                    <inertia ixx="2" ixy="0" ixz="0" iyy="2" iyz="0" izz="2"/>
+                </inertial>
+            </link>
+            <joint name="${link_name}_steer_TO_${parent_link}" type="revolute">
+                <parent link="base_link" />
+                <child link="${link_name}_steer" />
+                <origin xyz="0 0 0" rpy="0 0 0" />
+                <axis xyz="0 0 1" />
+                <limit upper="0.6" lower="-0.6" effort="0.0" velocity="0.0" />
+            </joint>
         </xacro:macro>
 </robot>

Commit message: the gazebo model is now responding to steering cmds. The way I have it implemented, all four wheels are able to pivot. Need to fix this or maybe make it configurable?

File: src/models/scte_vehicle/scte_description/urdf/scte_chassis.xacro (robot description, xacro)
@@ -103,4 +103,5 @@
                             rear_bumper_mount_joint_rpy="0 0 0"
     />
+    <!--
     <xacro:include filename="$(find scte_description)/urdf/scte_drive_axle.xacro"/>
     <xacro:scte_drive_axle link_name="front_axle"
@@ -119,32 +120,33 @@
                            drive_axle_joint_rpy="${M_PI * -0.5} 0 0"
     />
+    -->
     <xacro:include filename="$(find scte_description)/urdf/scte_wheel.xacro"/>
     <xacro:scte_wheel link_name="front_left_wheel"
-                      parent_link="front_axle"
+                      parent_link="base_link"
                       wheel_radius="${wheel_radius}"
                       wheel_length="${wheel_length}"
-                      wheel_joint_origin="0 0 ${drive_axle_length * 0.5}"
-                      wheel_joint_rpy="0 0 0"
+                      wheel_joint_origin="${scte_chassis_length * 0.63} ${drive_axle_length * 0.5} 0"
+                      wheel_joint_rpy="${M_PI * -0.5} 0 0"
     />
     <xacro:scte_wheel link_name="front_right_wheel"
-                      parent_link="front_axle"
+                      parent_link="base_link"
                       wheel_radius="${wheel_radius}"
                       wheel_length="${wheel_length}"
-                      wheel_joint_origin="0 0 ${drive_axle_length * -0.5}"
-                      wheel_joint_rpy="0 0 0"
+                      wheel_joint_origin="${scte_chassis_length * 0.63} ${drive_axle_length * -0.5} 0"
+                      wheel_joint_rpy="${M_PI * -0.5} 0 0"
     />
     <xacro:scte_wheel link_name="rear_left_wheel"
-                      parent_link="rear_axle"
+                      parent_link="base_link"
                       wheel_radius="${wheel_radius}"
                       wheel_length="${wheel_length}"
-                      wheel_joint_origin="0 0 ${drive_axle_length * 0.5}"
-                      wheel_joint_rpy="0 0 0"
+                      wheel_joint_origin="${scte_chassis_length * -0.63} ${drive_axle_length * 0.5} 0"
+                      wheel_joint_rpy="${M_PI * -0.5} 0 0"
     />
     <xacro:scte_wheel link_name="rear_right_wheel"
-                      parent_link="rear_axle"
+                      parent_link="base_link"
                       wheel_radius="${wheel_radius}"
                       wheel_length="${wheel_length}"
-                      wheel_joint_origin="0 0 ${drive_axle_length * -0.5}"
-                      wheel_joint_rpy="0 0 0"
+                      wheel_joint_origin="${scte_chassis_length * -0.63} ${drive_axle_length * -0.5} 0"
+                      wheel_joint_rpy="${M_PI * -0.5} 0 0"
     />
 </robot>

File: src/models/scte_vehicle/scte_description/urdf/scte_wheel.xacro (robot description, xacro)
@@ -7,4 +7,28 @@
     wheel_joint_rpy
     ">
+            <gazebo reference="${link_name}">
+                <mu1 value="1.0"/>
+                <mu2 value="1.0"/>
+                <kp value="10000000.0" />
+                <kd value="1.0" />
+                <fdir1 value="1 0 0"/>
+            </gazebo>
+            <!---->
+            <link name="${link_name}_steer">
+                <inertial>
+                    <origin xyz="-0.013054 -0.0295 0" rpy="0 0 0"/>
+                    <mass value="20.0"/>
+                    <inertia ixx="2" ixy="0" ixz="0" iyy="2" iyz="0" izz="2"/>
+                </inertial>
+            </link>
+            <joint name="${link_name}_steer_TO_${parent_link}" type="revolute">
+                <parent link="${parent_link}" />
+                <child link="${link_name}_steer" />
+                <origin xyz="${wheel_joint_origin}" rpy="0 0 0" />
+                <axis xyz="0 0 1" />
+                <limit upper="0.6" lower="-0.6" effort="0.0" velocity="0.0" />
+            </joint>
+            <!---->
+            <!---->
             <link name="${link_name}">
                 <inertial>
@@ -24,18 +48,11 @@
                 </collision>
             </link>
-            <gazebo reference="${link_name}">
-                <mu1 value="1.0"/>
-                <mu2 value="1.0"/>
-                <kp value="10000000.0" />
-                <kd value="1.0" />
-                <fdir1 value="1 0 0"/>
-            </gazebo>
             <joint name='${link_name}_TO_${parent_link}' type='continuous'>
-                <origin xyz="${wheel_joint_origin}" rpy="${wheel_joint_rpy}"/>
-                <parent link="${parent_link}"/>
+                <parent link="${link_name}_steer"/>
                 <child link="${link_name}"/>
-                <axis xyz="0 0 1" rpy="0 0 0"/>
+                <origin xyz="0 0 0" rpy="${wheel_joint_rpy}"/>
                 <axis xyz="0 0 1"/>
                 <dynamics damping="0.7"/>
+                <limit effort="1000.0" velocity="22.0"/>
             </joint>
             <transmission name="${link_name}_transmission" type="SimpleTransmission">
@@ -48,18 +65,5 @@
                 </joint>
             </transmission>
-            <link name="${link_name}_steer">
-                <inertial>
-                    <origin xyz="-0.013054 -0.0295 0" rpy="0 0 0"/>
-                    <mass value="20.0"/>
-                    <inertia ixx="2" ixy="0" ixz="0" iyy="2" iyz="0" izz="2"/>
-                </inertial>
-            </link>
-            <joint name="${link_name}_steer_TO_${parent_link}" type="revolute">
-                <parent link="base_link" />
-                <child link="${link_name}_steer" />
-                <origin xyz="0 0 0" rpy="0 0 0" />
-                <axis xyz="0 0 1" />
-                <limit upper="0.6" lower="-0.6" effort="0.0" velocity="0.0" />
-            </joint>
+            <!---->
         </xacro:macro>
 </robot>
