Commit message: added a way to enable steering per wheel

File: src/models/scte_vehicle/scte_description/urdf/scte_chassis.xacro (robot description, xacro)
@@ -103,5 +103,4 @@
                             rear_bumper_mount_joint_rpy="0 0 0"
     />
-    <!--
     <xacro:include filename="$(find scte_description)/urdf/scte_drive_axle.xacro"/>
     <xacro:scte_drive_axle link_name="front_axle"
@@ -120,33 +119,36 @@
                            drive_axle_joint_rpy="${M_PI * -0.5} 0 0"
     />
-    -->
     <xacro:include filename="$(find scte_description)/urdf/scte_wheel.xacro"/>
     <xacro:scte_wheel link_name="front_left_wheel"
-                      parent_link="base_link"
+                      parent_link="front_axle"
                       wheel_radius="${wheel_radius}"
                       wheel_length="${wheel_length}"
-                      wheel_joint_origin="${scte_chassis_length * 0.63} ${drive_axle_length * 0.5} 0"
+                      wheel_joint_origin="0 0 ${drive_axle_length * 0.5}"
                       wheel_joint_rpy="${M_PI * -0.5} 0 0"
+                      is_steerable="true"
     />
     <xacro:scte_wheel link_name="front_right_wheel"
-                      parent_link="base_link"
+                      parent_link="front_axle"
                       wheel_radius="${wheel_radius}"
                       wheel_length="${wheel_length}"
-                      wheel_joint_origin="${scte_chassis_length * 0.63} ${drive_axle_length * -0.5} 0"
+                      wheel_joint_origin="0 0 ${drive_axle_length * -0.5}"
                       wheel_joint_rpy="${M_PI * -0.5} 0 0"
+                      is_steerable="true"
     />
     <xacro:scte_wheel link_name="rear_left_wheel"
-                      parent_link="base_link"
+                      parent_link="rear_axle"
                       wheel_radius="${wheel_radius}"
                       wheel_length="${wheel_length}"
-                      wheel_joint_origin="${scte_chassis_length * -0.63} ${drive_axle_length * 0.5} 0"
+                      wheel_joint_origin="0 0 ${drive_axle_length * 0.5}"
                       wheel_joint_rpy="${M_PI * -0.5} 0 0"
+                      is_steerable="false"
     />
     <xacro:scte_wheel link_name="rear_right_wheel"
-                      parent_link="base_link"
+                      parent_link="rear_axle"
                       wheel_radius="${wheel_radius}"
                       wheel_length="${wheel_length}"
-                      wheel_joint_origin="${scte_chassis_length * -0.63} ${drive_axle_length * -0.5} 0"
+                      wheel_joint_origin="0 0 ${drive_axle_length * -0.5}"
                       wheel_joint_rpy="${M_PI * -0.5} 0 0"
+                      is_steerable="false"
     />
 </robot>

File: src/models/scte_vehicle/scte_description/urdf/scte_wheel.xacro (robot description, xacro)
@@ -6,4 +6,5 @@
     wheel_joint_origin
     wheel_joint_rpy
+    is_steerable
     ">
             <gazebo reference="${link_name}">
@@ -14,5 +15,4 @@
                 <fdir1 value="1 0 0"/>
             </gazebo>
-            <!---->
             <link name="${link_name}_steer">
                 <inertial>
@@ -22,13 +22,21 @@
                 </inertial>
             </link>
-            <joint name="${link_name}_steer_TO_${parent_link}" type="revolute">
-                <parent link="${parent_link}" />
-                <child link="${link_name}_steer" />
-                <origin xyz="${wheel_joint_origin}" rpy="0 0 0" />
-                <axis xyz="0 0 1" />
-                <limit upper="0.6" lower="-0.6" effort="0.0" velocity="0.0" />
-            </joint>
-            <!---->
-            <!---->
+            <xacro:if value="${is_steerable == 1}">
+                <joint name="${link_name}_steer_TO_${parent_link}" type="revolute">
+                    <parent link="${parent_link}" />
+                    <child link="${link_name}_steer" />
+                    <origin xyz="${wheel_joint_origin}" rpy="${M_PI * 0.5} 0 0" />
+                    <axis xyz="0 0 1" />
+                    <limit upper="0.6" lower="-0.6" effort="0.0" velocity="0.0" />
+                </joint>
+            </xacro:if>
+            <xacro:if value="${is_steerable == 0}">
+                <joint name="${link_name}_steer_TO_${parent_link}" type="fixed">
+                    <parent link="${parent_link}" />
+                    <child link="${link_name}_steer" />
+                    <origin xyz="${wheel_joint_origin}" rpy="${M_PI * 0.5} 0 0" />
+                    <axis xyz="0 0 1" />
+                </joint>
+            </xacro:if>
             <link name="${link_name}">
                 <inertial>
@@ -65,5 +73,4 @@
                 </joint>
             </transmission>
-            <!---->
         </xacro:macro>
 </robot>

Commit message: improved the code that distinguishes the steerable and non-steerable wheels

File: src/models/scte_vehicle/scte_description/urdf/scte_chassis.xacro (robot description, xacro)
@@ -138,4 +138,5 @@
                       wheel_steer_joint_name="front_left_wheel_steer_TO_front_axle"
                       is_steerable="true"
+                      flip="1"
     />
     <xacro:scte_wheel link_name="front_right_wheel"
@@ -148,4 +149,5 @@
                       wheel_steer_joint_name="front_right_wheel_steer_TO_front_axle"
                       is_steerable="true"
+                      flip="-1"
     />
     <xacro:scte_wheel link_name="rear_left_wheel"
@@ -154,8 +156,9 @@
                       wheel_length="${wheel_length}"
                       wheel_joint_origin="0 0 ${drive_axle_length * 0.5}"
-                      wheel_joint_rpy="${M_PI * -0.5} 0 0"
+                      wheel_joint_rpy="0 0 0"
                       wheel_joint_name="rear_left_wheel_TO_rear_axle"
                       wheel_steer_joint_name="rear_left_wheel_steer_TO_rear_axle"
                       is_steerable="false"
+                      flip="1"
     />
     <xacro:scte_wheel link_name="rear_right_wheel"
@@ -164,9 +167,9 @@
                       wheel_length="${wheel_length}"
                       wheel_joint_origin="0 0 ${drive_axle_length * -0.5}"
-                      wheel_joint_rpy="${M_PI * -0.5} 0 0"
+                      wheel_joint_rpy="0 0 0"
                       wheel_joint_name="rear_right_wheel_TO_rear_axle"
                       wheel_steer_joint_name="rear_right_wheel_steer_TO_rear_axle"
                       is_steerable="false"
+                      flip="1"
     />
-    -->
 </robot>

File: src/models/scte_vehicle/scte_description/urdf/scte_wheel.xacro (robot description, xacro)
@@ -9,4 +9,5 @@
     wheel_steer_joint_name
     is_steerable
+    flip
     ">
             <gazebo reference="${link_name}">
@@ -19,34 +20,4 @@
             <xacro:property name="wheel_radius_sq" value="${wheel_radius * wheel_radius}"/>
             <xacro:property name="wheel_length_sq" value="${wheel_length * wheel_length}"/>
-            <link name="${link_name}_steer">
-                <inertial>
-                    <origin xyz="-0.02 -0.03 0" rpy="0 0 0"/>
-                    <!-- not sure why this has arbitrary mass and inertial values in the example source-->
-                    <mass value="${wheel_mass * 2}"/>
-                    <!--inertia ixx="${(2/5 * wheel_mass) * wheel_radius_sq}" ixy="0" ixz="0"
-                             iyy="${(2/5 * wheel_mass) * wheel_radius_sq}" iyz="0"
-                             izz="${(2/5 * wheel_mass) * wheel_radius_sq}"/-->
-                    <inertia  ixx="${(1/12 * wheel_mass * 2) * (3 * wheel_radius_sq + wheel_length_sq)}" ixy="0" ixz="0"
-                              iyy="${(1/12 * wheel_mass * 2) * (3 * wheel_radius_sq + wheel_length_sq)}" iyz="0"
-                              izz="${(1/2 * wheel_mass * 2) * wheel_radius_sq}" />
-                </inertial>
-            </link>
-            <xacro:if value="${is_steerable == 1}">
-                <joint name="${link_name}_steer_TO_${parent_link}" type="revolute">
-                    <parent link="${parent_link}" />
-                    <child link="${link_name}_steer" />
-                    <origin xyz="${wheel_joint_origin}" rpy="${M_PI * 0.5} 0 0" />
-                    <axis xyz="0 0 1" />
-                    <limit upper="0.6" lower="-0.6" effort="0.0" velocity="0.0" />
-                </joint>
-            </xacro:if>
-            <xacro:if value="${is_steerable == 0}">
-                <joint name="${wheel_steer_joint_name}" type="fixed">
-                    <parent link="${parent_link}" />
-                    <child link="${link_name}_steer" />
-                    <origin xyz="${wheel_joint_origin}" rpy="${M_PI * 0.5} 0 0" />
-                    <axis xyz="0 0 1" />
-                </joint>
-            </xacro:if>
             <link name="${link_name}">
                 <inertial>
@@ -69,20 +40,48 @@
             </link>
             <joint name='${wheel_joint_name}' type='continuous'>
-                <parent link="${link_name}_steer"/>
+                <xacro:if value="${is_steerable == 1}">
+                    <parent link="${link_name}_steer"/>
+                    <origin xyz="0 0 0" rpy="${wheel_joint_rpy}"/>
+                </xacro:if>
+                <xacro:if value="${is_steerable == 0}">
+                    <parent link="${parent_link}"/>
+                    <origin xyz="${wheel_joint_origin}" rpy="${wheel_joint_rpy}"/>
+                </xacro:if>
                 <child link="${link_name}"/>
-                <origin xyz="0 0 0" rpy="${wheel_joint_rpy}"/>
                 <axis xyz="0 0 1"/>
                 <dynamics damping="0.7"/>
                 <limit effort="1000.0" velocity="22.0"/>
             </joint>
-            <transmission name="${link_name}_transmission" type="SimpleTransmission">
+            <xacro:if value="${is_steerable == 1}">
+                <link name="${link_name}_steer">
+                    <inertial>
+                        <origin xyz="-0.02 ${-0.03 * flip} 0" rpy="0 0 0"/>
+                        <!-- not sure why this has arbitrary mass and inertial values in the example source-->
+                        <mass value="${wheel_mass * 2}"/>
+                        <!--inertia ixx="${(2/5 * wheel_mass) * wheel_radius_sq}" ixy="0" ixz="0"
+                                 iyy="${(2/5 * wheel_mass) * wheel_radius_sq}" iyz="0"
+                                 izz="${(2/5 * wheel_mass) * wheel_radius_sq}"/-->
+                        <inertia  ixx="${(1/12 * wheel_mass * 2) * (3 * wheel_radius_sq + wheel_length_sq)}" ixy="0" ixz="0"
+                                  iyy="${(1/12 * wheel_mass * 2) * (3 * wheel_radius_sq + wheel_length_sq)}" iyz="0"
+                                  izz="${(1/2 * wheel_mass * 2) * wheel_radius_sq}" />
+                    </inertial>
+                </link>
+                <joint name="${link_name}_steer_TO_${parent_link}" type="revolute">
+                    <parent link="${parent_link}" />
+                    <child link="${link_name}_steer" />
+                    <origin xyz="${wheel_joint_origin}" rpy="${M_PI * 0.5} 0 0" />
+                    <axis xyz="0 0 1" />
+                    <limit upper="0.6" lower="-0.6" effort="0.0" velocity="0.0" />
+                </joint>
+            </xacro:if>
+            <!--transmission name="${link_name}_transmission" type="SimpleTransmission">
                 <type>transmission_interface/SimpleTransmission</type>
                 <actuator name="${link_name}_motor">
                     <mechanicalReduction>1</mechanicalReduction>
                 </actuator>
-                <joint name="${link_name}_TO_${parent_link}">
+                <joint name="${wheel_joint_name}">
                     <hardwareInterface>hardware_interface/VelocityJointInterface</hardwareInterface>
                 </joint>
-            </transmission>
+            </transmission-->
         </xacro:macro>
 </robot>

Commit message: updated vehicle wheel base and other specs with real values. messed with steering ratio

File: src/models/scte_vehicle/scte_description/urdf/scte_chassis.xacro (robot description, xacro)
@@ -35,5 +35,5 @@
     <link name='base_footprint'/>
     <joint name="base_link_TO_base_footprint" type="fixed">
-        <origin xyz="0 0 ${scte_chassis_depth - wheel_radius}" rpy="0 0 0"/>
+        <origin xyz="${scte_chassis_length * 0.63} 0 ${wheel_radius - scte_chassis_depth - 0.0075}" rpy="0 0 0"/>
         <parent link="base_footprint"/>
         <child link="base_link"/>
@@ -96,4 +96,5 @@
                                      shock_tower_joint_rpy="0 0 0"
     />
+    <!--TODO get rid of some of these magic number parameters -->
     <xacro:include filename="$(find scte_description)/urdf/scte_front_bumper.xacro"/>
     <xacro:scte_front_bumper link_name="front_bumper"

File: src/models/scte_vehicle/scte_description/urdf/scte_drive_axle.xacro (robot description, xacro)
@@ -37,4 +37,7 @@
             <child link="${link_name}"/>
         </joint>
+        <gazebo reference="${link_name}">
+            <selfCollide>false</selfCollide>
+        </gazebo>
     </xacro:macro>
 </robot>

Commit message: fixed camera orientation

File: src/models/scte_vehicle/scte_description/urdf/scte_chassis.xacro (robot description, xacro)
@@ -220,5 +220,5 @@
         https://berndpfrommer.github.io/tagslam_web/visualization/
     -->
-    <!--TODO drowan_20210117_BUG: The cameras are mounted sideways. Need to fix camera link and/or optical link...
+    <!--TODO drowan_20210117_BUG: The cameras are mounted sideways. Need to fix camera link and/or optical link...-->
     <!---->
     <xacro:logitech_c270_camera parent_link="camera_rig_bar" camera_link="driver_side_camera" joint_xyz="0.0 0.05 ${0.025 * 0.5}" joint_rpy="0 0 0"/>

File: src/sensors/logitech_c270_camera/urdf/logitech_c270.xacro (robot description, xacro)
@@ -4,5 +4,5 @@
     <!--https://answers.ros.org/question/331432/pass-parameters-of-xacro-file-in-another-xacro-file/-->
     <xacro:macro name="logitech_c270_camera" params="parent_link camera_link joint_xyz joint_rpy">
-        <link name='${camera_link}'>
+        <link name='${camera_link}_body'>
             <inertial>
                 <mass value="1.0"/>
@@ -31,12 +31,12 @@
             </collision>
         </link>
-        <joint name="${camera_link}_base_JOINT_${parent_link}_link" type="fixed">
+        <joint name="${camera_link}_TO_${parent_link}" type="fixed">
             <origin xyz="${joint_xyz}" rpy="${joint_rpy}"/>
             <parent link="${parent_link}"/>
-            <child link="${camera_link}"/>
+            <child link="${camera_link}_body"/>
         </joint>
-        <link name="${camera_link}_optical">
+        <link name="${camera_link}_base">
             <visual name='visual'>
-                <origin xyz="0 0 0" rpy="0 0 0"/>
+                <origin xyz="0.003 0 0" rpy="0 0 0"/>
                 <geometry>
                     <box size="0.01 0.01 0.01"/>
@@ -45,5 +45,5 @@
             </visual>
             <collision name='collision'>
-                <origin xyz="0 0 0" rpy="0 0 0"/>
+                <origin xyz="0.003 0 0" rpy="0 0 0"/>
                 <geometry>
                     <box size="0.01 0.01 0.01"/>
@@ -51,7 +51,13 @@
             </collision>
         </link>
-        <joint name="${camera_link}_base_optical_JOINT_${camera_link}_link" type="fixed">
-            <origin xyz="0.03 0.015 0" rpy="${M_PI/-2} 0 ${M_PI/-2}"/>
-            <parent link="${camera_link}"/>
+        <joint name="${camera_link}_base_TO_${camera_link}_body" type="fixed">
+            <origin xyz="0.03 0.015 0.0" rpy="0 0 0"/> <!-- ${M_PI/-2} 0 ${M_PI/-2} -->
+            <parent link="${camera_link}_body"/>
+            <child link="${camera_link}_base"/>
+        </joint>
+        <link name="${camera_link}_optical"/>
+        <joint name="${camera_link}_optical_TO_${camera_link}_base" type="fixed">
+            <origin xyz="0 0 0" rpy="${-pi/2} 0 ${-pi/2}"/>
+            <parent link="${camera_link}_base"/>
             <child link="${camera_link}_optical"/>
         </joint>

Commit message: copied example from the ros controllers folder. doesn't seem to work either

File: src/models/scte_vehicle/scte_description/urdf/scte_chassis.xacro (robot description, xacro)
@@ -81,4 +81,26 @@
         <child link="scte_chassis"/>
     </joint>
+    <!-- TODO DEBUG drowan_20210119: ackermann link/joints -->
+    <link name="rear_wheel_linkX">
+        <collision>
+            <origin rpy="${pi/2} 0 0" xyz="0 0 0"/>
+            <geometry>
+                <cylinder length="1" radius="0.5"/>
+            </geometry>
+        </collision>
+    </link>
+    <joint name="rear_wheel_joint" type="fixed">
+        <axis xyz="0 1 0"/>
+        <parent link="rear_axle"/>
+        <child link="rear_wheel_linkX"/>
+        <origin xyz="0 0 0"/>
+    </joint>
+    <link name="front_steer_linkX"/>
+    <joint name="front_steer_joint" type="continuous">
+        <axis xyz="0 1 0"/>
+        <parent link="front_axle"/>
+        <child link="front_steer_linkX"/>
+        <origin xyz="0 0 0"/>
+    </joint>
     <!---->
     <xacro:include filename="$(find scte_description)/urdf/scte_diff_and_shock_tower.xacro"/>
