Commit message: using the ackermann steer bot example to get scte bot working

File: src/models/scte_vehicle/scte_description/urdf/scte_chassis.xacro (robot description, xacro)
@@ -15,5 +15,5 @@
     <xacro:arg name="pub_tf" default="false"/>
     <xacro:property name="M_PI" value="3.14159265358979323846264338327950288"/>
-    <xacro:include filename="$(find scte_description)/urdf/scte.gazebo" />
+    <xacro:include filename="plugins/scte_plugins.gazebo" />
     <xacro:include filename="$(find scte_description)/urdf/materials.xacro" />
     <xacro:include filename="$(find scte_description)/urdf/macros.xacro" />
@@ -32,6 +32,14 @@
     <!--Wheel Properties-->
     <xacro:property name="wheel_mass" value="0.3"/>
-    <xacro:property name="wheel_radius" value="0.0525"/>
-    <xacro:property name="wheel_length" value="0.045"/>
+    <!--xacro:property name="wheel_radius" value="0.0525"/-->
+    <!--xacro:property name="wheel_length" value="0.045"/-->
+    <xacro:property name="deg_to_rad" value="0.01745329251994329577"/>
+    <!-- Constants for robot dimensions -->
+    <xacro:property name="wheel_radius" value="0.0525" /> <!-- Link 1 -->
+    <xacro:property name="wheel_thickness" value="0.045" /> <!-- Link 2 -->
+    <xacro:property name="wheel_length" value="0.47" /> <!-- separation between wheels? -->
+    <xacro:property name="wheel_width" value="${0.20 - wheel_thickness}" /> <!-- separation between wheels? -->
+    <xacro:property name="axel_offset" value="0.05" /> <!-- Space btw top of beam and the each joint -->
+    <xacro:property name="steer_offset" value="0.02" /> <!-- Link 1 -->
     <xacro:property name="shock_tower_height" value="0.105"/>
     <xacro:property name="shock_tower_width" value="0.14"/>
@@ -81,26 +89,4 @@
         <child link="scte_chassis"/>
     </joint>
-    <!-- TODO DEBUG drowan_20210119: ackermann link/joints -->
-    <link name="rear_wheel_linkX">
-        <collision>
-            <origin rpy="${pi/2} 0 0" xyz="0 0 0"/>
-            <geometry>
-                <cylinder length="1" radius="0.5"/>
-            </geometry>
-        </collision>
-    </link>
-    <joint name="rear_wheel_joint" type="fixed">
-        <axis xyz="0 1 0"/>
-        <parent link="rear_axle"/>
-        <child link="rear_wheel_linkX"/>
-        <origin xyz="0 0 0"/>
-    </joint>
-    <link name="front_steer_linkX"/>
-    <joint name="front_steer_joint" type="continuous">
-        <axis xyz="0 1 0"/>
-        <parent link="front_axle"/>
-        <child link="front_steer_linkX"/>
-        <origin xyz="0 0 0"/>
-    </joint>
     <!---->
     <xacro:include filename="$(find scte_description)/urdf/scte_diff_and_shock_tower.xacro"/>
@@ -156,4 +142,5 @@
                            drive_axle_joint_rpy="${M_PI * -0.5} 0 0"
     />
+    <!-- Wheel macros for audio bot implementation
     <xacro:include filename="$(find scte_description)/urdf/scte_wheel.xacro"/>
     <xacro:scte_wheel link_name="front_left_wheel"
@@ -201,4 +188,29 @@
                       flip="1"
     />
+    -->
+    <xacro:include filename="$(find scte_description)/urdf/scte_wheel.xacro"/>
+    <!-- joints for ackermann_steering_controller -->
+    <xacro:front_steer name="front" parent="base" radius="${wheel_radius}" thickness="${wheel_thickness}"
+                       length="${wheel_length}" width="${wheel_width}" axel_offset="${axel_offset}" steer_height="${wheel_radius+steer_offset}">
+        <origin xyz="${wheel_length/2-axel_offset} 0 0" rpy="${-90 * deg_to_rad} 0 0"/>
+    </xacro:front_steer>
+    <xacro:rear_wheel name="rear" parent="base" radius="${wheel_radius}" thickness="${wheel_thickness}">
+        <origin xyz="${-wheel_length/2+axel_offset} 0 0" rpy="${-90 * deg_to_rad} 0 0"/>
+    </xacro:rear_wheel>
+    <!-- Wheels -->
+    <xacro:front_wheel_lr name="front_right" parent="base" radius="${wheel_radius}" thickness="${wheel_thickness}"
+                          length="${wheel_length}" width="${wheel_width}" axel_offset="${axel_offset}" right_left="1" steer_height="${wheel_radius+steer_offset}">
+        <origin xyz="${wheel_length/2-axel_offset} ${wheel_width/2+axel_offset} 0" rpy="${-90 * deg_to_rad} 0 0"/>
+    </xacro:front_wheel_lr>
+    <xacro:front_wheel_lr name="front_left" parent="base" radius="${wheel_radius}" thickness="${wheel_thickness}"
+                          length="${wheel_length}" width="${wheel_width}" axel_offset="${axel_offset}" right_left="-1" steer_height="${wheel_radius+steer_offset}">
+        <origin xyz="${wheel_length/2-axel_offset} ${-wheel_width/2-axel_offset} ${scte_chassis_depth * -0.5}" rpy="${-90 * deg_to_rad} 0 0"/>
+    </xacro:front_wheel_lr>
+    <xacro:rear_wheel_lr name="rear_right" parent="base" radius="${wheel_radius}" thickness="${wheel_thickness}">
+        <origin xyz="${-wheel_length/2+axel_offset} ${wheel_width/2+axel_offset} ${scte_chassis_depth * -0.5}" rpy="${-90 * deg_to_rad} 0 0"/>
+    </xacro:rear_wheel_lr>
+    <xacro:rear_wheel_lr name="rear_left" parent="base" radius="${wheel_radius}" thickness="${wheel_thickness}">
+        <origin xyz="${-wheel_length/2+axel_offset} ${-wheel_width/2-axel_offset} ${scte_chassis_depth * -0.5}" rpy="${-90 * deg_to_rad} 0 0"/>
+    </xacro:rear_wheel_lr>
     <xacro:mounting_bar link_name="driver_mounting_bar"
                         parent_link="front_diff_tower"

File: src/models/scte_vehicle/scte_description/urdf/scte_wheel.xacro (robot description, xacro)
@@ -1,76 +1,190 @@
 <?xml version="1.0"?>
-<robot name="sctebot" xmlns:xacro="http://www.ros.org/wiki/xacro">
-    <xacro:macro name="scte_wheel" params="link_name parent_link
-    wheel_radius
-    wheel_length
-    wheel_joint_origin
-    wheel_joint_rpy
-    wheel_joint_name
-    wheel_steer_joint_name
-    is_steerable
-    flip
-    ">
-            <xacro:property name="wheel_friction" value="1.75" />
-            <xacro:property name="wheel_radius_sq" value="${wheel_radius * wheel_radius}"/>
-            <xacro:property name="wheel_length_sq" value="${wheel_length * wheel_length}"/>
-            <link name="${link_name}">
-                <inertial>
-                    <mass value="${wheel_mass}"/>
-                    <inertia  ixx="${(1/12 * wheel_mass) * (3 * wheel_radius_sq + wheel_length_sq)}" ixy="0" ixz="0"
-                              iyy="${(1/12 * wheel_mass) * (3 * wheel_radius_sq + wheel_length_sq)}" iyz="0"
-                              izz="${(1/2 * wheel_mass) * wheel_radius_sq}" />
-                </inertial>
-                <visual name='visual'>
-                    <geometry>
-                        <cylinder radius="${wheel_radius}" length="${wheel_length}"/>
-                    </geometry>
-                    <material name="green"/>
-                </visual>
-                <collision name='collision'>
-                    <geometry>
-                        <cylinder radius="${wheel_radius}" length="${wheel_length}"/>
-                    </geometry>
-                </collision>
-            </link>
-            <joint name='${wheel_joint_name}' type='continuous'>
-                <xacro:if value="${is_steerable == 1}">
-                    <parent link="${link_name}_steer"/>
-                    <origin xyz="0 0 0" rpy="${wheel_joint_rpy}"/>
-                </xacro:if>
-                <xacro:if value="${is_steerable == 0}">
-                    <parent link="${parent_link}"/>
-                    <origin xyz="${wheel_joint_origin}" rpy="${wheel_joint_rpy}"/>
-                </xacro:if>
-                <child link="${link_name}"/>
-                <axis xyz="0 0 1"/>
-                <dynamics damping="0.7"/>
-                <limit effort="1000.0" velocity="22.0"/>
-                <gazebo reference="${wheel_joint_name}">
-                    <mu1>${wheel_friction}</mu1>
-                    <mu2>${wheel_friction}</mu2>
-                </gazebo>
-            </joint>
-            <xacro:if value="${is_steerable == 1}">
-                <link name="${link_name}_steer">
-                    <inertial>
-                        <origin xyz="-0.02 ${-0.03 * flip} 0" rpy="0 0 0"/>
-                        <!-- not sure why this has arbitrary mass and inertial values in the example source-->
-                        <mass value="${wheel_mass * 2}"/>
-                        <!--inertia ixx="${(2/5 * wheel_mass) * wheel_radius_sq}" ixy="0" ixz="0"
-                                 iyy="${(2/5 * wheel_mass) * wheel_radius_sq}" iyz="0"
-                                 izz="${(2/5 * wheel_mass) * wheel_radius_sq}"/-->
-                        <inertia  ixx="${(1/12 * wheel_mass * 2) * (3 * wheel_radius_sq + wheel_length_sq)}" ixy="0" ixz="0"
-                                  iyy="${(1/12 * wheel_mass * 2) * (3 * wheel_radius_sq + wheel_length_sq)}" iyz="0"
-                                  izz="${(1/2 * wheel_mass * 2) * wheel_radius_sq}" />
-                    </inertial>
-                </link>
-                <joint name="${link_name}_steer_TO_${parent_link}" type="revolute">
-                    <parent link="${parent_link}" />
-                    <child link="${link_name}_steer" />
-                    <origin xyz="${wheel_joint_origin}" rpy="${M_PI * 0.5} 0 0" />
-                    <axis xyz="0 0 1" />
-                    <limit upper="0.6" lower="-0.6" effort="0.0" velocity="0.0" />
-                </joint>
-            </xacro:if>
-        </xacro:macro>
+<robot xmlns:xacro="http://www.ros.org/wiki/xacro">
+    <!-- Copied from ackermann_steering_bot example -->
+    <xacro:property name="steer_radius" value="0.05" /> <!-- Link 1 -->
+    <xacro:property name="steer_thickness" value="0.02" /> <!-- Link 1 -->
+    <xacro:property name="steer_effort"   value="10.0"/>
+    <xacro:property name="steer_velocity" value="5.0"/>
+    <xacro:macro name="front_steer" params="name parent radius thickness length width axel_offset steer_height *origin">
+        <link name="${name}_steer_link">
+            <inertial>
+                <origin xyz="0 0 0" rpy="0 0 0"/>
+                <mass value="1"/>
+                <inertia ixx="0.2" ixy="0" ixz="0" iyy="0.2" iyz="0" izz="0.2"/>
+            </inertial>
+            <visual>
+                <origin xyz="0 0 0" rpy="0 0 0"/>
+                <geometry>
+                    <cylinder radius="${steer_radius}" length="${steer_thickness}"/>
+                </geometry>
+            </visual>
+            <collision>
+                <origin xyz="0 0 0" rpy="0 0 0"/>
+                <geometry>
+                    <cylinder radius="${steer_radius}" length="${steer_thickness}"/>
+                </geometry>
+            </collision>
+        </link>
+        <joint name="${name}_steer_joint" type="revolute">
+            <parent link="${parent}_link"/>
+            <child link="${name}_steer_link"/>
+            <origin xyz="${length/2-axel_offset} 0 ${steer_height}" rpy="0 0 0"/>
+            <axis xyz="0 0 1"/>
+            <limit effort="${steer_effort}"
+                   lower="${-180.0 * deg_to_rad}" upper="${180.0 * deg_to_rad}"
+                   velocity="${steer_velocity}"/>
+        </joint>
+        <gazebo reference="${name}_steer_link">
+            <material>Gazebo/Yellow</material>
+        </gazebo>
+    </xacro:macro>
+    <xacro:macro name="front_wheel_lr" params="name parent radius thickness length width axel_offset right_left steer_height *origin">
+        <link name="${name}_steer_link">
+            <inertial>
+                <origin xyz="0 0 0" rpy="0 0 0"/>
+                <mass value="1"/>
+                <inertia ixx="0.2" ixy="0" ixz="0" iyy="0.2" iyz="0" izz="0.2"/>
+            </inertial>
+            <visual>
+                <origin xyz="0 0 0" rpy="0 0 0"/>
+                <geometry>
+                    <cylinder radius="${steer_radius}" length="${steer_thickness}"/>
+                </geometry>
+            </visual>
+            <collision>
+                <origin xyz="0 0 0" rpy="0 0 0"/>
+                <geometry>
+                    <cylinder radius="${steer_radius}" length="${steer_thickness}"/>
+                </geometry>
+            </collision>
+        </link>
+        <joint name="${name}_steer_joint" type="revolute">
+            <parent link="${parent}_link"/>
+            <child link="${name}_steer_link"/>
+            <origin xyz="${length/2-axel_offset} ${right_left*(width/2+axel_offset)} ${steer_height}" rpy="0 0 0"/>
+            <!--xacro:insert_block name="origin"/-->
+            <axis xyz="0 0 1"/>
+            <limit effort="${steer_effort}"
+                   lower="${-180.0 * deg_to_rad}" upper="${180.0 * deg_to_rad}"
+                   velocity="${steer_velocity}"/>
+        </joint>
+        <link name="${name}_wheel_link">
+            <inertial>
+                <origin xyz="0 0 0" rpy="0 0 0"/>
+                <mass value="1"/>
+                <inertia ixx="0.2" ixy="0" ixz="0" iyy="0.2" iyz="0" izz="0.2"/>
+            </inertial>
+            <visual>
+                <origin xyz="0 0 0" rpy="0 0 0"/>
+                <geometry>
+                    <cylinder radius="${wheel_radius}" length="${thickness}"/>
+                </geometry>
+            </visual>
+            <collision>
+                <origin xyz="0 0 0" rpy="0 0 0"/>
+                <geometry>
+                    <cylinder radius="${wheel_radius}" length="${thickness}"/>
+                </geometry>
+            </collision>
+        </link>
+        <joint name="${name}_wheel_joint" type="continuous">
+            <parent link="${name}_steer_link"/>
+            <child link="${name}_wheel_link"/>
+            <origin xyz="0 0 ${-steer_height}" rpy="${-90 * deg_to_rad} 0 0"/>
+            <axis xyz="0 0 1"/>
+        </joint>
+        <!-- Transmission is important to link the joints and the controller -->
+        <transmission name="${name}_steer_joint_trans" type="SimpleTransmission">
+            <actuator name="${name}_steer_joint_motor"/>
+            <joint name="${name}_steer_joint"/>
+            <mechanicalReduction>1</mechanicalReduction>
+            <motorTorqueConstant>1</motorTorqueConstant>
+        </transmission>
+        <transmission name="${name}_wheel_joint_trans" type="SimpleTransmission">
+            <actuator name="${name}_wheel_joint_motor"/>
+            <joint name="${name}_wheel_joint"/>
+            <mechanicalReduction>1</mechanicalReduction>
+            <motorTorqueConstant>1</motorTorqueConstant>
+        </transmission>
+        <gazebo reference="${name}_steer_link">
+            <material>Gazebo/Blue</material>
+        </gazebo>
+        <gazebo reference="${name}_wheel_link">
+            <material>Gazebo/Red</material>
+        </gazebo>
+    </xacro:macro>
+    <xacro:macro name="rear_wheel" params="name parent radius thickness *origin">
+        <link name="${name}_wheel_link">
+            <inertial>
+                <origin xyz="0 0 0" rpy="0 0 0"/>
+                <mass value="1"/>
+                <inertia ixx="0.2" ixy="0" ixz="0" iyy="0.2" iyz="0" izz="0.2"/>
+            </inertial>
+            <visual>
+                <origin xyz="0 0 0" rpy="0 0 0"/>
+                <geometry>
+                    <cylinder radius="${wheel_radius}" length="${thickness}"/>
+                </geometry>
+            </visual>
+            <collision>
+                <origin xyz="0 0 0" rpy="0 0 0"/>
+                <geometry>
+                    <cylinder radius="${wheel_radius}" length="${thickness}"/>
+                </geometry>
+            </collision>
+        </link>
+        <joint name="${name}_wheel_joint" type="continuous">
+            <parent link="${parent}_link"/>
+            <child link="${name}_wheel_link"/>
+            <xacro:insert_block name="origin"/>
+            <axis xyz="0 0 1"/>
+        </joint>
+        <!-- Transmission is important to link the joints and the controller -->
+        <transmission name="${name}_wheel_joint_trans" type="SimpleTransmission">
+            <actuator name="${name}_wheel_joint_motor"/>
+            <joint name="${name}_wheel_joint"/>
+            <mechanicalReduction>1</mechanicalReduction>
+            <motorTorqueConstant>1</motorTorqueConstant>
+        </transmission>
+        <gazebo reference="${name}_wheel_link">
+            <material>Gazebo/Yellow</material>
+        </gazebo>
+    </xacro:macro>
+    <xacro:macro name="rear_wheel_lr" params="name parent radius thickness *origin">
+        <link name="${name}_wheel_link">
+            <inertial>
+                <origin xyz="0 0 0" rpy="0 0 0"/>
+                <mass value="1"/>
+                <inertia ixx="0.2" ixy="0" ixz="0" iyy="0.2" iyz="0" izz="0.2"/>
+            </inertial>
+            <visual>
+                <origin xyz="0 0 0" rpy="0 0 0"/>
+                <geometry>
+                    <cylinder radius="${wheel_radius}" length="${thickness}"/>
+                </geometry>
+            </visual>
+            <collision>
+                <origin xyz="0 0 0" rpy="0 0 0"/>
+                <geometry>
+                    <cylinder radius="${wheel_radius}" length="${thickness}"/>
+                </geometry>
+            </collision>
+        </link>
+        <joint name="${name}_wheel_joint" type="continuous">
+            <parent link="${parent}_link"/>
+            <child link="${name}_wheel_link"/>
+            <xacro:insert_block name="origin"/>
+            <axis xyz="0 0 1"/>
+        </joint>
+        <!-- Transmission is important to link the joints and the controller -->
+        <transmission name="${name}_wheel_joint_trans" type="SimpleTransmission">
+            <actuator name="${name}_wheel_joint_motor"/>
+            <joint name="${name}_wheel_joint"/>
+            <mechanicalReduction>1</mechanicalReduction>
+            <motorTorqueConstant>1</motorTorqueConstant>
+        </transmission>
+        <gazebo reference="${name}_wheel_link">
+            <material>Gazebo/Red</material>
+        </gazebo>
+    </xacro:macro>
 </robot>
