Commit message: updated the xacro transmission components to work with noetic. Still need to figure out how to plug into steer_bot plugin. This may be a HW only plugin, not sure.

File: src/models/scte_vehicle/scte_description/urdf/scte_chassis.xacro (robot description, xacro)
@@ -201,15 +201,15 @@
     <!-- Wheels -->
     <xacro:front_wheel_lr name="front_right" parent="base" radius="${wheel_radius}" thickness="${wheel_thickness}"
-                          length="${wheel_length}" width="${wheel_width}" axel_offset="${axel_offset}" right_left="1" steer_height="${wheel_radius+steer_offset}">
+                          length="${wheel_length}" width="${wheel_width}" axel_offset="${axel_offset}" right_left="-1" steer_height="${wheel_radius+steer_offset}">
         <origin xyz="${wheel_length/2-axel_offset} ${wheel_width/2+axel_offset} 0" rpy="${-90 * deg_to_rad} 0 0"/>
     </xacro:front_wheel_lr>
     <xacro:front_wheel_lr name="front_left" parent="base" radius="${wheel_radius}" thickness="${wheel_thickness}"
-                          length="${wheel_length}" width="${wheel_width}" axel_offset="${axel_offset}" right_left="-1" steer_height="${wheel_radius+steer_offset}">
+                          length="${wheel_length}" width="${wheel_width}" axel_offset="${axel_offset}" right_left="1" steer_height="${wheel_radius+steer_offset}">
         <origin xyz="${wheel_length/2-axel_offset} ${-wheel_width/2-axel_offset} ${scte_chassis_depth * -0.5}" rpy="${-90 * deg_to_rad} 0 0"/>
     </xacro:front_wheel_lr>
-    <xacro:rear_wheel_lr name="rear_right" parent="base" radius="${wheel_radius}" thickness="${wheel_thickness}">
+    <xacro:rear_wheel_lr name="rear_left" parent="base" radius="${wheel_radius}" thickness="${wheel_thickness}">
         <origin xyz="${-wheel_length/2+axel_offset} ${wheel_width/2+axel_offset} ${scte_chassis_depth * -0.5}" rpy="${-90 * deg_to_rad} 0 0"/>
     </xacro:rear_wheel_lr>
-    <xacro:rear_wheel_lr name="rear_left" parent="base" radius="${wheel_radius}" thickness="${wheel_thickness}">
+    <xacro:rear_wheel_lr name="rear_right" parent="base" radius="${wheel_radius}" thickness="${wheel_thickness}">
         <origin xyz="${-wheel_length/2+axel_offset} ${-wheel_width/2-axel_offset} ${scte_chassis_depth * -0.5}" rpy="${-90 * deg_to_rad} 0 0"/>
     </xacro:rear_wheel_lr>

File: src/models/scte_vehicle/scte_description/urdf/scte_wheel.xacro (robot description, xacro)
@@ -95,4 +95,5 @@
         </joint>
         <!-- Transmission is important to link the joints and the controller -->
+        <!--
         <transmission name="${name}_steer_joint_trans">
             <type>SimpleTransmission</type>
@@ -109,4 +110,25 @@
             <motorTorqueConstant>1</motorTorqueConstant>
         </transmission>
+        -->
+        <transmission name="${name}_steer_joint_trans">
+            <type>transmission_interface/SimpleTransmission</type>
+            <joint name="${name}_steer_joint">
+                <hardwareInterface>hardware_interface/EffortJointInterface</hardwareInterface>
+            </joint>
+            <actuator name="${name}_steer_joint_motor">
+                <hardwareInterface>hardware_interface/EffortJointInterface</hardwareInterface>
+                <mechanicalReduction>1</mechanicalReduction>
+            </actuator>
+        </transmission>
+        <transmission name="${name}_wheel_joint_trans">
+            <type>transmission_interface/SimpleTransmission</type>
+            <joint name="${name}_wheel_joint">
+                <hardwareInterface>hardware_interface/EffortJointInterface</hardwareInterface>
+            </joint>
+            <actuator name="${name}_wheel_joint_motor">
+                <hardwareInterface>hardware_interface/EffortJointInterface</hardwareInterface>
+                <mechanicalReduction>1</mechanicalReduction>
+            </actuator>
+        </transmission>
         <gazebo reference="${name}_steer_link">
             <material>Gazebo/Blue</material>
@@ -143,4 +165,5 @@
         </joint>
         <!-- Transmission is important to link the joints and the controller -->
+        <!--
         <transmission name="${name}_wheel_joint_trans">
             <type>SimpleTransmission</type>
@@ -150,4 +173,15 @@
             <motorTorqueConstant>1</motorTorqueConstant>
         </transmission>
+        -->
+        <transmission name="${name}_wheel_joint_trans">
+            <type>transmission_interface/SimpleTransmission</type>
+            <joint name="${name}_wheel_joint">
+                <hardwareInterface>hardware_interface/EffortJointInterface</hardwareInterface>
+            </joint>
+            <actuator name="${name}_wheel_joint_motor">
+                <hardwareInterface>hardware_interface/EffortJointInterface</hardwareInterface>
+                <mechanicalReduction>1</mechanicalReduction>
+            </actuator>
+        </transmission>
         <gazebo reference="${name}_wheel_link">
             <material>Gazebo/Yellow</material>
@@ -179,6 +213,8 @@
             <xacro:insert_block name="origin"/>
             <axis xyz="0 0 1"/>
+            <dynamics damping="0.7"/>
         </joint>
         <!-- Transmission is important to link the joints and the controller -->
+        <!--
         <transmission name="${name}_wheel_joint_trans">
             <type>SimpleTransmission</type>
@@ -188,4 +224,15 @@
             <motorTorqueConstant>1</motorTorqueConstant>
         </transmission>
+        -->
+        <transmission name="${name}_wheel_joint_trans">
+            <type>transmission_interface/SimpleTransmission</type>
+            <joint name="${name}_wheel_joint">
+                <hardwareInterface>hardware_interface/EffortJointInterface</hardwareInterface>
+            </joint>
+            <actuator name="${name}_wheel_joint_motor">
+                <hardwareInterface>hardware_interface/EffortJointInterface</hardwareInterface>
+                <mechanicalReduction>1</mechanicalReduction>
+            </actuator>
+        </transmission>
         <gazebo reference="${name}_wheel_link">
             <material>Gazebo/Red</material>
