Commit message: commit prior to trying a clean slate with the model

File: src/models/scte_vehicle/scte_description/urdf/scte_chassis.xacro (robot description, xacro)
@@ -9,4 +9,13 @@
 http://wiki.ros.org/urdf/XML/joint#Elements
 -->
+<!--
+Geometry:
+The Ackermann steering controllers require the longitudinal
+separation between the front and back wheel axes and the
+lateral separation between the left and right front steering axes.
+For this model:
+wheel_separation_h = base_length - 2 * axle_offset = 0.4
+wheel_separation_w = base_width  + 2 * axle_offset = 0.4
+-->
 <!--Gazebo does not seem to like capital letters in the robot namespace-->
 <robot name="sctebot" xmlns:xacro="http://www.ros.org/wiki/xacro">
@@ -16,5 +25,4 @@
     <xacro:property name="M_PI" value="3.14159265358979323846264338327950288"/>
     <xacro:include filename="$(find scte_description)/urdf/plugins/scte_plugins.gazebo" />
-    <!--xacro:include filename="$(find scte_description)/urdf/plugins/scte_audi_bot_plugin.gazebo"/-->
     <xacro:include filename="plugins/scte_sensors.gazebo" />
     <xacro:include filename="$(find scte_description)/urdf/materials.xacro" />
@@ -34,13 +42,11 @@
     <!--Wheel Properties-->
     <xacro:property name="wheel_mass" value="0.3"/>
-    <!--xacro:property name="wheel_radius" value="0.0525"/-->
-    <!--xacro:property name="wheel_length" value="0.045"/-->
     <xacro:property name="deg_to_rad" value="0.01745329251994329577"/>
     <!-- Constants for robot dimensions -->
+    <xacro:property name="wheel_base" value="0.337"/>
+    <xacro:property name="wheel_track" value="0.251"/>
     <xacro:property name="wheel_radius" value="0.0525" /> <!-- Link 1 -->
     <xacro:property name="wheel_thickness" value="0.045" /> <!-- Link 2 -->
-    <xacro:property name="wheel_length" value="0.47" /> <!-- separation between wheels? -->
-    <xacro:property name="wheel_width" value="${0.20 - wheel_thickness}" /> <!-- separation between wheels? -->
-    <xacro:property name="axel_offset" value="0.05" /> <!-- Space btw top of beam and the each joint -->
+    <xacro:property name="axel_offset" value="0.05" /> <!-- Space between top of beam and the each joint -->
     <xacro:property name="steer_offset" value="0.02" /> <!-- Link 1 -->
     <xacro:property name="shock_tower_height" value="0.105"/>
@@ -93,145 +99,198 @@
     <!---->
     <xacro:include filename="$(find scte_description)/urdf/scte_diff_and_shock_tower.xacro"/>
-    <xacro:scte_diff_and_shock_tower link_name="front_diff_tower"
-                                parent_link="scte_chassis"
-                                diff_joint_xyz="${scte_chassis_length * 0.63} 0 0"
-                                diff_joint_rpy="0 0 0"
-                                diff_plate_size="0.07 0.07 ${scte_chassis_depth}"
-                                shock_tower_size="0.015 ${shock_tower_width} ${shock_tower_height}"
-                                shock_tower_joint_origin="0 0 ${shock_tower_height * 0.5}"
-                                shock_tower_joint_rpy="0 0 0"
-    />
-    <xacro:scte_diff_and_shock_tower link_name="rear_diff_tower"
-                                     parent_link="scte_chassis"
-                                     diff_joint_xyz="${scte_chassis_length * -0.63} 0 0"
-                                     diff_joint_rpy="0 0 0"
-                                     diff_plate_size="0.07 0.07 ${scte_chassis_depth}"
-                                     shock_tower_size="0.015 ${shock_tower_width} ${shock_tower_height}"
-                                     shock_tower_joint_origin="0 0 ${shock_tower_height * 0.5}"
-                                     shock_tower_joint_rpy="0 0 0"
+    <xacro:scte_diff_and_shock_tower
+        link_name="front_diff_tower"
+        parent_link="scte_chassis"
+        diff_joint_xyz="${scte_chassis_length * 0.63} 0 0"
+        diff_joint_rpy="0 0 0"
+        diff_plate_size="0.07 0.07 ${scte_chassis_depth}"
+        shock_tower_size="0.015 ${shock_tower_width} ${shock_tower_height}"
+        shock_tower_joint_origin="0 0 ${shock_tower_height * 0.5}"
+        shock_tower_joint_rpy="0 0 0"
+    />
+    <xacro:scte_diff_and_shock_tower
+        link_name="rear_diff_tower"
+        parent_link="scte_chassis"
+        diff_joint_xyz="${scte_chassis_length * -0.63} 0 0"
+        diff_joint_rpy="0 0 0"
+        diff_plate_size="0.07 0.07 ${scte_chassis_depth}"
+        shock_tower_size="0.015 ${shock_tower_width} ${shock_tower_height}"
+        shock_tower_joint_origin="0 0 ${shock_tower_height * 0.5}"
+        shock_tower_joint_rpy="0 0 0"
     />
     <!--TODO get rid of some of these magic number parameters -->
     <xacro:include filename="$(find scte_description)/urdf/scte_front_bumper.xacro"/>
-    <xacro:scte_front_bumper link_name="front_bumper"
-                             parent_link="front_diff_tower"
-                             front_skid_plate_size="0.07 0.07 ${scte_chassis_depth}"
-                             front_skid_plate_joint_xyz="${0.07} 0 ${0.07 * 0.30}"
-                             front_skid_plate_joint_rpy="0 ${M_PI/-6}  0"
-                             front_bumper_size="0.01 0.175 0.05"
+    <xacro:scte_front_bumper
+        link_name="front_bumper"
+        parent_link="front_diff_tower"
+        front_skid_plate_size="0.07 0.07 ${scte_chassis_depth}"
+        front_skid_plate_joint_xyz="${0.07} 0 ${0.07 * 0.30}"
+        front_skid_plate_joint_rpy="0 ${M_PI/-6}  0"
+        front_bumper_size="0.01 0.175 0.05"
     />
     <xacro:include filename="$(find scte_description)/urdf/scte_rear_bumper.xacro"/>
-    <xacro:scte_rear_bumper link_name="rear_bumper"
-                            parent_link="rear_diff_tower"
-                            rear_bumper_size="0.01 0.255 0.05"
-                            rear_bumper_mount_size="0.09 0.05 0.05"
-                            rear_bumper_mount_joint_xyz="${0.09 * -0.6} 0 ${shock_tower_height * 0.5}"
-                            rear_bumper_mount_joint_rpy="0 0 0"
+    <xacro:scte_rear_bumper
+        link_name="rear_bumper"
+        parent_link="rear_diff_tower"
+        rear_bumper_size="0.01 0.255 0.05"
+        rear_bumper_mount_size="0.09 0.05 0.05"
+        rear_bumper_mount_joint_xyz="${0.09 * -0.6} 0 ${shock_tower_height * 0.5}"
+        rear_bumper_mount_joint_rpy="0 0 0"
     />
     <xacro:include filename="$(find scte_description)/urdf/scte_drive_axle.xacro"/>
-    <xacro:scte_drive_axle link_name="front_axle"
-                     parent_link="front_diff_tower"
-                     drive_axle_radius="${drive_axle_radius}"
-                     drive_axle_length="${drive_axle_length}"
-                     drive_axle_joint_xyz="0 0 ${0.03 * 0.5}"
-                     drive_axle_joint_rpy="${M_PI * -0.5} 0 0"
-    />
-    <xacro:include filename="$(find scte_description)/urdf/scte_drive_axle.xacro"/>
-    <xacro:scte_drive_axle link_name="rear_axle"
-                           parent_link="rear_diff_tower"
-                           drive_axle_radius="${drive_axle_radius}"
-                           drive_axle_length="${drive_axle_length}"
-                           drive_axle_joint_xyz="0 0 ${0.03 * 0.5}"
-                           drive_axle_joint_rpy="${M_PI * -0.5} 0 0"
-    />
-    <!-- Wheel macros for audio bot implementation
+    <xacro:scte_drive_axle
+        link_name="front_axle"
+        parent_link="front_diff_tower"
+        drive_axle_radius="${drive_axle_radius}"
+        drive_axle_length="${drive_axle_length}"
+        drive_axle_joint_xyz="0 0 ${0.03 * 0.5}"
+        drive_axle_joint_rpy="${M_PI * -0.5} 0 0"
+    />
+    <xacro:scte_drive_axle
+        link_name="rear_axle"
+        parent_link="rear_diff_tower"
+        drive_axle_radius="${drive_axle_radius}"
+        drive_axle_length="${drive_axle_length}"
+        drive_axle_joint_xyz="0 0 ${0.03 * 0.5}"
+        drive_axle_joint_rpy="${M_PI * -0.5} 0 0"
+    />
+    <!-- Wheel macros for audibot implementation
+    <!XXxacro:include filename="$(find scte_description)/urdf/plugins/scte_audi_bot_plugin.gazebo"/XX>
+    <xacro:property name="wheel_length" value="0.47" /> <!XX separation between wheels? XX>
+    <xacro:property name="wheel_width" value="${0.20 - wheel_thickness}" /> <!XX separation between wheels? XX>
     <xacro:include filename="$(find scte_description)/urdf/scte_wheel.xacro"/>
-    <xacro:scte_wheel link_name="front_left_wheel"
-                      parent_link="front_axle"
-                      wheel_radius="${wheel_radius}"
-                      wheel_length="${wheel_length}"
-                      wheel_joint_origin="0 0 ${drive_axle_length * 0.5}"
-                      wheel_joint_rpy="${M_PI * -0.5} 0 0"
-                      wheel_joint_name="front_left_wheel_TO_front_axle"
-                      wheel_steer_joint_name="front_left_wheel_steer_TO_front_axle"
-                      is_steerable="true"
-                      flip="1"
-    />
-    <xacro:scte_wheel link_name="front_right_wheel"
-                      parent_link="front_axle"
-                      wheel_radius="${wheel_radius}"
-                      wheel_length="${wheel_length}"
-                      wheel_joint_origin="0 0 ${drive_axle_length * -0.5}"
-                      wheel_joint_rpy="${M_PI * -0.5} 0 0"
-                      wheel_joint_name="front_right_wheel_TO_front_axle"
-                      wheel_steer_joint_name="front_right_wheel_steer_TO_front_axle"
-                      is_steerable="true"
-                      flip="-1"
-    />
-    <xacro:scte_wheel link_name="rear_left_wheel"
-                      parent_link="rear_axle"
-                      wheel_radius="${wheel_radius}"
-                      wheel_length="${wheel_length}"
-                      wheel_joint_origin="0 0 ${drive_axle_length * 0.5}"
-                      wheel_joint_rpy="0 0 0"
-                      wheel_joint_name="rear_left_wheel_TO_rear_axle"
-                      wheel_steer_joint_name=""
-                      is_steerable="false"
-                      flip="1"
-    />
-    <xacro:scte_wheel link_name="rear_right_wheel"
-                      parent_link="rear_axle"
-                      wheel_radius="${wheel_radius}"
-                      wheel_length="${wheel_length}"
-                      wheel_joint_origin="0 0 ${drive_axle_length * -0.5}"
-                      wheel_joint_rpy="0 0 0"
-                      wheel_joint_name="rear_right_wheel_TO_rear_axle"
-                      wheel_steer_joint_name=""
-                      is_steerable="false"
-                      flip="1"
+    <xacro:scte_wheel
+        link_name="front_left_wheel"
+        parent_link="front_axle"
+        wheel_radius="${wheel_radius}"
+        wheel_length="${wheel_length}"
+        wheel_joint_origin="0 0 ${drive_axle_length * 0.5}"
+        wheel_joint_rpy="${M_PI * -0.5} 0 0"
+        wheel_joint_name="front_left_wheel_TO_front_axle"
+        wheel_steer_joint_name="front_left_wheel_steer_TO_front_axle"
+        is_steerable="true"
+        flip="1"
+    />
+    <xacro:scte_wheel
+        link_name="front_right_wheel"
+        parent_link="front_axle"
+        wheel_radius="${wheel_radius}"
+        wheel_length="${wheel_length}"
+        wheel_joint_origin="0 0 ${drive_axle_length * -0.5}"
+        wheel_joint_rpy="${M_PI * -0.5} 0 0"
+        wheel_joint_name="front_right_wheel_TO_front_axle"
+        wheel_steer_joint_name="front_right_wheel_steer_TO_front_axle"
+        is_steerable="true"
+        flip="-1"
+    />
+    <xacro:scte_wheel
+        link_name="rear_left_wheel"
+        parent_link="rear_axle"
+        wheel_radius="${wheel_radius}"
+        wheel_length="${wheel_length}"
+        wheel_joint_origin="0 0 ${drive_axle_length * 0.5}"
+        wheel_joint_rpy="0 0 0"
+        wheel_joint_name="rear_left_wheel_TO_rear_axle"
+        wheel_steer_joint_name=""
+        is_steerable="false"
+        flip="1"
+    />
+    <xacro:scte_wheel
+        link_name="rear_right_wheel"
+        parent_link="rear_axle"
+        wheel_radius="${wheel_radius}"
+        wheel_length="${wheel_length}"
+        wheel_joint_origin="0 0 ${drive_axle_length * -0.5}"
+        wheel_joint_rpy="0 0 0"
+        wheel_joint_name="rear_right_wheel_TO_rear_axle"
+        wheel_steer_joint_name=""
+        is_steerable="false"
+        flip="1"
     />
     -->
     <xacro:include filename="$(find scte_description)/urdf/scte_wheel.xacro"/>
     <!-- joints for ackermann_steering_controller -->
-    <xacro:front_steer name="front" parent="base" radius="${wheel_radius}" thickness="${wheel_thickness}"
-                       length="${wheel_length}" width="${wheel_width}" axel_offset="${axel_offset}" steer_height="${wheel_radius+steer_offset}">
-        <origin xyz="${wheel_length/2-axel_offset} 0 0" rpy="${-90 * deg_to_rad} 0 0"/>
+    <xacro:front_steer
+        name="front"
+        parent="base"
+        radius="${wheel_radius}"
+        thickness="${wheel_thickness}"
+        length="${wheel_base}"
+        width="${wheel_track}"
+        axel_offset="${axel_offset}"
+        steer_height="${wheel_radius+steer_offset}">
+        <!--origin xyz="${wheel_base/2-axel_offset} 0 0" rpy="${-90 * deg_to_rad} 0 0"/-->
     </xacro:front_steer>
-    <xacro:rear_wheel name="rear" parent="base" radius="${wheel_radius}" thickness="${wheel_thickness}">
-        <origin xyz="${-wheel_length/2+axel_offset} 0 0" rpy="${-90 * deg_to_rad} 0 0"/>
+    <!-- the "fake" rear wheel -->
+    <xacro:rear_wheel
+        name="rear"
+        parent="base"
+        radius="${wheel_radius}"
+        thickness="${wheel_thickness}">
+        <origin xyz="${-wheel_base/2+axel_offset} 0 0" rpy="${-90 * deg_to_rad} 0 0"/>
     </xacro:rear_wheel>
     <!-- Wheels -->
-    <xacro:front_wheel_lr name="front_right" parent="base" radius="${wheel_radius}" thickness="${wheel_thickness}"
-                          length="${wheel_length}" width="${wheel_width}" axel_offset="${axel_offset}" right_left="-1" steer_height="${wheel_radius+steer_offset}">
-        <origin xyz="${wheel_length/2-axel_offset} ${wheel_width/2+axel_offset} 0" rpy="${-90 * deg_to_rad} 0 0"/>
+    <xacro:front_wheel_lr
+        name="front_right"
+        parent="base"
+        radius="${wheel_radius}"
+        thickness="${wheel_thickness}"
+        length="${wheel_base}"
+        width="${wheel_track}"
+        axel_offset="${axel_offset}"
+        right_left="-1"
+        steer_height="${wheel_radius+steer_offset}">
+        <!--origin xyz="${wheel_base/2-axel_offset} ${wheel_track/2+axel_offset} ${scte_chassis_depth * -0.5}" rpy="${-90 * deg_to_rad} 0 0"/-->
     </xacro:front_wheel_lr>
-    <xacro:front_wheel_lr name="front_left" parent="base" radius="${wheel_radius}" thickness="${wheel_thickness}"
-                          length="${wheel_length}" width="${wheel_width}" axel_offset="${axel_offset}" right_left="1" steer_height="${wheel_radius+steer_offset}">
-        <origin xyz="${wheel_length/2-axel_offset} ${-wheel_width/2-axel_offset} ${scte_chassis_depth * -0.5}" rpy="${-90 * deg_to_rad} 0 0"/>
+    <xacro:front_wheel_lr
+        name="front_left"
+        parent="base"
+        radius="${wheel_radius}"
+        thickness="${wheel_thickness}"
+        length="${wheel_base}"
+        width="${wheel_track}"
+        axel_offset="${axel_offset}"
+        right_left="1"
+        steer_height="${wheel_radius+steer_offset}">
+        <!--origin xyz="${wheel_base/2-axel_offset} ${-wheel_track/2-axel_offset} ${scte_chassis_depth * -0.5}" rpy="${-90 * deg_to_rad} 0 0"/-->
     </xacro:front_wheel_lr>
-    <xacro:rear_wheel_lr name="rear_left" parent="base" radius="${wheel_radius}" thickness="${wheel_thickness}">
-        <origin xyz="${-wheel_length/2+axel_offset} ${wheel_width/2+axel_offset} ${scte_chassis_depth * -0.5}" rpy="${-90 * deg_to_rad} 0 0"/>
+    <xacro:rear_wheel_lr
+        name="rear_left"
+        parent="base"
+        radius="${wheel_radius}"
+        thickness="${wheel_thickness}">
+        <origin xyz="${-wheel_base/2+axel_offset} ${wheel_track/2+axel_offset} ${scte_chassis_depth * -0.5}" rpy="${-90 * deg_to_rad} 0 0"/>
     </xacro:rear_wheel_lr>
-    <xacro:rear_wheel_lr name="rear_right" parent="base" radius="${wheel_radius}" thickness="${wheel_thickness}">
-        <origin xyz="${-wheel_length/2+axel_offset} ${-wheel_width/2-axel_offset} ${scte_chassis_depth * -0.5}" rpy="${-90 * deg_to_rad} 0 0"/>
+    <xacro:rear_wheel_lr
+        name="rear_right"
+        parent="base"
+        radius="${wheel_radius}"
+        thickness="${wheel_thickness}">
+        <origin xyz="${-wheel_base/2+axel_offset} ${-wheel_track/2-axel_offset} ${scte_chassis_depth * -0.5}" rpy="${-90 * deg_to_rad} 0 0"/>
     </xacro:rear_wheel_lr>
-    <xacro:mounting_bar link_name="driver_mounting_bar"
-                        parent_link="front_diff_tower"
-                        bar_origin="${scte_chassis_length * -0.63} ${shock_tower_width * 0.5} ${shock_tower_height * 1.0}"
-                        bar_rpy="0 0 0"
-    />
-    <xacro:mounting_bar link_name="passenger_mounting_bar"
-                        parent_link="front_diff_tower"
-                        bar_origin="${scte_chassis_length * -0.63} ${shock_tower_width * -0.5} ${shock_tower_height * 1.0}"
-                        bar_rpy="0 0 0"
-    />
-    <xacro:computer_enclosure link_name="computer_enclosure"
-                              parent_link="driver_mounting_bar"
-                              enclosure_origin="0 ${(scte_chassis_width * -0.5) + (0.025 * 0.5)} ${0.06 * 0.5}"
-                              enclosure_rpy="0 0 0"
-    />
-    <xacro:camera_rig link_name="camera_rig"
-                      parent_link="computer_enclosure"
-                      camera_rig_origin="${0.260 * -0.45} 0 ${0.06 * 1.0}"
-                      camera_rig_rpy="0 0 0"
+    <!-- mounting hardware -->
+    <xacro:mounting_bar
+        link_name="driver_mounting_bar"
+        parent_link="front_diff_tower"
+        bar_origin="${scte_chassis_length * -0.63} ${shock_tower_width * 0.5} ${shock_tower_height * 1.0}"
+        bar_rpy="0 0 0"
+    />
+    <xacro:mounting_bar
+        link_name="passenger_mounting_bar"
+        parent_link="front_diff_tower"
+        bar_origin="${scte_chassis_length * -0.63} ${shock_tower_width * -0.5} ${shock_tower_height * 1.0}"
+        bar_rpy="0 0 0"
+    />
+    <xacro:computer_enclosure
+        link_name="computer_enclosure"
+        parent_link="driver_mounting_bar"
+        enclosure_origin="0 ${(scte_chassis_width * -0.5) + (0.025 * 0.5)} ${0.06 * 0.5}"
+        enclosure_rpy="0 0 0"
+    />
+    <xacro:camera_rig
+        link_name="camera_rig"
+        parent_link="computer_enclosure"
+        camera_rig_origin="${0.260 * -0.45} 0 ${0.06 * 1.0}"
+        camera_rig_rpy="0 0 0"
     />
     <!-- Sim IMU -->

File: src/models/scte_vehicle/scte_description/urdf/scte_wheel.xacro (robot description, xacro)
@@ -6,5 +6,14 @@
     <xacro:property name="steer_effort"   value="10.0"/>
     <xacro:property name="steer_velocity" value="5.0"/>
-    <xacro:macro name="front_steer" params="name parent radius thickness length width axel_offset steer_height *origin">
+    <xacro:macro name="front_steer"
+                 params="
+                 name
+                 parent
+                 radius
+                 thickness
+                 length
+                 width
+                 axel_offset
+                 steer_height">
         <link name="${name}_steer_link">
             <inertial>
@@ -39,5 +48,15 @@
         </gazebo>
     </xacro:macro>
-    <xacro:macro name="front_wheel_lr" params="name parent radius thickness length width axel_offset right_left steer_height *origin">
+    <xacro:macro name="front_wheel_lr"
+        params="
+            name
+            parent
+            radius
+            thickness
+            length
+            width
+            axel_offset
+            right_left
+            steer_height">
         <link name="${name}_steer_link">
             <inertial>
@@ -138,5 +157,11 @@
         </gazebo>
     </xacro:macro>
-    <xacro:macro name="rear_wheel" params="name parent radius thickness *origin">
+    <xacro:macro name="rear_wheel"
+         params="
+             name
+             parent
+             radius
+             thickness
+             *origin">
         <link name="${name}_wheel_link">
             <inertial>
@@ -188,5 +213,11 @@
         </gazebo>
     </xacro:macro>
-    <xacro:macro name="rear_wheel_lr" params="name parent radius thickness *origin">
+    <xacro:macro name="rear_wheel_lr"
+        params="
+            name
+            parent
+            radius
+            thickness
+            *origin">
         <link name="${name}_wheel_link">
             <inertial>
