Commit message: checkin of work using steer bot as xacro base

File: src/models/scte_vehicle/scte_description/urdf/scte_chassis.xacro (robot description, xacro)
@@ -10,11 +10,13 @@
 -->
 <!--
-Geometry:
-The Ackermann steering controllers require the longitudinal
-separation between the front and back wheel axes and the
-lateral separation between the left and right front steering axes.
-For this model:
-wheel_separation_h = base_length - 2 * axle_offset = 0.4
-wheel_separation_w = base_width  + 2 * axle_offset = 0.4
+    Robot model adapted from https://github.com/CIR-KIT/steer_drive_ros/blob/kinetic-devel/steer_drive_controller/test/common/urdf/steerbot.xacro
+    Geometry:
+    The Ackermann steering controllers require the longitudinal
+    separation between the front and back wheel axes and the
+    lateral separation between the left and right front steering axes.
+    For this model:
+    wheel_separation_h = base_length - 2 * axle_offset = 0.4
+    wheel_separation_w = base_width  + 2 * axle_offset = 0.4
+    Modified from the steer_bot example found here: https://github.com/srmainwaring/steer_bot
 -->
 <!--Gazebo does not seem to like capital letters in the robot namespace-->

File: src/models/scte_vehicle/scte_description/urdf/scte_wheel.xacro (robot description, xacro)
@@ -1,42 +1,43 @@
 <?xml version="1.0"?>
 <robot xmlns:xacro="http://www.ros.org/wiki/xacro">
-    <!-- Copied from ackermann_steering_bot example -->
-    <xacro:property name="steer_radius" value="0.05" /> <!-- Link 1 -->
-    <xacro:property name="steer_thickness" value="0.02" /> <!-- Link 1 -->
-    <xacro:property name="steer_effort"   value="10.0"/>
+    <!-- Properties -->
+    <xacro:property name="steer_effort" value="10.0"/>
     <xacro:property name="steer_velocity" value="5.0"/>
+    <xacro:property name="steer_limit_deg" value="45.0"/>
+    <!-- Bicycle model front steering link (required for steer_drive_controller) -->
     <xacro:macro name="front_steer"
                  params="
-                 name
-                 parent
-                 radius
-                 thickness
-                 length
-                 width
-                 axel_offset
-                 steer_height">
+                    name
+                    parent
+                    steer_radius
+                    steer_thickness
+                    steer_mass
+                    base_length
+                    base_width
+                    axle_offset
+                    steer_height">
         <link name="${name}_steer_link">
-            <inertial>
-                <origin xyz="0 0 0" rpy="0 0 0"/>
-                <mass value="1"/>
-                <inertia ixx="0.2" ixy="0" ixz="0" iyy="0.2" iyz="0" izz="0.2"/>
-            </inertial>
-            <visual>
-                <origin xyz="0 0 0" rpy="0 0 0"/>
-                <geometry>
-                    <cylinder radius="${steer_radius}" length="${steer_thickness}"/>
-                </geometry>
-            </visual>
-            <collision>
-                <origin xyz="0 0 0" rpy="0 0 0"/>
-                <geometry>
-                    <cylinder radius="${steer_radius}" length="${steer_thickness}"/>
-                </geometry>
-            </collision>
+            <visual>
+                <origin xyz="0 0 0" rpy="0 0 0"/>
+                <geometry>
+                    <cylinder radius="${steer_radius}" length="${steer_thickness}"/>
+                </geometry>
+                <material name="yellow" />
+            </visual>
+            <collision>
+                <origin xyz="0 0 0" rpy="0 0 0"/>
+                <geometry>
+                    <cylinder radius="${steer_radius}" length="${steer_thickness}"/>
+                </geometry>
+            </collision>
+            <xacro:solid_cylinder_inertial
+                    rpy="0 0 0" xyz="0 0 0"
+                    mass="${steer_mass}"
+                    radius="${steer_radius}" length="${steer_thickness}" />
         </link>
         <joint name="${name}_steer_joint" type="revolute">
             <parent link="${parent}_link"/>
             <child link="${name}_steer_link"/>
-            <origin xyz="${length/2-axel_offset} 0 ${steer_height}" rpy="0 0 0"/>
+            <origin xyz="${base_length/2-axle_offset} 0 ${steer_height}" rpy="0 0 0"/>
             <axis xyz="0 0 1"/>
             <limit effort="${steer_effort}"
@@ -44,66 +45,80 @@
                    velocity="${steer_velocity}"/>
         </joint>
+        <transmission name="${name}_steer_joint_trans">
+            <type>transmission_interface/SimpleTransmission</type>
+            <actuator name="${name}_steer_joint_motor">
+                <mechanicalReduction>1</mechanicalReduction>
+                <hardwareInterface>hardware_interface/PositionJointInterface</hardwareInterface>
+            </actuator>
+            <joint name="${name}_steer_joint">
+                <hardwareInterface>hardware_interface/PositionJointInterface</hardwareInterface>
+            </joint>
+        </transmission>
         <gazebo reference="${name}_steer_link">
             <material>Gazebo/Yellow</material>
         </gazebo>
     </xacro:macro>
+    <!-- Car steering model front (steerable) wheel links (left/right) -->
     <xacro:macro name="front_wheel_lr"
-        params="
-            name
-            parent
-            radius
-            thickness
-            length
-            width
-            axel_offset
-            right_left
-            steer_height">
+                 params="
+                    name
+                    parent
+                    reflect
+                    wheel_radius
+                    wheel_thickness
+                    wheel_mass
+                    steer_radius
+                    steer_thickness
+                    steer_mass
+                    base_length
+                    base_width
+                    axle_offset
+                    steer_height">
         <link name="${name}_steer_link">
-            <inertial>
-                <origin xyz="0 0 0" rpy="0 0 0"/>
-                <mass value="1"/>
-                <inertia ixx="0.2" ixy="0" ixz="0" iyy="0.2" iyz="0" izz="0.2"/>
-            </inertial>
-            <visual>
-                <origin xyz="0 0 0" rpy="0 0 0"/>
-                <geometry>
-                    <cylinder radius="${steer_radius}" length="${steer_thickness}"/>
-                </geometry>
-            </visual>
-            <collision>
-                <origin xyz="0 0 0" rpy="0 0 0"/>
-                <geometry>
-                    <cylinder radius="${steer_radius}" length="${steer_thickness}"/>
-                </geometry>
-            </collision>
+            <visual>
+                <origin xyz="0 0 0" rpy="0 0 0"/>
+                <geometry>
+                    <cylinder radius="${steer_radius}" length="${steer_thickness}"/>
+                </geometry>
+                <material name="blue" />
+            </visual>
+            <collision>
+                <origin xyz="0 0 0" rpy="0 0 0"/>
+                <geometry>
+                    <cylinder radius="${steer_radius}" length="${steer_thickness}"/>
+                </geometry>
+            </collision>
+            <xacro:solid_cylinder_inertial
+                    rpy="0 0 0" xyz="0 0 0"
+                    mass="${steer_mass}"
+                    radius="${steer_radius}" length="${steer_thickness}" />
         </link>
         <joint name="${name}_steer_joint" type="revolute">
             <parent link="${parent}_link"/>
             <child link="${name}_steer_link"/>
-            <origin xyz="${length/2-axel_offset} ${right_left*(width/2+axel_offset)} ${steer_height}" rpy="0 0 0"/>
-            <!--xacro:insert_block name="origin"/-->
+            <origin xyz="${base_length/2-axle_offset} ${reflect*(base_width/2+axle_offset)} ${steer_height}" rpy="0 0 0"/>
             <axis xyz="0 0 1"/>
             <limit effort="${steer_effort}"
-                   lower="${-180.0 * deg_to_rad}" upper="${180.0 * deg_to_rad}"
+                   lower="${steer_limit_deg * deg_to_rad * -1.0}" upper="${steer_limit_deg * deg_to_rad}"
                    velocity="${steer_velocity}"/>
         </joint>
         <link name="${name}_wheel_link">
-            <inertial>
-                <origin xyz="0 0 0" rpy="0 0 0"/>
-                <mass value="1"/>
-                <inertia ixx="0.2" ixy="0" ixz="0" iyy="0.2" iyz="0" izz="0.2"/>
-            </inertial>
-            <visual>
-                <origin xyz="0 0 0" rpy="0 0 0"/>
-                <geometry>
-                    <cylinder radius="${wheel_radius}" length="${thickness}"/>
-                </geometry>
-            </visual>
-            <collision>
-                <origin xyz="0 0 0" rpy="0 0 0"/>
-                <geometry>
-                    <cylinder radius="${wheel_radius}" length="${thickness}"/>
-                </geometry>
-            </collision>
+            <visual>
+                <origin xyz="0 0 0" rpy="0 0 0"/>
+                <geometry>
+                    <cylinder radius="${wheel_radius}" length="${wheel_thickness}"/>
+                </geometry>
+                <material name="red" />
+            </visual>
+            <collision>
+                <origin xyz="0 0 0" rpy="0 0 0"/>
+                <geometry>
+                    <cylinder radius="${wheel_radius}" length="${wheel_thickness}"/>
+                </geometry>
+            </collision>
+            <xacro:solid_cylinder_inertial
+                    rpy="0 0 0" xyz="0 0 0"
+                    mass="${wheel_mass}"
+                    radius="${wheel_radius}" length="${wheel_thickness}" />
         </link>
         <joint name="${name}_wheel_joint" type="continuous">
@@ -113,40 +128,23 @@
             <axis xyz="0 0 1"/>
         </joint>
-        <!-- Transmission is important to link the joints and the controller -->
-        <!--
         <transmission name="${name}_steer_joint_trans">
-            <type>SimpleTransmission</type>
-            <actuator name="${name}_steer_joint_motor"/>
-            <joint name="${name}_steer_joint"/>
-            <mechanicalReduction>1</mechanicalReduction>
-            <motorTorqueConstant>1</motorTorqueConstant>
+            <type>transmission_interface/SimpleTransmission</type>
+            <actuator name="${name}_steer_joint_motor">
+                <mechanicalReduction>1</mechanicalReduction>
+                <hardwareInterface>hardware_interface/PositionJointInterface</hardwareInterface>
+            </actuator>
+            <joint name="${name}_steer_joint">
+                <hardwareInterface>hardware_interface/PositionJointInterface</hardwareInterface>
+            </joint>
         </transmission>
         <transmission name="${name}_wheel_joint_trans">
-            <type>SimpleTransmission</type>
-            <actuator name="${name}_wheel_joint_motor"/>
-            <joint name="${name}_wheel_joint"/>
-            <mechanicalReduction>1</mechanicalReduction>
-            <motorTorqueConstant>1</motorTorqueConstant>
-        </transmission>
-        -->
-        <transmission name="${name}_steer_joint_trans">
-            <type>transmission_interface/SimpleTransmission</type>
-            <joint name="${name}_steer_joint">
-                <hardwareInterface>hardware_interface/EffortJointInterface</hardwareInterface>
-            </joint>
-            <actuator name="${name}_steer_joint_motor">
-                <hardwareInterface>hardware_interface/EffortJointInterface</hardwareInterface>
-                <mechanicalReduction>1</mechanicalReduction>
-            </actuator>
-        </transmission>
-        <transmission name="${name}_wheel_joint_trans">
-            <type>transmission_interface/SimpleTransmission</type>
+            <type>transmission_interface/SimpleTransmission</type>
+            <actuator name="${name}_wheel_joint_motor">
+                <mechanicalReduction>1</mechanicalReduction>
+                <hardwareInterface>hardware_interface/VelocityJointInterface</hardwareInterface>
+            </actuator>
             <joint name="${name}_wheel_joint">
-                <hardwareInterface>hardware_interface/EffortJointInterface</hardwareInterface>
-            </joint>
-            <actuator name="${name}_wheel_joint_motor">
-                <hardwareInterface>hardware_interface/EffortJointInterface</hardwareInterface>
-                <mechanicalReduction>1</mechanicalReduction>
-            </actuator>
+                <hardwareInterface>hardware_interface/VelocityJointInterface</hardwareInterface>
+            </joint>
         </transmission>
         <gazebo reference="${name}_steer_link">
@@ -157,29 +155,31 @@
         </gazebo>
     </xacro:macro>
+    <!-- Bicycle model rear wheel link (required for steer_drive_controller) -->
     <xacro:macro name="rear_wheel"
-         params="
-             name
-             parent
-             radius
-             thickness
-             *origin">
-        <link name="${name}_wheel_link">
-            <inertial>
-                <origin xyz="0 0 0" rpy="0 0 0"/>
-                <mass value="1"/>
-                <inertia ixx="0.2" ixy="0" ixz="0" iyy="0.2" iyz="0" izz="0.2"/>
-            </inertial>
-            <visual>
-                <origin xyz="0 0 0" rpy="0 0 0"/>
-                <geometry>
-                    <cylinder radius="${wheel_radius}" length="${thickness}"/>
-                </geometry>
-            </visual>
-            <collision>
-                <origin xyz="0 0 0" rpy="0 0 0"/>
-                <geometry>
-                    <cylinder radius="${wheel_radius}" length="${thickness}"/>
-                </geometry>
-            </collision>
+                 params="
+      name
+      parent
+      wheel_radius
+      wheel_thickness
+      wheel_mass
+      *origin">
+        <link name="${name}_wheel_link">
+            <visual>
+                <origin xyz="0 0 0" rpy="0 0 0"/>
+                <geometry>
+                    <cylinder radius="${wheel_radius}" length="${wheel_thickness}"/>
+                </geometry>
+                <material name="yellow" />
+            </visual>
+            <collision>
+                <origin xyz="0 0 0" rpy="0 0 0"/>
+                <geometry>
+                    <cylinder radius="${wheel_radius}" length="${wheel_thickness}"/>
+                </geometry>
+            </collision>
+            <xacro:solid_cylinder_inertial
+                    rpy="0 0 0" xyz="0 0 0"
+                    mass="${wheel_mass}"
+                    radius="${wheel_radius}" length="${wheel_thickness}" />
         </link>
         <joint name="${name}_wheel_joint" type="continuous">
@@ -189,80 +189,102 @@
             <axis xyz="0 0 1"/>
         </joint>
-        <!-- Transmission is important to link the joints and the controller -->
-        <!--
         <transmission name="${name}_wheel_joint_trans">
-            <type>SimpleTransmission</type>
-            <actuator name="${name}_wheel_joint_motor"/>
-            <joint name="${name}_wheel_joint"/>
-            <mechanicalReduction>1</mechanicalReduction>
-            <motorTorqueConstant>1</motorTorqueConstant>
-        </transmission>
-        -->
+            <type>transmission_interface/SimpleTransmission</type>
+            <actuator name="${name}_wheel_joint_motor">
+                <mechanicalReduction>1</mechanicalReduction>
+                <hardwareInterface>hardware_interface/VelocityJointInterface</hardwareInterface>
+            </actuator>
+            <joint name="${name}_wheel_joint">
+                <hardwareInterface>hardware_interface/VelocityJointInterface</hardwareInterface>
+            </joint>
+        </transmission>
+        <gazebo reference="${name}_wheel_link">
+            <material>Gazebo/Yellow</material>
+        </gazebo>
+    </xacro:macro>
+    <!-- Bicycle model front wheel link (passive - no transmission) -->
+    <xacro:macro name="front_wheel"
+                 params="
+      name
+      parent
+      wheel_radius
+      wheel_thickness
+      wheel_mass
+      *origin">
+        <link name="${name}_wheel_link">
+            <visual>
+                <origin xyz="0 0 0" rpy="0 0 0"/>
+                <geometry>
+                    <cylinder radius="${wheel_radius}" length="${wheel_thickness}"/>
+                </geometry>
+                <material name="yellow" />
+            </visual>
+            <collision>
+                <origin xyz="0 0 0" rpy="0 0 0"/>
+                <geometry>
+                    <cylinder radius="${wheel_radius}" length="${wheel_thickness}"/>
+                </geometry>
+            </collision>
+            <xacro:solid_cylinder_inertial
+                    rpy="0 0 0" xyz="0 0 0"
+                    mass="${wheel_mass}"
+                    radius="${wheel_radius}" length="${wheel_thickness}" />
+        </link>
+        <joint name="${name}_wheel_joint" type="continuous">
+            <parent link="${parent}_link"/>
+            <child link="${name}_wheel_link"/>
+            <xacro:insert_block name="origin"/>
+            <axis xyz="0 0 1"/>
+        </joint>
+        <gazebo reference="${name}_wheel_link">
+            <material>Gazebo/Yellow</material>
+        </gazebo>
+        <gazebo reference="${name}_wheel_joint">
+            <provideFeedback>true</provideFeedback>
+        </gazebo>
+    </xacro:macro>
+    <!-- Car steering model rear wheel links (left/right) -->
+    <xacro:macro name="rear_wheel_lr"
+                 params="
+      name
+      parent
+      wheel_radius
+      wheel_thickness
+      wheel_mass
+      *origin">
+        <link name="${name}_wheel_link">
+            <visual>
+                <origin xyz="0 0 0" rpy="0 0 0"/>
+                <geometry>
+                    <cylinder radius="${wheel_radius}" length="${wheel_thickness}"/>
+                </geometry>
+                <material name="red" />
+            </visual>
+            <collision>
+                <origin xyz="0 0 0" rpy="0 0 0"/>
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