Commit message: improved the models inertial properties. still needs lots of work. front wheels dont seem to turn much when rear wheels spin. center of masses seem offset.

File: src/models/scte_vehicle/scte_description/urdf/equipment/camera_rig.xacro (robot description, xacro)
@@ -3,5 +3,5 @@
 <link name="stereo_camera_bar_support">
     <inertial>
-        <mass value="${scte_total_mass * 0.01}"/>
+        <mass value="${scte_chassis_mass * 0.01}"/>
         <origin xyz="0 0 0" rpy="0 0 0"/>
         <inertia
@@ -32,5 +32,5 @@
 <link name="stereo_camera_bar">
 <inertial>
-    <mass value="${scte_total_mass * 0.01}"/>
+    <mass value="${scte_chassis_mass * 0.01}"/>
     <origin xyz="0 0 0" rpy="0 0 0"/>
     <inertia
@@ -71,5 +71,5 @@
         <link name="debug_stereo_perception_camera">
             <inertial>
-                <mass value="${scte_total_mass * 0.0001}"/>
+                <mass value="${scte_chassis_mass * 0.0001}"/>
                 <origin xyz="0 0 0" rpy="0 0 0"/>
                 <inertia

File: src/models/scte_vehicle/scte_description/urdf/equipment/computer_enclosure.xacro (robot description, xacro)
@@ -2,5 +2,5 @@
 <link name="main_computer_enclosure">
     <inertial>
-        <mass value="${scte_total_mass * 0.02}"/>
+        <mass value="${scte_chassis_mass * 0.02}"/>
         <origin xyz="0 0 0" rpy="0 0 0"/>
         <inertia

File: src/models/scte_vehicle/scte_description/urdf/equipment/mounting_bars_temp.xacro (robot description, xacro)
@@ -6,5 +6,5 @@
     <link name="driver_side_mounting_bar">
         <inertial>
-            <mass value="${scte_total_mass * 0.02}"/>
+            <mass value="${scte_chassis_mass * 0.02}"/>
             <origin xyz="0 0 0" rpy="0 0 0"/>
             <inertia
@@ -35,5 +35,5 @@
     <link name="passenger_side_mounting_bar">
         <inertial>
-            <mass value="${scte_total_mass * 0.02}"/>
+            <mass value="${scte_chassis_mass * 0.02}"/>
             <origin xyz="0 0 0" rpy="0 0 0"/>
             <inertia

File: src/models/scte_vehicle/scte_description/urdf/scte_chassis.xacro (robot description, xacro)
@@ -12,14 +12,20 @@
 <robot name="sctebot" xmlns:xacro="http://www.ros.org/wiki/xacro">
     <xacro:arg name="robot_namespace" default="/DEFAULTNAMESPACE2"/>
+    <xacro:arg name="tf_freq" default="100.0"/>
+    <xacro:arg name="pub_tf" default="false"/>
     <xacro:property name="M_PI" value="3.14159265358979323846264338327950288"/>
     <xacro:include filename="$(find scte_description)/urdf/scte.gazebo" />
     <xacro:include filename="$(find scte_description)/urdf/materials.xacro" />
     <xacro:include filename="$(find scte_description)/urdf/macros.xacro" />
-    <xacro:property name="scte_total_mass" value="50"/>
+    <xacro:property name="scte_chassis_mass" value="2.9"/>
     <xacro:property name="scte_chassis_length" value="0.292"/>
     <xacro:property name="scte_chassis_width" value="0.165"/>
     <xacro:property name="scte_chassis_depth" value="0.00635"/>
+    <xacro:property name="scte_chassis_length_sq" value="${scte_chassis_length * scte_chassis_length}"/>
+    <xacro:property name="scte_chassis_width_sq" value="${scte_chassis_width * scte_chassis_width}"/>
+    <xacro:property name="scte_chassis_depth_sq" value="${scte_chassis_depth * scte_chassis_depth}"/>
     <!--Wheel Properties-->
-    <xacro:property name="wheel_radius" value="0.05"/>
+    <xacro:property name="wheel_mass" value="0.5"/>
+    <xacro:property name="wheel_radius" value="0.0525"/>
     <xacro:property name="wheel_length" value="0.045"/>
     <xacro:property name="shock_tower_height" value="0.105"/>
@@ -51,7 +57,9 @@
     <link name="inertial_link">
         <inertial>
-            <mass value="${scte_total_mass * 0.90}" />
+            <mass value="${scte_chassis_mass}" />
             <origin xyz="0 0 0" />
-            <inertia ixx="0.6022" ixy="-0.02364" ixz="-0.1197" iyy="1.7386" iyz="-0.001544" izz="2.0296" />
+            <inertia ixx="${(1/12 * scte_chassis_mass) * (scte_chassis_depth_sq + scte_chassis_width_sq)}" ixy="0" ixz="0"
+                     iyy="${(1/12 * scte_chassis_mass) * (scte_chassis_depth_sq + scte_chassis_length_sq)}" iyz="0"
+                     izz="${(1/12 * scte_chassis_mass) * (scte_chassis_length_sq + scte_chassis_width_sq)}" />
         </inertial>
     </link>
@@ -68,4 +76,5 @@
         <child link="scte_chassis"/>
     </joint>
+    <!---->
     <xacro:include filename="$(find scte_description)/urdf/scte_diff_and_shock_tower.xacro"/>
     <xacro:scte_diff_and_shock_tower link_name="front_diff_tower"
@@ -126,4 +135,6 @@
                       wheel_joint_origin="0 0 ${drive_axle_length * 0.5}"
                       wheel_joint_rpy="${M_PI * -0.5} 0 0"
+                      wheel_joint_name="front_left_wheel_TO_front_axle"
+                      wheel_steer_joint_name="front_left_wheel_steer_TO_front_axle"
                       is_steerable="true"
     />
@@ -134,4 +145,6 @@
                       wheel_joint_origin="0 0 ${drive_axle_length * -0.5}"
                       wheel_joint_rpy="${M_PI * -0.5} 0 0"
+                      wheel_joint_name="front_right_wheel_TO_front_axle"
+                      wheel_steer_joint_name="front_right_wheel_steer_TO_front_axle"
                       is_steerable="true"
     />
@@ -142,4 +155,6 @@
                       wheel_joint_origin="0 0 ${drive_axle_length * 0.5}"
                       wheel_joint_rpy="${M_PI * -0.5} 0 0"
+                      wheel_joint_name="rear_left_wheel_TO_rear_axle"
+                      wheel_steer_joint_name="rear_left_wheel_steer_TO_rear_axle"
                       is_steerable="false"
     />
@@ -150,5 +165,8 @@
                       wheel_joint_origin="0 0 ${drive_axle_length * -0.5}"
                       wheel_joint_rpy="${M_PI * -0.5} 0 0"
+                      wheel_joint_name="rear_right_wheel_TO_rear_axle"
+                      wheel_steer_joint_name="rear_right_wheel_steer_TO_rear_axle"
                       is_steerable="false"
     />
+    -->
 </robot>

File: src/models/scte_vehicle/scte_description/urdf/scte_diff_and_shock_tower.xacro (robot description, xacro)
@@ -12,9 +12,9 @@
         <link name="${link_name}">
             <intertial>
-                <mass value="${scte_total_mass * 0.05}"/>
+                <mass value="${scte_chassis_mass * 0.05}"/>
                 <inertia
-                        ixx="1" ixy="0" ixz="0"
-                        iyy="1" iyz="0"
-                        izz="1"
+                        ixx="1e-6" ixy="0" ixz="0"
+                        iyy="1e-6" iyz="0"
+                        izz="1e-6"
                 />
             </intertial>
@@ -39,9 +39,9 @@
         <link name="${link_name}_shock_tower">
             <inertial>
-                <mass value="${scte_total_mass * 0.25 * 0.05}"/>
+                <mass value="${scte_chassis_mass * 0.25 * 0.05}"/>
                 <inertia
-                        ixx="1" ixy="0" ixz="0"
-                        iyy="1" iyz="0"
-                        izz="1"
+                        ixx="1e-6" ixy="0" ixz="0"
+                        iyy="1e-6" iyz="0"
+                        izz="1e-6"
                 />
             </inertial>

File: src/models/scte_vehicle/scte_description/urdf/scte_drive_axle.xacro (robot description, xacro)
@@ -14,9 +14,9 @@
             <inertial>
                 <origin xyz="0 0 0" rpy="0 0 0" />
-                <mass value="1" />
+                <mass value="0.05" />
                 <inertia
-                        ixx="1.0" ixy="0.0" ixz="0.0"
-                        iyy="1.0" iyz="0.0"
-                        izz="1.0" />
+                        ixx="1e-6" ixy="0.0" ixz="0.0"
+                        iyy="1e-6" iyz="0.0"
+                        izz="1e-6" />
             </inertial>
             <visual name='visual'>

File: src/models/scte_vehicle/scte_description/urdf/scte_front_bumper.xacro (robot description, xacro)
@@ -9,12 +9,12 @@
         <!--front skid plate-->
         <link name="${link_name}_skid_plate">
-            <intertial>
-                <mass value="${scte_total_mass * 0.05}"/>
+            <!--intertial>
+                <mass value="${scte_chassis_mass * 0.05}"/>
                 <inertia
-                        ixx="1" ixy="0" ixz="0"
-                        iyy="1" iyz="0"
-                        izz="1"
+                        ixx="1e-6" ixy="0" ixz="0"
+                        iyy="1e-6" iyz="0"
+                        izz="1e-6"
                 />
-            </intertial>
+            </intertial-->
             <visual>
                 <geometry>
@@ -35,12 +35,12 @@
         </joint>
         <link name="${link_name}">
-            <intertial>
-                <mass value="${scte_total_mass * 0.05}"/>
+            <!--intertial>
+                <mass value="${scte_chassis_mass * 0.05}"/>
                 <inertia
-                        ixx="1" ixy="0" ixz="0"
-                        iyy="1" iyz="0"
-                        izz="1"
+                        ixx="1e-6" ixy="0" ixz="0"
+                        iyy="1e-6" iyz="0"
+                        izz="1e-6"
                 />
-            </intertial>
+            </intertial-->
             <visual>
                 <geometry>

File: src/models/scte_vehicle/scte_description/urdf/scte_rear_bumper.xacro (robot description, xacro)
@@ -8,12 +8,12 @@
         <!--rear bumper assembly-->
         <link name="${link_name}_mount">
-            <intertial>
-                <mass value="${scte_total_mass * 0.05}"/>
+            <!--intertial>
+                <mass value="${scte_chassis_mass * 0.05}"/>
                 <inertia
-                        ixx="1" ixy="0" ixz="0"
-                        iyy="1" iyz="0"
-                        izz="1"
+                        ixx="1e-6" ixy="0" ixz="0"
+                        iyy="1e-6" iyz="0"
+                        izz="1e-6"
                 />
-            </intertial>
+            </intertial-->
             <visual>
                 <geometry>
@@ -35,12 +35,12 @@
         <!---->
         <link name="${link_name}">
-            <intertial>
-                <mass value="${scte_total_mass * 0.05}"/>
+            <!--intertial>
+                <mass value="${scte_chassis_mass * 0.05}"/>
                 <inertia
-                        ixx="1" ixy="0" ixz="0"
-                        iyy="1" iyz="0"
-                        izz="1"
+                        ixx="1e-6" ixy="0" ixz="0"
+                        iyy="1e-6" iyz="0"
+                        izz="1e-6"
                 />
-            </intertial>
+            </intertial-->
             <visual>
                 <geometry>

File: src/models/scte_vehicle/scte_description/urdf/scte_wheel.xacro (robot description, xacro)
@@ -6,4 +6,6 @@
     wheel_joint_origin
     wheel_joint_rpy
+    wheel_joint_name
+    wheel_steer_joint_name
     is_steerable
     ">
@@ -15,9 +17,17 @@
                 <fdir1 value="1 0 0"/>
             </gazebo>
+            <xacro:property name="wheel_radius_sq" value="${wheel_radius * wheel_radius}"/>
+            <xacro:property name="wheel_length_sq" value="${wheel_length * wheel_length}"/>
             <link name="${link_name}_steer">
                 <inertial>
-                    <origin xyz="-0.013054 -0.0295 0" rpy="0 0 0"/>
-                    <mass value="20.0"/>
-                    <inertia ixx="2" ixy="0" ixz="0" iyy="2" iyz="0" izz="2"/>
+                    <origin xyz="-0.02 -0.03 0" rpy="0 0 0"/>
+                    <!-- not sure why this has arbitrary mass and inertial values in the example source-->
+                    <mass value="${wheel_mass * 2}"/>
+                    <!--inertia ixx="${(2/5 * wheel_mass) * wheel_radius_sq}" ixy="0" ixz="0"
+                             iyy="${(2/5 * wheel_mass) * wheel_radius_sq}" iyz="0"
+                             izz="${(2/5 * wheel_mass) * wheel_radius_sq}"/-->
+                    <inertia  ixx="${(1/12 * wheel_mass * 2) * (3 * wheel_radius_sq + wheel_length_sq)}" ixy="0" ixz="0"
+                              iyy="${(1/12 * wheel_mass * 2) * (3 * wheel_radius_sq + wheel_length_sq)}" iyz="0"
+                              izz="${(1/2 * wheel_mass * 2) * wheel_radius_sq}" />
                 </inertial>
             </link>
@@ -32,5 +42,5 @@
             </xacro:if>
             <xacro:if value="${is_steerable == 0}">
-                <joint name="${link_name}_steer_TO_${parent_link}" type="fixed">
+                <joint name="${wheel_steer_joint_name}" type="fixed">
                     <parent link="${parent_link}" />
                     <child link="${link_name}_steer" />
@@ -41,6 +51,8 @@
             <link name="${link_name}">
                 <inertial>
-                    <mass value="${scte_total_mass * 0.25 * 0.05}"/>
-                    <inertia  ixx="0.02467" ixy="0" ixz="0" iyy="0.04411" iyz="0" izz="0.02467" />
+                    <mass value="${wheel_mass}"/>
+                    <inertia  ixx="${(1/12 * wheel_mass) * (3 * wheel_radius_sq + wheel_length_sq)}" ixy="0" ixz="0"
+                              iyy="${(1/12 * wheel_mass) * (3 * wheel_radius_sq + wheel_length_sq)}" iyz="0"
+                              izz="${(1/2 * wheel_mass) * wheel_radius_sq}" />
                 </inertial>
                 <visual name='visual'>
@@ -56,5 +68,5 @@
                 </collision>
             </link>
-            <joint name='${link_name}_TO_${parent_link}' type='continuous'>
+            <joint name='${wheel_joint_name}' type='continuous'>
                 <parent link="${link_name}_steer"/>
                 <child link="${link_name}"/>
