Commit message: reworked and added in the other xacro files that describe the rest of the model. also added in gazebo sensor simulation plugins

File: src/models/scte_vehicle/scte_description/urdf/equipment/camera_rig.xacro (robot description, xacro)
@@ -1,75 +1,11 @@
-<!--SENSORS-->
-<!---->
-<link name="stereo_camera_bar_support">
-    <inertial>
-        <mass value="${scte_chassis_mass * 0.01}"/>
-        <origin xyz="0 0 0" rpy="0 0 0"/>
-        <inertia
-                ixx="1" ixy="0" ixz="0"
-                iyy="1" iyz="0"
-                izz="1"
-        />
-    </inertial>
-    <visual name='visual'>
-        <origin xyz="0 0 0" rpy="0 0 0"/>
-        <geometry>
-            <cylinder radius="0.01" length="0.06"/>
-        </geometry>
-        <material name="blue"/>
-    </visual>
-    <collision name='collision'>
-        <origin xyz="0 0 0" rpy="0 0 0"/>
-        <geometry>
-            <cylinder radius="0.01" length="0.06"/>
-        </geometry>
-    </collision>
-</link>
-<joint name="stereo_camera_bar_support_JOINED_main_computer_enclosure" type="fixed">
-<origin xyz="${0.260 * -0.45} 0 ${0.06 * 1.0}" rpy="0 0 0"/>
-<parent link="main_computer_enclosure"/>
-<child link="stereo_camera_bar_support"/>
-</joint>
-<link name="stereo_camera_bar">
-<inertial>
-    <mass value="${scte_chassis_mass * 0.01}"/>
-    <origin xyz="0 0 0" rpy="0 0 0"/>
-    <inertia
-            ixx="1" ixy="0" ixz="0"
-            iyy="1" iyz="0"
-            izz="1"
-    />
-</inertial>
-<visual name='visual'>
-    <origin xyz="0 0 0" rpy="0 0 0"/>
-    <geometry>
-        <box size="0.03 0.202 0.004"/>
-    </geometry>
-    <material name="blue"/>
-</visual>
-<collision name='collision'>
-    <origin xyz="0 0 0" rpy="0 0 0"/>
-    <geometry>
-        <box size="0.03 0.202 0.004"/>
-    </geometry>
-</collision>
-</link>
-<joint name="stereo_camera_bar_JOINED_stereo_camera_bar_support" type="fixed">
-<origin xyz="0 0 ${0.06 * 0.5}" rpy="0 0 0"/>
-<parent link="stereo_camera_bar_support"/>
-<child link="stereo_camera_bar"/>
-</joint>
-<xacro:include filename="$(find logitech_c270_camera)/urdf/logitech_c270.xacro"/>
-        <!--
-            https://answers.ros.org/question/9840/how-do-you-get-stereo_image_proc-to-include-a-frame_id-so-that-rviz-will-accept-the-point-cloud-messages/
-            - stereo projection/point cloud uses the left cameras frame_id to determine how to draw the image
-            may need to use image_rect for the video to align with the model
-            https://berndpfrommer.github.io/tagslam_web/visualization/
-        -->
-<xacro:logitech_c270_camera parent_link="stereo_camera_bar" camera_link="driver_side_camera" joint_xyz="0.0 0.05 ${0.025 * 0.5}" joint_rpy="0 0 0"/>
-<xacro:logitech_c270_camera parent_link="stereo_camera_bar" camera_link="passenger_side_camera" joint_xyz="0.0 -0.05 ${0.025 * 0.5}" joint_rpy="0 0 0"/>
-        <!--
-        <link name="debug_stereo_perception_camera">
+<?xml version="1.0"?>
+<robot name="sctebot" xmlns:xacro="http://www.ros.org/wiki/xacro">
+    <xacro:macro name="camera_rig" params="link_name parent_link
+    camera_rig_origin
+    camera_rig_rpy
+    ">
+        <link name="${link_name}_support">
             <inertial>
-                <mass value="${scte_chassis_mass * 0.0001}"/>
+                <mass value="${scte_chassis_mass * 0.01}"/>
                 <origin xyz="0 0 0" rpy="0 0 0"/>
                 <inertia
@@ -82,5 +18,5 @@
                 <origin xyz="0 0 0" rpy="0 0 0"/>
                 <geometry>
-                    <box size="0.05 0.05 0.05"/>
+                    <cylinder radius="0.01" length="0.06"/>
                 </geometry>
                 <material name="blue"/>
@@ -89,12 +25,42 @@
                 <origin xyz="0 0 0" rpy="0 0 0"/>
                 <geometry>
-                    <box size="0.05 0.05 0.05"/>
+                    <cylinder radius="0.01" length="0.06"/>
                 </geometry>
             </collision>
         </link>
-        <joint name="debug_stereo_perception_camera_JOINED_stereo_camera_bar" type="fixed">
-            <origin xyz="0 0.5 0" rpy="${M_PI/-2} 0 ${M_PI/-2}"/>
-            <parent link="stereo_camera_bar"/>
-            <child link="debug_stereo_perception_camera"/>
+        <joint name="${link_name}_support_TO_${parent_link}" type="fixed">
+            <origin xyz="${camera_rig_origin}" rpy="${camera_rig_rpy}"/>
+            <parent link="${parent_link}"/>
+            <child link="${link_name}_support"/>
         </joint>
-        -->
+        <link name="${link_name}_bar">
+            <inertial>
+                <mass value="${scte_chassis_mass * 0.01}"/>
+                <origin xyz="0 0 0" rpy="0 0 0"/>
+                <inertia
+                        ixx="1" ixy="0" ixz="0"
+                        iyy="1" iyz="0"
+                        izz="1"
+                />
+            </inertial>
+            <visual name='visual'>
+                <origin xyz="0 0 0" rpy="0 0 0"/>
+                <geometry>
+                    <box size="0.03 0.202 0.004"/>
+                </geometry>
+                <material name="blue"/>
+            </visual>
+            <collision name='collision'>
+                <origin xyz="0 0 0" rpy="0 0 0"/>
+                <geometry>
+                    <box size="0.03 0.202 0.004"/>
+                </geometry>
+            </collision>
+        </link>
+        <joint name="${link_name}_bar_TO_${link_name}_support" type="fixed">
+            <origin xyz="0 0 ${0.06 * 0.5}" rpy="0 0 0"/>
+            <parent link="${link_name}_support"/>
+            <child link="${link_name}_bar"/>
+        </joint>
+    </xacro:macro>
+</robot>

File: src/models/scte_vehicle/scte_description/urdf/equipment/mounting_bars.xacro (robot description, xacro)
@@ -1,8 +1,12 @@
 <?xml version="1.0"?>
 <robot name="sctebot" xmlns:xacro="http://www.ros.org/wiki/xacro">
-    <xacro:macro name="computer_enclosure" params="link_name parent_link
-    enclosure_origin
-    enclosure_rpy
+    <xacro:macro name="mounting_bar" params="link_name
+    parent_link
+    bar_origin
+    bar_rpy
     ">
+        <xacro:property name="mounting_bars_length" value="0.45"/>
+        <xacro:property name="mounting_bars_width" value="0.025"/>
+        <xacro:property name="mounting_bars_depth" value="0.005"/>
         <link name="${link_name}">
             <inertial>
@@ -18,19 +22,17 @@
                 <origin xyz="0 0 0" rpy="0 0 0"/>
                 <geometry>
-                    <box size="0.26 0.185 0.06"/>
+                    <box size="${mounting_bars_length} ${mounting_bars_width} ${mounting_bars_depth}"/>
                 </geometry>
-                <material name="none">
-                    <color rgba="${122/255} ${125/255} ${121/255} 0.5"/>
-                </material>
+                <material name="green"/>
             </visual>
             <collision name='collision'>
                 <origin xyz="0 0 0" rpy="0 0 0"/>
                 <geometry>
-                    <box size="0.26 0.185 0.06"/>
+                    <box size="${mounting_bars_length} ${mounting_bars_width} ${mounting_bars_depth}"/>
                 </geometry>
             </collision>
         </link>
         <joint name="${link_name}_TO_${parent_link}" type="fixed">
-            <origin xyz="${enclosure_origin}" rpy="${enclosure_rpy}"/>
+            <origin xyz="${bar_origin}" rpy="${bar_rpy}"/>
             <parent link="${parent_link}"/>
             <child link="${link_name}"/>

File: src/models/scte_vehicle/scte_description/urdf/scte_chassis.xacro (robot description, xacro)
@@ -18,4 +18,9 @@
     <xacro:include filename="$(find scte_description)/urdf/materials.xacro" />
     <xacro:include filename="$(find scte_description)/urdf/macros.xacro" />
+    <xacro:include filename="$(find ydlidar_ros)/urdf/ydlidar.urdf"/>
+    <xacro:include filename="$(find logitech_c270_camera)/urdf/logitech_c270.xacro"/>
+    <xacro:include filename="$(find scte_description)/urdf/equipment/mounting_bars.xacro"/>
+    <xacro:include filename="$(find scte_description)/urdf/equipment/computer_enclosure.xacro"/>
+    <xacro:include filename="$(find scte_description)/urdf/equipment/camera_rig.xacro"/>
     <xacro:property name="scte_chassis_mass" value="2.9"/>
     <xacro:property name="scte_chassis_length" value="0.292"/>
@@ -26,5 +31,5 @@
     <xacro:property name="scte_chassis_depth_sq" value="${scte_chassis_depth * scte_chassis_depth}"/>
     <!--Wheel Properties-->
-    <xacro:property name="wheel_mass" value="0.5"/>
+    <xacro:property name="wheel_mass" value="0.3"/>
     <xacro:property name="wheel_radius" value="0.0525"/>
     <xacro:property name="wheel_length" value="0.045"/>
@@ -174,3 +179,49 @@
                       flip="1"
     />
+    <xacro:mounting_bar link_name="driver_mounting_bar"
+                        parent_link="front_diff_tower"
+                        bar_origin="${scte_chassis_length * -0.63} ${shock_tower_width * 0.5} ${shock_tower_height * 1.0}"
+                        bar_rpy="0 0 0"
+    />
+    <xacro:mounting_bar link_name="passenger_mounting_bar"
+                        parent_link="front_diff_tower"
+                        bar_origin="${scte_chassis_length * -0.63} ${shock_tower_width * -0.5} ${shock_tower_height * 1.0}"
+                        bar_rpy="0 0 0"
+    />
+    <xacro:computer_enclosure link_name="computer_enclosure"
+                              parent_link="driver_mounting_bar"
+                              enclosure_origin="0 ${(scte_chassis_width * -0.5) + (0.025 * 0.5)} ${0.06 * 0.5}"
+                              enclosure_rpy="0 0 0"
+    />
+    <xacro:camera_rig link_name="camera_rig"
+                      parent_link="computer_enclosure"
+                      camera_rig_origin="${0.260 * -0.45} 0 ${0.06 * 1.0}"
+                      camera_rig_rpy="0 0 0"
+    />
+    <!-- Sim IMU -->
+    <link name="imu_link"/>
+    <joint name="imu_link_TO_computer_enclosure" type="fixed">
+        <origin xyz="0 0 0" rpy="0 0 0"/>
+        <parent link="computer_enclosure"/>
+        <child link="imu_link"/>
+    </joint>
+    <!-- LIDAR -->
+    <!--link name="base_laser"/-->
+    <joint name="ydlidar_base_TO_computer_enclosure" type="fixed">
+        <origin xyz="0.090 0 0.0305" rpy="0 0 0"/>
+        <parent link="computer_enclosure"/>
+        <child link="base_laser"/>
+    </joint>
+    <!-- Cameras -->
+    <!--
+        https://answers.ros.org/question/9840/how-do-you-get-stereo_image_proc-to-include-a-frame_id-so-that-rviz-will-accept-the-point-cloud-messages/
+        - stereo projection/point cloud uses the left cameras frame_id to determine how to draw the image
+        may need to use image_rect for the video to align with the model
+        https://berndpfrommer.github.io/tagslam_web/visualization/
+    -->
+    <!--TODO drowan_20210117_BUG: The cameras are mounted sideways. Need to fix camera link and/or optical link...
+    <!---->
+    <xacro:logitech_c270_camera parent_link="camera_rig_bar" camera_link="driver_side_camera" joint_xyz="0.0 0.05 ${0.025 * 0.5}" joint_rpy="0 0 0"/>
+    <xacro:logitech_c270_camera parent_link="camera_rig_bar" camera_link="passenger_side_camera" joint_xyz="0.0 -0.05 ${0.025 * 0.5}" joint_rpy="0 0 0"/>
+    <!---->
 </robot>

File: src/models/scte_vehicle/scte_description/urdf/scte_wheel.xacro (robot description, xacro)
@@ -11,11 +11,5 @@
     flip
     ">
-            <gazebo reference="${link_name}">
-                <mu1 value="1.0"/>
-                <mu2 value="1.0"/>
-                <kp value="10000000.0" />
-                <kd value="1.0" />
-                <fdir1 value="1 0 0"/>
-            </gazebo>
+            <xacro:property name="wheel_friction" value="1.75" />
             <xacro:property name="wheel_radius_sq" value="${wheel_radius * wheel_radius}"/>
             <xacro:property name="wheel_length_sq" value="${wheel_length * wheel_length}"/>
@@ -52,4 +46,8 @@
                 <dynamics damping="0.7"/>
                 <limit effort="1000.0" velocity="22.0"/>
+                <gazebo reference="${wheel_joint_name}">
+                    <mu1>${wheel_friction}</mu1>
+                    <mu2>${wheel_friction}</mu2>
+                </gazebo>
             </joint>
             <xacro:if value="${is_steerable == 1}">
@@ -75,13 +73,4 @@
                 </joint>
             </xacro:if>
-            <!--transmission name="${link_name}_transmission" type="SimpleTransmission">
-                <type>transmission_interface/SimpleTransmission</type>
-                <actuator name="${link_name}_motor">
-                    <mechanicalReduction>1</mechanicalReduction>
-                </actuator>
-                <joint name="${wheel_joint_name}">
-                    <hardwareInterface>hardware_interface/VelocityJointInterface</hardwareInterface>
-                </joint>
-            </transmission-->
         </xacro:macro>
 </robot>
