Commit message: simplified xacro/urdf

File: src/models/scte_vehicle/scte_description/urdf/equipment/camera_rig.xacro (robot description, xacro)
@@ -7,5 +7,5 @@
         <link name="${link_name}_support">
             <inertial>
-                <mass value="${scte_chassis_mass * 0.01}"/>
+                <mass value="${base_mass * 0.01}"/>
                 <origin xyz="0 0 0" rpy="0 0 0"/>
                 <inertia
@@ -36,5 +36,5 @@
         <link name="${link_name}_bar">
             <inertial>
-                <mass value="${scte_chassis_mass * 0.01}"/>
+                <mass value="${base_mass * 0.01}"/>
                 <origin xyz="0 0 0" rpy="0 0 0"/>
                 <inertia

File: src/models/scte_vehicle/scte_description/urdf/equipment/computer_enclosure.xacro (robot description, xacro)
@@ -7,5 +7,5 @@
         <link name="${link_name}">
             <inertial>
-                <mass value="${scte_chassis_mass * 0.02}"/>
+                <mass value="${base_mass * 0.02}"/>
                 <origin xyz="0 0 0" rpy="0 0 0"/>
                 <inertia

File: src/models/scte_vehicle/scte_description/urdf/scte_chassis.xacro (robot description, xacro)
@@ -16,73 +16,75 @@
     lateral separation between the left and right front steering axes.
     For this model:
-    wheel_separation_h = base_length - 2 * axle_offset = 0.4
-    wheel_separation_w = base_width  + 2 * axle_offset = 0.4
+    wheel_separation_h = base_length - 2 * axle_offset = 0.442 - (2 * 0.05) = .342
+    wheel_separation_w = base_width  + 2 * axle_offset = 0.442 + (2 * 0.05) = .542
     Modified from the steer_bot example found here: https://github.com/srmainwaring/steer_bot
 -->
 <!--Gazebo does not seem to like capital letters in the robot namespace-->
-<robot name="sctebot" xmlns:xacro="http://www.ros.org/wiki/xacro">
+<robot name="scte_bot" xmlns:xacro="http://www.ros.org/wiki/xacro">
     <xacro:arg name="robot_namespace" default="/"/>
-    <xacro:arg name="tf_freq" default="100.0"/>
-    <xacro:arg name="pub_tf" default="true"/>
-    <xacro:property name="M_PI" value="3.14159265358979323846264338327950288"/>
+    <!-- ackermann components and gazebo plugins -->
     <xacro:include filename="$(find scte_description)/urdf/plugins/scte_plugins.gazebo" />
-    <xacro:include filename="plugins/scte_sensors.gazebo" />
-    <xacro:include filename="$(find scte_description)/urdf/materials.xacro" />
-    <xacro:include filename="$(find scte_description)/urdf/macros.xacro" />
-    <xacro:include filename="$(find ydlidar_ros)/urdf/ydlidar.urdf"/>
-    <xacro:include filename="$(find logitech_c270_camera)/urdf/logitech_c270.xacro"/>
-    <xacro:include filename="$(find scte_description)/urdf/equipment/mounting_bars.xacro"/>
-    <xacro:include filename="$(find scte_description)/urdf/equipment/computer_enclosure.xacro"/>
-    <xacro:include filename="$(find scte_description)/urdf/equipment/camera_rig.xacro"/>
-    <xacro:property name="scte_chassis_mass" value="2.9"/>
-    <xacro:property name="scte_chassis_length" value="0.292"/>
-    <xacro:property name="scte_chassis_width" value="0.165"/>
-    <xacro:property name="scte_chassis_depth" value="0.00635"/>
-    <xacro:property name="scte_chassis_length_sq" value="${scte_chassis_length * scte_chassis_length}"/>
-    <xacro:property name="scte_chassis_width_sq" value="${scte_chassis_width * scte_chassis_width}"/>
-    <xacro:property name="scte_chassis_depth_sq" value="${scte_chassis_depth * scte_chassis_depth}"/>
-    <!--Wheel Properties-->
-    <xacro:property name="wheel_mass" value="0.3"/>
+    <xacro:include filename="$(find scte_description)/urdf/scte_wheel.xacro"/>
+    <xacro:include filename="$(find scte_description)/urdf/scte_inertials.xacro"/>
+    <!-- sensor gazebo plugins -->
+    <xacro:include filename="$(find scte_description)/urdf/plugins/scte_sensors.gazebo" />
+    <!-- physical components -->
+    <!-- Math constants -->
     <xacro:property name="deg_to_rad" value="0.01745329251994329577"/>
-    <!-- Constants for robot dimensions -->
-    <xacro:property name="wheel_base" value="0.337"/>
-    <xacro:property name="wheel_track" value="0.251"/>
-    <xacro:property name="wheel_radius" value="0.0525" /> <!-- Link 1 -->
-    <xacro:property name="wheel_thickness" value="0.045" /> <!-- Link 2 -->
-    <xacro:property name="axel_offset" value="0.05" /> <!-- Space between top of beam and the each joint -->
-    <xacro:property name="steer_offset" value="0.02" /> <!-- Link 1 -->
-    <xacro:property name="shock_tower_height" value="0.105"/>
-    <xacro:property name="shock_tower_width" value="0.14"/>
-    <xacro:property name="drive_axle_length" value="0.25"/>
-    <xacro:property name="drive_axle_radius" value="0.005"/>
+    <!-- Robot base dimensions -->
+    <xacro:property name="base_length" value="0.442" /> <!-- wheel base derived from this -->
+    <xacro:property name="base_width" value="0.157" /> <!-- wheel track derived from this -->
+    <xacro:property name="base_height" value="0.01" />
+    <xacro:property name="base_mass" value="5" />
+    <!-- Wheel link dimensions -->
+    <xacro:property name="wheel_radius" value="0.0525" />
+    <xacro:property name="wheel_thickness" value="0.048" />
+    <xacro:property name="wheel_mass" value="1" />
+    <!-- Steering link dimensions -->
+    <xacro:property name="steer_radius" value="0.005" />
+    <xacro:property name="steer_thickness" value="0.02" />
+    <xacro:property name="steer_mass" value="1" />
+    <!-- Axle positions -->
+    <xacro:property name="axle_offset" value="0.05" />
+    <xacro:property name="steer_offset" value="0.02" />
+    <!-- scte dims -->
+    <xacro:property name="scte_chassis_length_sq" value="${base_length * base_length}"/>
+    <xacro:property name="scte_chassis_width_sq" value="${base_width * base_width}"/>
+    <xacro:property name="scte_chassis_height_sq" value="${base_height * base_height}"/>
+    <!-- base footprint for nav -->
     <link name='base_footprint'/>
     <joint name="base_link_TO_base_footprint" type="fixed">
-        <origin xyz="${scte_chassis_length * 0.63} 0 ${wheel_radius - scte_chassis_depth - 0.0075}" rpy="0 0 0"/>
+        <origin xyz="0 0 0" rpy="0 0 0"/>
         <parent link="base_footprint"/>
         <child link="base_link"/>
     </joint>
-    <link name='base_link'>
-        <visual name='visual'>
+    <!-- Base link -->
+    <link name="base_link">
+        <visual>
             <origin xyz="0 0 0" rpy="0 0 0"/>
             <geometry>
-                <box size="${scte_chassis_length} ${scte_chassis_width} ${scte_chassis_depth}"/>
+                <box size="${base_length} ${base_width} ${base_height}"/>
             </geometry>
-            <material name="blue"/>
+            <material name="green" />
         </visual>
-        <collision name='collision'>
+        <collision>
             <origin xyz="0 0 0" rpy="0 0 0"/>
             <geometry>
-                <box size="${scte_chassis_length} ${scte_chassis_width} ${scte_chassis_depth}"/>
+                <box size="${base_length} ${base_width} ${base_height}"/>
             </geometry>
         </collision>
+        <!--xacro:solid_cuboid_inertial
+                rpy="0 0 0" xyz="0 0 0"
+                mass="${base_mass}"
+                x="${base_length}" y="${base_width}" z="${base_height}" /-->
     </link>
     <!-- Inertial link stores the robot's inertial information -->
     <link name="inertial_link">
         <inertial>
-            <mass value="${scte_chassis_mass}" />
+            <mass value="${base_mass}" />
             <origin xyz="0 0 0" />
-            <inertia ixx="${(1/12 * scte_chassis_mass) * (scte_chassis_depth_sq + scte_chassis_width_sq)}" ixy="0" ixz="0"
-                     iyy="${(1/12 * scte_chassis_mass) * (scte_chassis_depth_sq + scte_chassis_length_sq)}" iyz="0"
-                     izz="${(1/12 * scte_chassis_mass) * (scte_chassis_length_sq + scte_chassis_width_sq)}" />
+            <inertia ixx="${(1/12 * base_mass) * (scte_chassis_height_sq + scte_chassis_width_sq)}" ixy="0" ixz="0"
+                     iyy="${(1/12 * base_mass) * (scte_chassis_height_sq + scte_chassis_length_sq)}" iyz="0"
+                     izz="${(1/12 * base_mass) * (scte_chassis_length_sq + scte_chassis_width_sq)}" />
         </inertial>
     </link>
@@ -92,207 +94,105 @@
         <child link="inertial_link" />
     </joint>
-    <!--CHASSIS-->
-    <link name="scte_chassis"/>
-    <joint name="scte_chassis_to_base_link_joint" type="fixed">
-        <origin xyz="0 0 0" rpy="0 0 0"/>
-        <parent link="base_link"/>
-        <child link="scte_chassis"/>
-    </joint>
-    <!---->
-    <xacro:include filename="$(find scte_description)/urdf/scte_diff_and_shock_tower.xacro"/>
-    <xacro:scte_diff_and_shock_tower
-        link_name="front_diff_tower"
-        parent_link="scte_chassis"
-        diff_joint_xyz="${scte_chassis_length * 0.63} 0 0"
-        diff_joint_rpy="0 0 0"
-        diff_plate_size="0.07 0.07 ${scte_chassis_depth}"
-        shock_tower_size="0.015 ${shock_tower_width} ${shock_tower_height}"
-        shock_tower_joint_origin="0 0 ${shock_tower_height * 0.5}"
-        shock_tower_joint_rpy="0 0 0"
-    />
-    <xacro:scte_diff_and_shock_tower
-        link_name="rear_diff_tower"
-        parent_link="scte_chassis"
-        diff_joint_xyz="${scte_chassis_length * -0.63} 0 0"
-        diff_joint_rpy="0 0 0"
-        diff_plate_size="0.07 0.07 ${scte_chassis_depth}"
-        shock_tower_size="0.015 ${shock_tower_width} ${shock_tower_height}"
-        shock_tower_joint_origin="0 0 ${shock_tower_height * 0.5}"
-        shock_tower_joint_rpy="0 0 0"
-    />
-    <!--TODO get rid of some of these magic number parameters -->
+    <!-- Front steer and rear wheel joints required for ackermann_steering_controller -->
+    <xacro:front_steer
+            name="front"
+            parent="base"
+            steer_radius="${steer_radius}"
+            steer_thickness="${steer_thickness}"
+            steer_mass="${steer_mass}"
+            base_length="${base_length}"
+            base_width="${base_width}"
+            axle_offset="${axle_offset}"
+            steer_height="${wheel_radius+steer_offset}">
+    </xacro:front_steer>
+    <xacro:rear_wheel
+            name="rear"
+            parent="base"
+            wheel_radius="${wheel_radius/4}"
+            wheel_thickness="${wheel_thickness/2}"
+            wheel_mass="${wheel_mass/32}">
+        <origin xyz="${-base_length/2+axle_offset} 0 0" rpy="${-90 * deg_to_rad} 0 0"/>
+    </xacro:rear_wheel>
+    <!-- Steerable front wheels -->
+    <xacro:front_wheel_lr
+            name="front_right"
+            parent="base"
+            reflect="-1"
+            wheel_radius="${wheel_radius}"
+            wheel_thickness="${wheel_thickness}"
+            wheel_mass="${wheel_mass}"
+            steer_radius="${steer_radius}"
+            steer_thickness="${steer_thickness}"
+            steer_mass="${steer_mass}"
+            base_length="${base_length}"
+            base_width="${base_width}"
+            axle_offset="${axle_offset}"
+            steer_height="${wheel_radius+steer_offset}">
+    </xacro:front_wheel_lr>
+    <xacro:front_wheel_lr
+            name="front_left"
+            parent="base"
+            reflect="1"
+            wheel_radius="${wheel_radius}"
+            wheel_thickness="${wheel_thickness}"
+            wheel_mass="${wheel_mass}"
+            steer_radius="${steer_radius}"
+            steer_thickness="${steer_thickness}"
+            steer_mass="${steer_mass}"
+            base_length="${base_length}"
+            base_width="${base_width}"
+            axle_offset="${axle_offset}"
+            steer_height="${wheel_radius+steer_offset}">
+    </xacro:front_wheel_lr>
+    <!-- Rear wheels -->
+    <xacro:rear_wheel_lr
+            name="rear_right"
+            parent="base"
+            wheel_radius="${wheel_radius}"
+            wheel_thickness="${wheel_thickness}"
+            wheel_mass="${wheel_mass}">
+        <origin xyz="${-base_length/2+axle_offset} ${-base_width/2-axle_offset} 0" rpy="${-90 * deg_to_rad} 0 0"/>
+    </xacro:rear_wheel_lr>
+    <xacro:rear_wheel_lr
+            name="rear_left"
+            parent="base"
+            wheel_radius="${wheel_radius}"
+            wheel_thickness="${wheel_thickness}"
+            wheel_mass="${wheel_mass}">
+        <origin xyz="${-base_length/2+axle_offset} ${+base_width/2+axle_offset} 0" rpy="${-90 * deg_to_rad} 0 0"/>
+    </xacro:rear_wheel_lr>
+    <!-- Bumpers -->
     <xacro:include filename="$(find scte_description)/urdf/scte_front_bumper.xacro"/>
     <xacro:scte_front_bumper
-        link_name="front_bumper"
-        parent_link="front_diff_tower"
-        front_skid_plate_size="0.07 0.07 ${scte_chassis_depth}"
-        front_skid_plate_joint_xyz="${0.07} 0 ${0.07 * 0.30}"
-        front_skid_plate_joint_rpy="0 ${M_PI/-6}  0"
-        front_bumper_size="0.01 0.175 0.05"
+            link_name="front_bumper"
+            parent_link="base_link"
+            front_skid_plate_size="0.07 0.07 ${0.0105}"
+            front_skid_plate_joint_xyz="${base_length * 0.5} 0 ${0.07 * 0.30}"
+            front_skid_plate_joint_rpy="0 ${pi/-6}  0"
+            front_bumper_size="0.01 0.175 0.05"
     />
     <xacro:include filename="$(find scte_description)/urdf/scte_rear_bumper.xacro"/>
     <xacro:scte_rear_bumper
-        link_name="rear_bumper"
-        parent_link="rear_diff_tower"
-        rear_bumper_size="0.01 0.255 0.05"
-        rear_bumper_mount_size="0.09 0.05 0.05"
-        rear_bumper_mount_joint_xyz="${0.09 * -0.6} 0 ${shock_tower_height * 0.5}"
-        rear_bumper_mount_joint_rpy="0 0 0"
-    />
-    <xacro:include filename="$(find scte_description)/urdf/scte_drive_axle.xacro"/>
-    <xacro:scte_drive_axle
-        link_name="front_axle"
-        parent_link="front_diff_tower"
-        drive_axle_radius="${drive_axle_radius}"
-        drive_axle_length="${drive_axle_length}"
-        drive_axle_joint_xyz="0 0 ${0.03 * 0.5}"
-        drive_axle_joint_rpy="${M_PI * -0.5} 0 0"
-    />
-    <xacro:scte_drive_axle
-        link_name="rear_axle"
-        parent_link="rear_diff_tower"
-        drive_axle_radius="${drive_axle_radius}"
-        drive_axle_length="${drive_axle_length}"
-        drive_axle_joint_xyz="0 0 ${0.03 * 0.5}"
-        drive_axle_joint_rpy="${M_PI * -0.5} 0 0"
-    />
-    <!-- Wheel macros for audibot implementation
-    <!XXxacro:include filename="$(find scte_description)/urdf/plugins/scte_audi_bot_plugin.gazebo"/XX>
-    <xacro:property name="wheel_length" value="0.47" /> <!XX separation between wheels? XX>
-    <xacro:property name="wheel_width" value="${0.20 - wheel_thickness}" /> <!XX separation between wheels? XX>
-    <xacro:include filename="$(find scte_description)/urdf/scte_wheel.xacro"/>
-    <xacro:scte_wheel
-        link_name="front_left_wheel"
-        parent_link="front_axle"
-        wheel_radius="${wheel_radius}"
-        wheel_length="${wheel_length}"
-        wheel_joint_origin="0 0 ${drive_axle_length * 0.5}"
-        wheel_joint_rpy="${M_PI * -0.5} 0 0"
-        wheel_joint_name="front_left_wheel_TO_front_axle"
-        wheel_steer_joint_name="front_left_wheel_steer_TO_front_axle"
-        is_steerable="true"
-        flip="1"
-    />
-    <xacro:scte_wheel
-        link_name="front_right_wheel"
-        parent_link="front_axle"
-        wheel_radius="${wheel_radius}"
-        wheel_length="${wheel_length}"
-        wheel_joint_origin="0 0 ${drive_axle_length * -0.5}"
-        wheel_joint_rpy="${M_PI * -0.5} 0 0"
-        wheel_joint_name="front_right_wheel_TO_front_axle"
-        wheel_steer_joint_name="front_right_wheel_steer_TO_front_axle"
-        is_steerable="true"
-        flip="-1"
-    />
-    <xacro:scte_wheel
-        link_name="rear_left_wheel"
-        parent_link="rear_axle"
-        wheel_radius="${wheel_radius}"
-        wheel_length="${wheel_length}"
-        wheel_joint_origin="0 0 ${drive_axle_length * 0.5}"
-        wheel_joint_rpy="0 0 0"
-        wheel_joint_name="rear_left_wheel_TO_rear_axle"
-        wheel_steer_joint_name=""
-        is_steerable="false"
-        flip="1"
-    />
-    <xacro:scte_wheel
-        link_name="rear_right_wheel"
-        parent_link="rear_axle"
-        wheel_radius="${wheel_radius}"
-        wheel_length="${wheel_length}"
-        wheel_joint_origin="0 0 ${drive_axle_length * -0.5}"
-        wheel_joint_rpy="0 0 0"
-        wheel_joint_name="rear_right_wheel_TO_rear_axle"
-        wheel_steer_joint_name=""
-        is_steerable="false"
-        flip="1"
-    />
-    -->
-    <xacro:include filename="$(find scte_description)/urdf/scte_wheel.xacro"/>
-    <!-- joints for ackermann_steering_controller -->
-    <xacro:front_steer
-        name="front"
-        parent="base"
-        radius="${wheel_radius}"
-        thickness="${wheel_thickness}"
-        length="${wheel_base}"
-        width="${wheel_track}"
-        axel_offset="${axel_offset}"
-        steer_height="${wheel_radius+steer_offset}">
-        <!--origin xyz="${wheel_base/2-axel_offset} 0 0" rpy="${-90 * deg_to_rad} 0 0"/-->
-    </xacro:front_steer>
-    <!-- the "fake" rear wheel -->
-    <xacro:rear_wheel
-        name="rear"
-        parent="base"
-        radius="${wheel_radius}"
-        thickness="${wheel_thickness}">
-        <origin xyz="${-wheel_base/2+axel_offset} 0 0" rpy="${-90 * deg_to_rad} 0 0"/>
-    </xacro:rear_wheel>
-    <!-- Wheels -->
-    <xacro:front_wheel_lr
-        name="front_right"
-        parent="base"
-        radius="${wheel_radius}"
-        thickness="${wheel_thickness}"
-        length="${wheel_base}"
-        width="${wheel_track}"
-        axel_offset="${axel_offset}"
-        right_left="-1"
-        steer_height="${wheel_radius+steer_offset}">
-        <!--origin xyz="${wheel_base/2-axel_offset} ${wheel_track/2+axel_offset} ${scte_chassis_depth * -0.5}" rpy="${-90 * deg_to_rad} 0 0"/-->
-    </xacro:front_wheel_lr>
-    <xacro:front_wheel_lr
-        name="front_left"
-        parent="base"
-        radius="${wheel_radius}"
-        thickness="${wheel_thickness}"
-        length="${wheel_base}"
-        width="${wheel_track}"
-        axel_offset="${axel_offset}"
-        right_left="1"
-        steer_height="${wheel_radius+steer_offset}">
-        <!--origin xyz="${wheel_base/2-axel_offset} ${-wheel_track/2-axel_offset} ${scte_chassis_depth * -0.5}" rpy="${-90 * deg_to_rad} 0 0"/-->
-    </xacro:front_wheel_lr>
-    <xacro:rear_wheel_lr
-        name="rear_left"
-        parent="base"
-        radius="${wheel_radius}"
-        thickness="${wheel_thickness}">
-        <origin xyz="${-wheel_base/2+axel_offset} ${wheel_track/2+axel_offset} ${scte_chassis_depth * -0.5}" rpy="${-90 * deg_to_rad} 0 0"/>
-    </xacro:rear_wheel_lr>
-    <xacro:rear_wheel_lr
-        name="rear_right"
-        parent="base"
-        radius="${wheel_radius}"
-        thickness="${wheel_thickness}">
-        <origin xyz="${-wheel_base/2+axel_offset} ${-wheel_track/2-axel_offset} ${scte_chassis_depth * -0.5}" rpy="${-90 * deg_to_rad} 0 0"/>
-    </xacro:rear_wheel_lr>
-    <!-- mounting hardware -->
-    <xacro:mounting_bar
-        link_name="driver_mounting_bar"
-        parent_link="front_diff_tower"
-        bar_origin="${scte_chassis_length * -0.63} ${shock_tower_width * 0.5} ${shock_tower_height * 1.0}"
-        bar_rpy="0 0 0"
-    />
-    <xacro:mounting_bar
-        link_name="passenger_mounting_bar"
-        parent_link="front_diff_tower"
-        bar_origin="${scte_chassis_length * -0.63} ${shock_tower_width * -0.5} ${shock_tower_height * 1.0}"
-        bar_rpy="0 0 0"
-    />
+            link_name="rear_bumper"
+            parent_link="base_link"
+            rear_bumper_size="0.01 0.255 0.05"
+            rear_bumper_mount_size="0.09 0.05 0.05"
+            rear_bumper_mount_joint_xyz="${base_length * -0.6} 0 ${0.105 * 0.5}"
+            rear_bumper_mount_joint_rpy="0 0 0"
+    />
+    <!-- Sensors and Compute Hardware -->
+    <xacro:include filename="$(find scte_description)/urdf/equipment/computer_enclosure.xacro"/>
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
File: src/models/scte_vehicle/scte_description/urdf/scte_front_bumper.xacro (robot description, xacro)
@@ -56,5 +56,5 @@
         </link>
         <joint name="${link_name}_TO_${parent_link}" type="fixed">
-            <origin xyz="${0.07 * 0.70} 0 ${0.07 * 0.35}" rpy="0 ${M_PI/6} 0"/>
+            <origin xyz="${0.07 * 0.70} 0 ${0.07 * 0.35}" rpy="0 ${pi/6} 0"/>
             <parent link="${link_name}_skid_plate"/>
             <child link="${link_name}"/>
