Commit message: navsat map node working I think. fine tuning the ackermann odom rates

File: sctebot_description/urdf/sctebot_chassis.xacro (robot description, xacro)
@@ -197,5 +197,5 @@
             camera_rig_rpy="0 0 0"
     />
-    <!-- Sim IMU -->
+    <!-- imu link -->
     <link name="imu_link"/>
     <joint name="imu_link_TO_computer_enclosure" type="fixed">
@@ -203,4 +203,11 @@
         <parent link="computer_enclosure"/>
         <child link="imu_link"/>
+    </joint>
+    <!-- gps link -->
+    <link name="gps_link"/>
+    <joint name="gps_link_TO_computer_enclosure" type="fixed">
+        <origin xyz="0 0 0" rpy="0 0 0"/>
+        <parent link="computer_enclosure"/>
+        <child link="gps_link"/>
     </joint>
     <!-- LIDAR -->

File: sctebot_description/urdf/sctebot_sensors.xacro (robot description, xacro)
@@ -1,28 +1,28 @@
 <?xml version="1.0"?>
 <robot xmlns:xacro="http://www.ros.org/wiki/xacro">
-    <!--gazebo reference is the link the sensor is attached to it seems-->
-    <!---->
-    <gazebo reference="base_link">
-        <gravity>true</gravity>
-        <sensor name="imu_sensor" type="imu">
-          <always_on>true</always_on>
-          <update_rate>100</update_rate>
-          <visualize>true</visualize>
-          <topic>__default_topic__</topic>
-          <plugin filename="libgazebo_ros_imu_sensor.so" name="imu_plugin">
-            <robotNamespace>$(arg robot_namespace)</robotNamespace>
-            <topicName>imu</topicName>
-            <bodyName>imu_link</bodyName>
-            <frameName>imu_link</frameName>
-            <updateRateHZ>50.0</updateRateHZ>
-            <gaussianNoise>0.0</gaussianNoise>
-            <xyzOffset>0 0 0</xyzOffset>
-            <rpyOffset>0 0 0</rpyOffset>
-            <initialOrientationAsReference>false</initialOrientationAsReference>
-          </plugin>
-          <pose>0 0 0 0 0 0</pose>
-        </sensor>
-    </gazebo>
-    <!---->
+  <!--gazebo reference is the link the sensor is attached to it seems-->
+  <!---->
+  <gazebo reference="base_link">
+    <gravity>true</gravity>
+      <sensor name="imu_sensor" type="imu">
+        <always_on>true</always_on>
+        <update_rate>100</update_rate>
+        <visualize>true</visualize>
+        <topic>__default_topic__</topic>
+        <plugin filename="libgazebo_ros_imu_sensor.so" name="imu_plugin">
+          <robotNamespace>$(arg robot_namespace)</robotNamespace>
+          <topicName>imu</topicName>
+          <bodyName>imu_link</bodyName>
+          <frameName>imu_link</frameName>
+          <updateRateHZ>50.0</updateRateHZ>
+          <gaussianNoise>0.0</gaussianNoise>
+          <xyzOffset>0 0 0</xyzOffset>
+          <rpyOffset>0 0 0</rpyOffset>
+          <initialOrientationAsReference>false</initialOrientationAsReference>
+        </plugin>
+        <pose>0 0 0 0 0 0</pose>
+      </sensor>
+  </gazebo>
+  <!---->
   <gazebo>
     <plugin name="hector_gps" filename="libhector_gazebo_ros_gps.so">
@@ -30,13 +30,13 @@
       <robotNamespace>$(arg robot_namespace)</robotNamespace>
       <bodyName>base_link</bodyName>
-      <frameId>map</frameId>
-      <topicName>gps/fix</topicName>
-      <velocityTopicName>gps/fix_velocity</velocityTopicName>
+      <frameId>gps_link</frameId>
+      <topicName>hector_sim/gps/fix</topicName>
+      <velocityTopicName>hector_sim/gps/fix_velocity</velocityTopicName>
       <referenceLatitude>32.75394484000334</referenceLatitude>
       <referenceLongitude>-117.21848979362261</referenceLongitude>
       <referenceHeading>0.0</referenceHeading>
       <referenceLatitude>0.0</referenceLatitude>
-      <status>STATUS_FIX</status>
-      <service>SERVICE_GPS</service>
+      <!--status>STATUS_FIX</status>
+      <service>SERVICE_GPS</service-->
       <drift>5.0 5.0 5.0</drift>
       <drifFrequency>0.0 0.0 0.0</drifFrequency>
@@ -48,96 +48,96 @@
     </plugin>
   </gazebo>
-    <!--
-        - Noise is sampled independently per pixel on each frame.
-        That pixel's noise value is added to each of its color
-        channels, which at that point lie in the range [0,1].
-        - ROS and gazebo use different camera axis conventions,
-        this may cause the virtual camera to point in the wrong direction
-    -->
-    <!--
-    <gazebo reference="driver_side_camera_base">
-        <sensor type="camera" name="driver_camera">
-          <visualize>true</visualize>
-          <update_rate>30.0</update_rate>
-          <camera name="head">
-            <horizontal_fov>1.43</horizontal_fov>
-            <image>
-              <width>320</width>
-              <height>240</height>
-              <format>R8G8B8</format>
-            </image>
-            <clip>
-              <near>0.02</near>
-              <far>300</far>
-            </clip>
-            <noise>
-              <type>gaussian</type>
-              <mean>0.0</mean>
-              <stddev>0.007</stddev>
-            </noise>
-          </camera>
-          <plugin name="camera_controller" filename="libgazebo_ros_camera.so">
-            <robotNamespace>$(arg robot_namespace)</robotNamespace>
-            <alwaysOn>true</alwaysOn>
-            <updateRate>10.0</updateRate>
-            <cameraName>driver_camera</cameraName>
-            <imageTopicName>image_raw</imageTopicName>
-            <cameraInfoTopicName>camera_info</cameraInfoTopicName>
-            <frameName>driver_side_camera_base</frameName>
-            <hackBaseline>0.07</hackBaseline>
-            <distortionK1>0.0</distortionK1>
-            <distortionK2>0.0</distortionK2>
-            <distortionK3>0.0</distortionK3>
-            <distortionT1>0.0</distortionT1>
-            <distortionT2>0.0</distortionT2>
-          </plugin>
-        </sensor>
-    </gazebo>
-    -->
-    <!--
-    <gazebo reference="passenger_side_camera_base">
-        <sensor type="camera" name="passenger_camera">
-          <visualize>true</visualize>
-          <update_rate>30.0</update_rate>
-          <camera name="head">
-            <horizontal_fov>1.43</horizontal_fov>
-            <image>
-              <width>320</width>
-              <height>240</height>
-              <format>R8G8B8</format>
-            </image>
-            <clip>
-              <near>0.02</near>
-              <far>300</far>
-            </clip>
-            <noise>
-              <type>gaussian</type>
-              <mean>0.0</mean>
-              <stddev>0.007</stddev>
-            </noise>
-          </camera>
-          <plugin name="camera_controller" filename="libgazebo_ros_camera.so">
-            <robotNamespace>$(arg robot_namespace)</robotNamespace>
-            <alwaysOn>true</alwaysOn>
-            <updateRate>10.0</updateRate>
-            <cameraName>passenger_camera</cameraName>
-            <imageTopicName>image_raw</imageTopicName>
-            <cameraInfoTopicName>camera_info</cameraInfoTopicName>
-            <frameName>passenger_side_camera_base</frameName>
-            <hackBaseline>0.07</hackBaseline>
-            <distortionK1>0.0</distortionK1>
-            <distortionK2>0.0</distortionK2>
-            <distortionK3>0.0</distortionK3>
-            <distortionT1>0.0</distortionT1>
-            <distortionT2>0.0</distortionT2>
-          </plugin>
-        </sensor>
-    </gazebo>
-    -->
+  <!--
+  - Noise is sampled independently per pixel on each frame.
+  That pixel's noise value is added to each of its color
+  channels, which at that point lie in the range [0,1].
+  - ROS and gazebo use different camera axis conventions,
+  this may cause the virtual camera to point in the wrong direction
+  -->
+  <!--
+  <gazebo reference="driver_side_camera_base">
+    <sensor type="camera" name="driver_camera">
+      <visualize>true</visualize>
+      <update_rate>30.0</update_rate>
+      <camera name="head">
+        <horizontal_fov>1.43</horizontal_fov>
+        <image>
+          <width>320</width>
+          <height>240</height>
+          <format>R8G8B8</format>
+        </image>
+        <clip>
+          <near>0.02</near>
+          <far>300</far>
+        </clip>
+        <noise>
+          <type>gaussian</type>
+          <mean>0.0</mean>
+          <stddev>0.007</stddev>
+        </noise>
+      </camera>
+      <plugin name="camera_controller" filename="libgazebo_ros_camera.so">
+        <robotNamespace>$(arg robot_namespace)</robotNamespace>
+        <alwaysOn>true</alwaysOn>
+        <updateRate>10.0</updateRate>
+        <cameraName>driver_camera</cameraName>
+        <imageTopicName>image_raw</imageTopicName>
+        <cameraInfoTopicName>camera_info</cameraInfoTopicName>
+        <frameName>driver_side_camera_base</frameName>
+        <hackBaseline>0.07</hackBaseline>
+        <distortionK1>0.0</distortionK1>
+        <distortionK2>0.0</distortionK2>
+        <distortionK3>0.0</distortionK3>
+        <distortionT1>0.0</distortionT1>
+        <distortionT2>0.0</distortionT2>
+      </plugin>
+    </sensor>
+  </gazebo>
+  -->
+  <!--
+  <gazebo reference="passenger_side_camera_base">
+    <sensor type="camera" name="passenger_camera">
+      <visualize>true</visualize>
+      <update_rate>30.0</update_rate>
+      <camera name="head">
+      <horizontal_fov>1.43</horizontal_fov>
+        <image>
+          <width>320</width>
+          <height>240</height>
+          <format>R8G8B8</format>
+        </image>
+        <clip>
+          <near>0.02</near>
+          <far>300</far>
+        </clip>
+        <noise>
+          <type>gaussian</type>
+          <mean>0.0</mean>
+          <stddev>0.007</stddev>
+        </noise>
+      </camera>
+      <plugin name="camera_controller" filename="libgazebo_ros_camera.so">
+        <robotNamespace>$(arg robot_namespace)</robotNamespace>
+        <alwaysOn>true</alwaysOn>
+        <updateRate>10.0</updateRate>
+        <cameraName>passenger_camera</cameraName>
+        <imageTopicName>image_raw</imageTopicName>
+        <cameraInfoTopicName>camera_info</cameraInfoTopicName>
+        <frameName>passenger_side_camera_base</frameName>
+        <hackBaseline>0.07</hackBaseline>
+        <distortionK1>0.0</distortionK1>
+        <distortionK2>0.0</distortionK2>
+        <distortionK3>0.0</distortionK3>
+        <distortionT1>0.0</distortionT1>
+        <distortionT2>0.0</distortionT2>
+      </plugin>
+    </sensor>
+  </gazebo>
+  -->
   <!-- hokuyo
-    Noise parameters based on published spec for Hokuyo laser
-    achieving "+-30mm" accuracy at range < 10m.  A mean of 0.0m and
-    stddev of 0.01m will put 99.7% of samples within 0.03m of the true
-    reading.
+  Noise parameters based on published spec for Hokuyo laser
+  achieving "+-30mm" accuracy at range < 10m.  A mean of 0.0m and
+  stddev of 0.01m will put 99.7% of samples within 0.03m of the true
+  reading.
   -->
   <!--
@@ -150,8 +150,8 @@
         <scan>
           <horizontal>
-            <samples>5000</samples>
-            <resolution>1</resolution>
-            <min_angle>${pi * -1.0}</min_angle>
-            <max_angle>${pi * 1.0}</max_angle>
+          <samples>5000</samples>
+          <resolution>1</resolution>
+          <min_angle>${pi * -1.0}</min_angle>
+          <max_angle>${pi * 1.0}</max_angle>
           </horizontal>
         </scan>

Commit message: added realsense camera launch files and added model to xacro

File: sctebot_description/urdf/sctebot_chassis.xacro (robot description, xacro)
@@ -233,4 +233,9 @@
     <xacro:logitech_c270_camera parent_link="camera_rig_bar" camera_link="passenger_side_camera" joint_xyz="0.0 -0.05 ${0.025 * 0.5}" joint_rpy="0 0 0"/>
     <!---->
+    <!-- intel Realsense d455 -->
+    <xacro:include filename="$(find realsense2_description)/urdf/_d435i.urdf.xacro"/>
+    <xacro:sensor_d435i parent="computer_enclosure" name="d455">
+        <origin xyz="0 0 0.25" rpy="0 0 0"/>
+    </xacro:sensor_d435i>
     <!-- Colour -->
     <gazebo reference="base_link">

Commit message: working on integrating sensors for localization

File: sctebot_description/urdf/sctebot_chassis.xacro (robot description, xacro)
@@ -215,5 +215,5 @@
     <xacro:include filename="$(find ydlidar_ros)/urdf/ydlidar.urdf"/>
     <joint name="ydlidar_base_TO_computer_enclosure" type="fixed">
-        <origin xyz="0.090 0 0.0305" rpy="0 0 0"/>
+        <origin xyz="0.090 0 0.0305" rpy="0 0 0"/> <!--0.0305-->
         <parent link="computer_enclosure"/>
         <child link="base_laser"/>
@@ -235,6 +235,6 @@
     <!-- intel Realsense d455 -->
     <xacro:include filename="$(find realsense2_description)/urdf/_d435i.urdf.xacro"/>
-    <xacro:sensor_d435i parent="computer_enclosure" name="d455">
-        <origin xyz="0 0 0.25" rpy="0 0 0"/>
+    <xacro:sensor_d435i parent="camera_rig_bar" name="d455">
+        <origin xyz="0 0 0" rpy="0 0 0"/>
     </xacro:sensor_d435i>
     <!-- Colour -->

File: sctebot_description/urdf/sctebot_sensors.xacro (robot description, xacro)
@@ -2,5 +2,5 @@
 <robot xmlns:xacro="http://www.ros.org/wiki/xacro">
   <!--gazebo reference is the link the sensor is attached to it seems-->
-  <!---->
+  <!--
   <gazebo reference="imu_link">
     <gravity>true</gravity>
@@ -15,5 +15,5 @@
           <bodyName>imu_link</bodyName>
           <frameName>imu_link</frameName>
-          <updateRateHZ>50.0</updateRateHZ>
+          <updateRateHZ>400.0</updateRateHZ>
           <gaussianNoise>0.0</gaussianNoise>
           <xyzOffset>0 0 0</xyzOffset>
@@ -24,5 +24,5 @@
       </sensor>
   </gazebo>
-  <!---->
+  -->
   <gazebo>
     <plugin name="hector_gps" filename="libhector_gazebo_ros_gps.so">
@@ -198,5 +198,5 @@
   reading.
   -->
-  <!---->
+  <!--
   <gazebo reference="laser_frame">
     <sensor type="ray" name="head_hokuyo_sensor">
@@ -231,4 +231,4 @@
     </sensor>
   </gazebo>
-  <!---->
+  -->
 </robot>

Commit message: got rid of footprint since RViz was complaining about it

File: sctebot_description/urdf/sctebot_chassis.xacro (robot description, xacro)
@@ -59,10 +59,10 @@
     <xacro:property name="scte_chassis_height_sq" value="${base_height * base_height}"/>
     <!-- base footprint for nav -->
-    <link name='base_footprint'/>
+    <!--link name='base_footprint'/>
     <joint name="base_link_TO_base_footprint" type="fixed">
         <origin xyz="0 0 0" rpy="0 0 0"/>
         <parent link="base_footprint"/>
         <child link="base_link"/>
-    </joint>
+    </joint-->
     <!-- Base link -->
     <link name="base_link">

Commit message: add base_footprint back into chassis xarco, update robot localization yamls to match. Testing ROS navigation, requires a base_footprint

File: sctebot_description/urdf/sctebot_chassis.xacro (robot description, xacro)
@@ -59,14 +59,14 @@
     <xacro:property name="scte_chassis_height_sq" value="${base_height * base_height}"/>
     <!-- base footprint for nav -->
-    <!--link name='base_footprint'/>
+    <link name='base_footprint'/>
     <joint name="base_link_TO_base_footprint" type="fixed">
         <origin xyz="0 0 0" rpy="0 0 0"/>
         <parent link="base_footprint"/>
         <child link="base_link"/>
-    </joint-->
+    </joint>
     <!-- Base link -->
     <link name="base_link">
         <visual>
-            <origin xyz="0 0 0" rpy="0 0 0"/>
+            <origin xyz="0 0 ${wheel_radius * 2.0}" rpy="0 0 0"/>
             <geometry>
                 <box size="${base_length} ${base_width} ${base_height}"/>
@@ -75,5 +75,5 @@
         </visual>
         <collision>
-            <origin xyz="0 0 0" rpy="0 0 0"/>
+            <origin xyz="0 0 ${wheel_radius * 2.0}" rpy="0 0 0"/>
             <geometry>
                 <box size="${base_length} ${base_width} ${base_height}"/>

Commit message: adjust steerbot odom to use velocity instead of position per doc regarding how to fuse odom info that says to favor velocity over postion

File: sctebot_description/urdf/sctebot_chassis.xacro (robot description, xacro)
@@ -17,5 +17,5 @@
     For this model:
     wheel_separation_h = base_length - 2 * axle_offset = 0.442 - (2 * 0.05) = .342
-    wheel_separation_w = base_width  + 2 * axle_offset = 0.442 + (2 * 0.05) = .542
+    wheel_separation_w = base_width  + 2 * axle_offset = 0.157 + (2 * 0.05) = .257
     Modified from the steer_bot example found here: https://github.com/srmainwaring/steer_bot
 -->
@@ -39,5 +39,5 @@
     <!-- region Robot base dimensions -->
     <xacro:property name="base_length" value="0.442" /> <!-- wheel base derived from this -->
-    <xacro:property name="base_width" value="0.157" /> <!-- wheel track derived from this -->
+    <xacro:property name="base_width" value="0.157" />  <!-- wheel track derived from this -->
     <xacro:property name="base_height" value="0.01" />
     <xacro:property name="base_mass" value="5" />
