Commit message: relocate the realsense sensor to match where it is on the hardware. cleaned up xacro files.

File: sctebot_description/urdf/equipment/camera_rig.xacro (robot description, xacro)
@@ -1,7 +1,7 @@
 <?xml version="1.0"?>
 <robot name="sctebot" xmlns:xacro="http://www.ros.org/wiki/xacro">
-    <xacro:macro name="camera_rig" params="link_name parent_link
-    camera_rig_origin
-    camera_rig_rpy
+    <xacro:macro
+            name="camera_rig"
+            params="link_name parent_link camera_rig_origin camera_rig_rpy
     ">
         <link name="${link_name}_support">

File: sctebot_description/urdf/sctebot_chassis.xacro (robot description, xacro)
@@ -23,19 +23,26 @@
 <robot name="sctebot" xmlns:xacro="http://www.ros.org/wiki/xacro">
     <xacro:arg name="robot_namespace" default="/"/>
+    <xacro:arg name="enable_gazebo_stereo_camera" default="True"/>
+    <xacro:arg name="enable_logitech_stereo_camera" default="False"/>
+    <xacro:arg name="enable_realsense_d435i_stereo_camera" default="True"/>
+    <xacro:arg name="enable_ydlidar" default="True"/>
     <!-- ackermann components and gazebo plugins -->
-    <xacro:include filename="$(find sctebot_description)/urdf/plugins/sctebot_plugins.gazebo" />
+    <xacro:include filename="$(find sctebot_description)/urdf/plugins/sctebot_plugins.gazebo"/>
     <xacro:include filename="$(find sctebot_description)/urdf/sctebot_wheel.xacro"/>
     <xacro:include filename="$(find sctebot_description)/urdf/sctebot_inertials.xacro"/>
     <xacro:include filename="$(find sctebot_description)/urdf/sctebot_materials.xacro"/>
     <!-- sensor gazebo plugins -->
-    <xacro:include filename="$(find sctebot_description)/urdf/sctebot_sensors.xacro" />
+    <xacro:include filename="$(find sctebot_description)/urdf/sctebot_sensors.xacro">
+        <!--xacro:arg name="gazebo_stereo_camera_name" value="${gazebo_stereo_camera_name}"/-->
+    </xacro:include>
     <!-- physical components -->
     <!-- Math constants -->
     <xacro:property name="deg_to_rad" value="0.01745329251994329577"/>
-    <!-- Robot base dimensions -->
+    <!-- region Robot base dimensions -->
     <xacro:property name="base_length" value="0.442" /> <!-- wheel base derived from this -->
     <xacro:property name="base_width" value="0.157" /> <!-- wheel track derived from this -->
     <xacro:property name="base_height" value="0.01" />
     <xacro:property name="base_mass" value="5" />
+    <!-- endregion -->
     <!-- Wheel link dimensions -->
     <xacro:property name="wheel_radius" value="0.0525" />
@@ -190,12 +197,5 @@
             enclosure_rpy="0 0 0"
     />
-    <xacro:include filename="$(find sctebot_description)/urdf/equipment/camera_rig.xacro"/>
-    <xacro:camera_rig
-            link_name="camera_rig"
-            parent_link="computer_enclosure"
-            camera_rig_origin="${0.260 * -0.45} 0 ${0.06 * 1.0}"
-            camera_rig_rpy="0 0 0"
-    />
-    <!-- simulated imu link -->
+    <!-- region IMU link -->
     <link name="imu_link"/>
     <joint name="imu_link_TO_computer_enclosure" type="fixed">
@@ -204,5 +204,6 @@
         <child link="imu_link"/>
     </joint>
-    <!-- gps link -->
+    <!-- endregion -->
+    <!-- region GPS link -->
     <link name="gps_link"/>
     <joint name="gps_link_TO_computer_enclosure" type="fixed">
@@ -211,14 +212,25 @@
         <child link="gps_link"/>
     </joint>
-    <!-- LIDAR -->
-    <!---->
-    <xacro:include filename="$(find ydlidar_ros)/urdf/ydlidar.urdf"/>
-    <joint name="ydlidar_base_TO_computer_enclosure" type="fixed">
-        <origin xyz="0.090 0 0.0305" rpy="0 0 0"/> <!--0.0305-->
-        <parent link="computer_enclosure"/>
-        <child link="base_laser"/>
-    </joint>
-    <!---->
-    <!-- Cameras -->
+    <!-- endregion -->
+    <!-- region YDLIDAR link -->
+    <xacro:if value="$(arg enable_ydlidar)">
+        <xacro:include filename="$(find ydlidar_ros)/urdf/ydlidar.urdf"/>
+        <joint name="ydlidar_base_TO_computer_enclosure" type="fixed">
+            <origin xyz="0.090 0 0.0305" rpy="0 0 0"/> <!--0.0305-->
+            <parent link="computer_enclosure"/>
+            <child link="base_laser"/>
+        </joint>
+    </xacro:if>
+    <!-- endregion -->
+    <!-- region Stereo Cameras -->
+    <!-- region Realsense d435i Stereo Camera -->
+    <xacro:if value="$(arg enable_realsense_d435i_stereo_camera)">
+        <xacro:include filename="$(find realsense2_description)/urdf/_d435i.urdf.xacro"/>
+        <xacro:sensor_d435i parent="computer_enclosure" name="realsense_d435i">
+            <origin xyz="${(0.26 * 0.5) + (0.02505 * 0.5)} 0 0.005" rpy="0 0 0"/>
+        </xacro:sensor_d435i>
+    </xacro:if>
+    <!-- endregion -->
+    <!-- region Logitech Stereo Cameras -->
     <!--
         https://answers.ros.org/question/9840/how-do-you-get-stereo_image_proc-to-include-a-frame_id-so-that-rviz-will-accept-the-point-cloud-messages/
@@ -226,19 +238,41 @@
         may need to use image_rect for the video to align with the model
         https://berndpfrommer.github.io/tagslam_web/visualization/
+        TODO drowan_20220709_BUG: The cameras are mounted incorrectly. Need to fix camera link and/or optical link...
     -->
-    <!--TODO drowan_20210117_BUG: The cameras are mounted sideways. Need to fix camera link and/or optical link...-->
-    <!---->
-    <xacro:include filename="$(find logitech_c270_camera)/urdf/logitech_c270.xacro"/>
-    <xacro:logitech_c270_camera parent_link="camera_rig_bar" camera_link="driver_side_camera" joint_xyz="0.0 0.05 ${0.025 * 0.5}" joint_rpy="0 0 0"/>
-    <xacro:logitech_c270_camera parent_link="camera_rig_bar" camera_link="passenger_side_camera" joint_xyz="0.0 -0.05 ${0.025 * 0.5}" joint_rpy="0 0 0"/>
-    <!---->
-    <!--
-    intel Realsense d455
-    d455_link
-    -->
-    <xacro:include filename="$(find realsense2_description)/urdf/_d435i.urdf.xacro"/>
-    <xacro:sensor_d435i parent="camera_rig_bar" name="realsense_d435i">
-        <origin xyz="0 0 0" rpy="0 0 0"/>
-    </xacro:sensor_d435i>
+    <xacro:if value="$(arg enable_logitech_stereo_camera)">
+        <xacro:include filename="$(find sctebot_description)/urdf/equipment/camera_rig.xacro"/>
+        <xacro:camera_rig
+                link_name="camera_rig"
+                parent_link="computer_enclosure"
+                camera_rig_origin="${0.260 * -0.45} 0 ${0.06 * -0.04}"
+                camera_rig_rpy="0 0 ${pi}"
+        />
+        <xacro:include filename="$(find logitech_c270_camera)/urdf/logitech_c270.xacro"/>
+        <xacro:logitech_c270_camera
+                parent_link="camera_rig_bar"
+                camera_link="logitech_driver_side_camera"
+                joint_xyz="0.0 0.05 ${0.025 * 0.5}"
+                joint_rpy="0 0 0"
+        />
+        <xacro:logitech_c270_camera
+                parent_link="camera_rig_bar"
+                camera_link="logitech_passenger_side_camera"
+                joint_xyz="0.0 -0.05 ${0.025 * 0.5}"
+                joint_rpy="0 0 0"
+        />
+    </xacro:if>
+    <!-- endregion -->
+    <!-- region Gazebo Stereo Camera Sensor -->
+    <xacro:if value="$(arg enable_gazebo_stereo_camera)">
+        <xacro:include filename="$(find sctebot_description)/urdf/gazebo_sensors/gazebo_stereo_camera.xacro"/>
+        <xacro:gazebo_stereo_camera
+                parent_link="computer_enclosure"
+                camera_link="gazebo_stereo_camera"
+                joint_xyz="${(0.26 * 0.5) + (0.02505 * 0.5)} 0 0.018"
+                joint_rpy="0.0 0.0 0.0"
+        />
+    </xacro:if>
+    <!-- endregion -->
+    <!-- endregion -->
     <!-- Colour -->
     <gazebo reference="base_link">

File: sctebot_description/urdf/sctebot_sensors.xacro (robot description, xacro)
@@ -2,5 +2,5 @@
 <robot xmlns:xacro="http://www.ros.org/wiki/xacro">
   <!--gazebo reference is the link the sensor is attached to it seems-->
-  <!---->
+  <!-- region IMU -->
   <gazebo reference="imu_link">
     <gravity>true</gravity>
@@ -24,5 +24,6 @@
       </sensor>
   </gazebo>
-  <!---->
+  <!-- endregion -->
+  <!-- region GPS -->
   <gazebo>
     <plugin name="hector_gps" filename="libhector_gazebo_ros_gps.so">
@@ -48,4 +49,6 @@
     </plugin>
   </gazebo>
+  <!-- endregion -->
+  <!-- region Right and Left Cameras -->
   <!--
   - Noise is sampled independently per pixel on each frame.
@@ -55,6 +58,6 @@
   this may cause the virtual camera to point in the wrong direction
   -->
-  <!--
-  <gazebo reference="driver_side_camera_base">
+  <!---->
+  <gazebo reference="logitech_driver_side_camera_base">
     <sensor type="camera" name="driver_camera">
       <visualize>true</visualize>
@@ -80,8 +83,8 @@
         <alwaysOn>true</alwaysOn>
         <updateRate>10.0</updateRate>
-        <cameraName>stereo_fwd/camera/left</cameraName>
+        <cameraName>logitech_stereo_rear/camera/left</cameraName>
         <imageTopicName>image_raw</imageTopicName>
         <cameraInfoTopicName>camera_info</cameraInfoTopicName>
-        <frameName>/driver_side_camera_optical</frameName>
+        <frameName>logitech_driver_side_camera_optical</frameName>
         <hackBaseline>0.07</hackBaseline>
         <distortionK1>0.0</distortionK1>
@@ -93,7 +96,7 @@
     </sensor>
   </gazebo>
-  -->
-  <!--
-  <gazebo reference="passenger_side_camera_base">
+  <!---->
+  <!---->
+  <gazebo reference="logitech_passenger_side_camera_base">
     <sensor type="camera" name="passenger_camera">
       <visualize>true</visualize>
@@ -119,8 +122,8 @@
         <alwaysOn>true</alwaysOn>
         <updateRate>10.0</updateRate>
-        <cameraName>stereo_fwd/camera/right</cameraName>
+        <cameraName>logitech_stereo_rear/camera/right</cameraName>
         <imageTopicName>image_raw</imageTopicName>
         <cameraInfoTopicName>camera_info</cameraInfoTopicName>
-        <frameName>/passenger_side_camera_optical</frameName>
+        <frameName>logitech_passenger_side_camera_optical</frameName>
         <hackBaseline>0.07</hackBaseline>
         <distortionK1>0.0</distortionK1>
@@ -132,16 +135,19 @@
     </sensor>
   </gazebo>
-  -->
-  <!--
-  Stereo camera plugin
-  -->
-  <gazebo reference="driver_side_camera_base">
+  <!---->
+  <!-- endregion -->
+  <!-- region "Realsense" Stereo Camera -->
+  <xacro:property name="gazebo_stereo_camera_name" default="gazebo_stereo_camera"/>
+  <gazebo reference="${gazebo_stereo_camera_name}_body">
+    <!-- stereo section -->
     <sensor type="multicamera" name="stereo_camera">
       <update_rate>30.0</update_rate>
       <camera name="left">
-        <horizontal_fov>1.3962634</horizontal_fov>
-        <image>
-          <width>800</width>
-          <height>800</height>
+        <pose>0 0.0475 0 0 0 0</pose>
+        <horizontal_fov>1.13446</horizontal_fov>
+        <vertical_fov>1.01229</vertical_fov>
+        <image>
+          <width>1280</width>
+          <height>720</height>
           <format>R8G8B8</format>
         </image>
@@ -157,9 +163,10 @@
       </camera>
       <camera name="right">
-        <pose>0 -0.07 0 0 0 0</pose>
-        <horizontal_fov>1.3962634</horizontal_fov>
-        <image>
-          <width>800</width>
-          <height>800</height>
+        <pose>0 -0.0475 0 0 0 0</pose>
+        <horizontal_fov>1.13446</horizontal_fov>
+        <vertical_fov>1.01229</vertical_fov>
+        <image>
+          <width>1280</width>
+          <height>720</height>
           <format>R8G8B8</format>
         </image>
@@ -180,6 +187,5 @@
         <imageTopicName>image_raw</imageTopicName>
         <cameraInfoTopicName>camera_info</cameraInfoTopicName>
-        <frameName>/driver_side_camera_optical</frameName>
-        <!--<rightFrameName>right_camera_optical_frame</rightFrameName>-->
+        <frameName>gazebo_stereo_camera_optical_frame</frameName>
         <hackBaseline>0.07</hackBaseline>
         <distortionK1>0.0</distortionK1>
@@ -190,6 +196,45 @@
       </plugin>
     </sensor>
-  </gazebo>
-  <!-- /sctebot/multisense_sl/camera/left/image_raw -->
+    <!-- mono section -->
+    <sensor type="camera" name="mono_color_camera">
+      <visualize>true</visualize>
+      <update_rate>30.0</update_rate>
+      <camera name="mono_color">
+        <pose>0 0 0 0 0 0</pose>
+        <horizontal_fov>1.20428</horizontal_fov>
+        <vertical_fov>0.733038</vertical_fov>
+        <image>
+          <width>1920</width>
+          <height>1080</height>
+          <format>R8G8B8</format>
+        </image>
+        <clip>
+          <near>0.02</near>
+          <far>300</far>
+        </clip>
+        <noise>
+          <type>gaussian</type>
+          <mean>0.0</mean>
+          <stddev>0.007</stddev>
+        </noise>
+      </camera>
+      <plugin name="camera_controller" filename="libgazebo_ros_camera.so">
+        <alwaysOn>true</alwaysOn>
+        <updateRate>10.0</updateRate>
+        <cameraName>stereo_fwd/color</cameraName>
+        <imageTopicName>image_raw</imageTopicName>
+        <cameraInfoTopicName>camera_info</cameraInfoTopicName>
+        <frameName>gazebo_stereo_camera_optical_frame</frameName>
+        <hackBaseline>0.07</hackBaseline>
+        <distortionK1>0.0</distortionK1>
+        <distortionK2>0.0</distortionK2>
+        <distortionK3>0.0</distortionK3>
+        <distortionT1>0.0</distortionT1>
+        <distortionT2>0.0</distortionT2>
+      </plugin>
+    </sensor>
+  </gazebo>
+  <!-- endregion -->
+  <!-- region LIDAR -->
   <!-- hokuyo
   Noise parameters based on published spec for Hokuyo laser
@@ -232,4 +277,6 @@
   </gazebo>
   -->
+  <!-- endregion -->
+  <!-- region 1D LIDAR -->
   <gazebo reference="laser_frame">
     <material>Gazebo/FlatBlack</material>
@@ -284,3 +331,4 @@
     </sensor>
   </gazebo>
+  <!-- endregion -->
 </robot>

File: sctebot_sensors/logitech_c270_camera/urdf/logitech_c270.xacro (robot description, xacro)
@@ -52,5 +52,5 @@
         </link>
         <joint name="${camera_link}_base_TO_${camera_link}_body" type="fixed">
-            <origin xyz="0.03 0.015 0.0" rpy="0 0 0"/> <!-- ${M_PI/-2} 0 ${M_PI/-2} -->
+            <origin xyz="0.03 0.015 0.0" rpy="0 0 0"/>
             <parent link="${camera_link}_body"/>
             <child link="${camera_link}_base"/>
