Commit message: updated urdf model to reflect current sctebot configuration. Found a height mapped model for gazebo to sim within. Working on integrating it.

File: sctebot_description/urdf/equipment/computer_enclosure.xacro (robot description, xacro)
@@ -1,8 +1,11 @@
 <?xml version="1.0"?>
 <robot name="sctebot" xmlns:xacro="http://www.ros.org/wiki/xacro">
-    <xacro:macro name="computer_enclosure" params="link_name parent_link
-    enclosure_origin
-    enclosure_rpy
-    ">
+    <xacro:macro name="computer_enclosure"
+                 params="
+                 link_name
+                 parent_link
+                 enclosure_origin
+                 enclosure_rpy
+                 enclosure_size">
         <link name="${link_name}">
             <inertial>
@@ -18,5 +21,6 @@
                 <origin xyz="0 0 0" rpy="0 0 0"/>
                 <geometry>
-                    <box size="0.26 0.185 0.06"/>
+                    <!--box size="0.295 0.245 0.116"/-->
+                    <box size="${enclosure_size}"/>
                 </geometry>
                 <material name="none">
@@ -27,5 +31,6 @@
                 <origin xyz="0 0 0" rpy="0 0 0"/>
                 <geometry>
-                    <box size="0.26 0.185 0.06"/>
+                    <!--box size="0.295 0.245 0.116"/-->
+                    <box size="${enclosure_size}"/>
                 </geometry>
             </collision>

File: sctebot_description/urdf/gazebo_sensors/gazebo_stereo_camera.xacro (robot description, xacro)
@@ -1,5 +1,5 @@
 <?xml version='1.0'?>
 <robot name="gazebo_stereo_camera" xmlns:xacro="http://www.ros.org/wiki/xacro">
-    <xacro:macro name="gazebo_stereo_camera" params="parent_link camera_link joint_xyz joint_rpy">
+    <xacro:macro name="gazebo_stereo_camera" params="parent_link camera_link origin_xyz origin_rpy">
         <link name="${camera_link}_body">
             <visual name='visual'>
@@ -18,5 +18,5 @@
         </link>
         <joint name="${camera_link}_TO_${parent_link}" type="fixed">
-            <origin xyz="${joint_xyz}" rpy="${joint_rpy}"/>
+            <origin xyz="${origin_xyz}" rpy="${origin_rpy}"/>
             <parent link="${parent_link}"/>
             <child link="${camera_link}_body"/>

File: sctebot_description/urdf/sctebot_chassis.xacro (robot description, xacro)
@@ -23,5 +23,5 @@
 <robot name="sctebot" xmlns:xacro="http://www.ros.org/wiki/xacro">
     <xacro:arg name="robot_namespace" default="/"/>
-    <xacro:arg name="enable_gazebo_stereo_camera" default="True"/>
+    <xacro:arg name="enable_mock_realsense_camera" default="True"/>
     <xacro:arg name="enable_logitech_stereo_camera" default="False"/>
     <xacro:arg name="enable_realsense_d435i_stereo_camera" default="False"/>
@@ -54,5 +54,5 @@
     <xacro:property name="axle_offset" value="0.05" />
     <xacro:property name="steer_offset" value="0.02" />
-    <!-- scte dims -->
+    <!-- scte dimensions -->
     <xacro:property name="scte_chassis_length_sq" value="${base_length * base_length}"/>
     <xacro:property name="scte_chassis_width_sq" value="${base_width * base_width}"/>
@@ -80,8 +80,4 @@
             </geometry>
         </collision>
-        <!--xacro:solid_cuboid_inertial
-                rpy="0 0 0" xyz="0 0 0"
-                mass="${base_mass}"
-                x="${base_length}" y="${base_width}" z="${base_height}" /-->
     </link>
     <!-- Inertial link stores the robot's inertial information -->
@@ -100,4 +96,5 @@
         <child link="inertial_link" />
     </joint>
+    <!-- region Wheels and Bumpers -->
     <!-- Front steer and rear wheel joints required for ackermann_steering_controller -->
     <xacro:front_steer
@@ -168,5 +165,4 @@
         <origin xyz="${-base_length/2+axle_offset} ${+base_width/2+axle_offset} 0" rpy="${-90 * deg_to_rad} 0 0"/>
     </xacro:rear_wheel_lr>
-    <!-- Bumpers -->
     <xacro:include filename="sctebot_front_bumper.xacro"/>
     <xacro:scte_front_bumper
@@ -187,16 +183,36 @@
             rear_bumper_mount_joint_rpy="0 0 0"
     />
+    <!-- endregion -->
     <!-- Sensors and Compute Hardware -->
+    <xacro:property name="computer_enclosure_length" value="0.295"/>
+    <xacro:property name="computer_enclosure_width" value="0.245"/>
+    <xacro:property name="computer_enclosure_height" value="0.116"/>
     <xacro:include filename="$(find sctebot_description)/urdf/equipment/computer_enclosure.xacro"/>
     <xacro:computer_enclosure
             link_name="computer_enclosure"
             parent_link="base_link"
-            enclosure_origin="0 0 0.105"
+            enclosure_origin="0 0 0.174"
             enclosure_rpy="0 0 0"
+            enclosure_size="${computer_enclosure_length} ${computer_enclosure_width} ${computer_enclosure_height}"
     />
     <!-- region IMU link -->
-    <link name="imu_link"/>
+    <xacro:property name="imu_module_height" value="0.022"/>
+    <link name="imu_link">
+        <visual name='visual'>
+                <origin xyz="0 0 0" rpy="0 0 0"/>
+                <geometry>
+                    <box size="0.06 0.035 ${imu_module_height}"/>
+                </geometry>
+                <material name="blue"/>
+        </visual>
+        <collision name='collision'>
+            <origin xyz="0 0 0" rpy="0 0 0"/>
+            <geometry>
+                <box size="0.06 0.035 ${imu_module_height}"/>
+            </geometry>
+        </collision>
+    </link>
     <joint name="imu_link_TO_computer_enclosure" type="fixed">
-        <origin xyz="0 0 0" rpy="0 0 0"/>
+        <origin xyz="0 0 ${(computer_enclosure_height - imu_module_height) * 0.5}" rpy="0 0 0"/>
         <parent link="computer_enclosure"/>
         <child link="imu_link"/>
@@ -204,7 +220,22 @@
     <!-- endregion -->
     <!-- region GPS link -->
-    <link name="gps_link"/>
+    <xacro:property name="gps_module_height" value="0.022"/>
+    <link name="gps_link">
+        <visual name='visual'>
+                <origin xyz="0 0 0" rpy="0 0 0"/>
+                <geometry>
+                    <box size="0.035 0.06 ${gps_module_height}"/>
+                </geometry>
+                <material name="blue"/>
+        </visual>
+        <collision name='collision'>
+            <origin xyz="0 0 0" rpy="0 0 0"/>
+            <geometry>
+                <box size="0.035 0.06 ${gps_module_height}"/>
+            </geometry>
+        </collision>
+    </link>
     <joint name="gps_link_TO_computer_enclosure" type="fixed">
-        <origin xyz="0 0 0" rpy="0 0 0"/>
+        <origin xyz="-0.125 0.075 ${(computer_enclosure_height + gps_module_height) * 0.5}" rpy="0 0 0"/>
         <parent link="computer_enclosure"/>
         <child link="gps_link"/>
@@ -215,5 +246,5 @@
         <xacro:include filename="$(find ydlidar_ros)/urdf/ydlidar.urdf"/>
         <joint name="ydlidar_base_TO_computer_enclosure" type="fixed">
-            <origin xyz="0.090 0 0.0305" rpy="0 0 0"/> <!--0.0305-->
+            <origin xyz="0 0 ${computer_enclosure_height * 0.5}" rpy="0 0 0"/>
             <parent link="computer_enclosure"/>
             <child link="base_laser"/>
@@ -223,9 +254,21 @@
     <!-- region Stereo Cameras -->
     <!-- region Realsense d435i Stereo Camera -->
+    <xacro:property name="realsense_camera_x_offset" value="${computer_enclosure_length * 0.5 -  0.0125}"/>
+    <xacro:property name="realsense_camera_height" value="0.025"/>
     <xacro:if value="$(arg enable_realsense_d435i_stereo_camera)">
         <xacro:include filename="$(find realsense2_description)/urdf/_d435i.urdf.xacro"/>
         <xacro:sensor_d435i parent="computer_enclosure" name="realsense_d435i">
-            <origin xyz="${(0.26 * 0.5) + (0.02505 * 0.5)} 0 0.005" rpy="0 0 0"/>
+            <origin xyz="${realsense_camera_x_offset} 0 ${(computer_enclosure_height) * 0.5}" rpy="0 0 0"/>
         </xacro:sensor_d435i>
+    </xacro:if>
+    <!-- Gazebo mock Realsense Stereo Camera Sensor -->
+    <xacro:if value="$(arg enable_mock_realsense_camera)">
+        <xacro:include filename="$(find sctebot_description)/urdf/gazebo_sensors/gazebo_stereo_camera.xacro"/>
+        <xacro:gazebo_stereo_camera
+                parent_link="computer_enclosure"
+                camera_link="gazebo_stereo_camera"
+                origin_xyz="${realsense_camera_x_offset} 0 ${(computer_enclosure_height + realsense_camera_height) * 0.5}"
+                origin_rpy="0.0 0.0 0.0"
+        />
     </xacro:if>
     <!-- endregion -->
@@ -238,35 +281,18 @@
         TODO drowan_20220709_BUG: The cameras are mounted incorrectly. Need to fix camera link and/or optical link...
     -->
+    <xacro:property name="logitech_camera_height" value="0.025"/>
     <xacro:if value="$(arg enable_logitech_stereo_camera)">
-        <xacro:include filename="$(find sctebot_description)/urdf/equipment/camera_rig.xacro"/>
-        <xacro:camera_rig
-                link_name="camera_rig"
-                parent_link="computer_enclosure"
-                camera_rig_origin="${0.260 * -0.45} 0 ${0.06 * -0.04}"
-                camera_rig_rpy="0 0 ${pi}"
-        />
         <xacro:include filename="$(find logitech_c270_camera)/urdf/logitech_c270.xacro"/>
         <xacro:logitech_c270_camera
-                parent_link="camera_rig_bar"
+                parent_link="computer_enclosure"
                 camera_link="logitech_driver_side_camera"
-                joint_xyz="0.0 0.05 ${0.025 * 0.5}"
-                joint_rpy="0 0 0"
+                joint_xyz="-0.075 0.125 ${(computer_enclosure_height + logitech_camera_height) * 0.5}"
+                joint_rpy="0 0 ${pi}"
         />
         <xacro:logitech_c270_camera
-                parent_link="camera_rig_bar"
+                parent_link="computer_enclosure"
                 camera_link="logitech_passenger_side_camera"
-                joint_xyz="0.0 -0.05 ${0.025 * 0.5}"
-                joint_rpy="0 0 0"
-        />
-    </xacro:if>
-    <!-- endregion -->
-    <!-- region Gazebo Stereo Camera Sensor -->
-    <xacro:if value="$(arg enable_gazebo_stereo_camera)">
-        <xacro:include filename="$(find sctebot_description)/urdf/gazebo_sensors/gazebo_stereo_camera.xacro"/>
-        <xacro:gazebo_stereo_camera
-                parent_link="computer_enclosure"
-                camera_link="gazebo_stereo_camera"
-                joint_xyz="${(0.26 * 0.5) + (0.02505 * 0.5)} 0 0.018"
-                joint_rpy="0.0 0.0 0.0"
+                joint_xyz="-0.075 -0.125 ${(computer_enclosure_height + logitech_camera_height) * 0.5}"
+                joint_rpy="0 0 ${pi}"
         />
     </xacro:if>

File: sctebot_description/urdf/sctebot_sensors.xacro (robot description, xacro)
@@ -32,6 +32,10 @@
       <topicName>gazebo/gps/fix</topicName>
       <velocityTopicName>gazebo/gps/fix_velocity</velocityTopicName>
-      <referenceLatitude>37.738448530273594</referenceLatitude>
-      <referenceLongitude>-119.56968071496732</referenceLongitude>
+      <!-- Yosemite -->
+      <!--referenceLatitude>37.738448530273594</referenceLatitude>
+      <referenceLongitude>-119.56968071496732</referenceLongitude-->
+      <!-- ksql airport -->
+      <referenceLatitude>37.52207695839262</referenceLatitude>
+      <referenceLongitude>-122.25621399060579</referenceLongitude>
       <referenceHeading>0.0</referenceHeading>
       <referenceLatitude>0.0</referenceLatitude>
