Commit message: minor tweak to gazebo stereo camera orientation

File: sctebot_description/urdf/gazebo_sensors/gazebo_stereo_camera.xacro (robot description, xacro)
@@ -39,5 +39,6 @@
         <joint name="${camera_link}_base_TO_${camera_link}_body" type="fixed">
             <!-- TODO fix the orientation so that the point cloud matches the actual frame -->
-            <origin xyz="0.03 0.015 0.0" rpy="0 1 0"/>
+            <origin xyz="0.01 0.0 0.0" rpy="${(7 * pi) / 2} 0 ${(3 * pi) / 2}"/>
+            <!--origin xyz="0.03 0.015 0.0" rpy="${(7 * pi) / 2} 0 ${(3 * pi) / 2}"/-->
             <parent link="${camera_link}_body"/>
             <child link="${camera_link}_base"/>
